File: Frank/chum-bucket/PCB/CHARGER.sch (KiCad schematic (older format))
At the start: 61 parts, among them Q101 2N7002K, Q102 BSS84, U100 BTS6142DAUMA1, U101 BQ2461x, U102 INA196, U103 CSD87331

Commit message: ready for review? maybe. (not really)
Parts:
- L101: footprint (none) -> CHUM_BUCKET_FOOTPRINTS:PA5005
- R102, R106, R109: footprint (none) -> Resistor_SMD:R_0603_1608Metric
- U103: footprint (none) -> CHUM_BUCKET_FOOTPRINTS:CSD87331Q3D
- gave numbers to parts that had none: 3
Changed lines of the file:
@@
 F 0 "U103" H 6300 2850 50  0000 L CNN
 F 1 "CSD87331" H 6200 2750 50  0000 L CNN
-F 2 "" H 6550 2500 50  0001 C CNN
+F 2 "CHUM_BUCKET_FOOTPRINTS:CSD87331Q3D" H 6550 2500 50  0001 C CNN
 F 3 "http://www.ti.com/lit/ds/symlink/csd87331q3d.pdf?HQS=TI-null-null-digikeymode-df-pf-null-wwe&ts=1591542758219&ref_url=http://www.ti.com/general/docs/suppproductinfo.tsp?distId%3D10&gotoUrl=http://www.ti.com/lit/gpn/csd87331q3d" H 6550 2500 50  0001 C CNN
 F 4 "296-29695-2-ND" H 6550 2500 50  0001 C CNN "Digikey"
@@
 F 0 "L101" V 7440 2750 50  0000 C CNN
 F 1 "4.7uH" V 7349 2750 50  0000 C CNN
-F 2 "" H 7250 2750 50  0001 C CNN
+F 2 "CHUM_BUCKET_FOOTPRINTS:PA5005" H 7250 2750 50  0001 C CNN
 F 3 "https://products.pulseelex.com/files/product_files/P809.pdf" H 7250 2750 50  0001 C CNN
 F 4 "553-4104-2-ND" V 7250 2750 50  0001 C CNN "Digikey"
@@
 F 0 "R106" H 1759 5546 50  0000 L CNN
 F 1 "330" H 1759 5455 50  0000 L CNN
-F 2 "" H 1700 5500 50  0001 C CNN
+F 2 "Resistor_SMD:R_0603_1608Metric" H 1700 5500 50  0001 C CNN
 F 3 "~" H 1700 5500 50  0001 C CNN
 F 4 "0.1%" H 1850 5350 50  0000 C CNN "Tolerance"
@@
 F 0 "R102" H 1409 5546 50  0000 L CNN
 F 1 "3.3k" H 1409 5455 50  0000 L CNN
-F 2 "" H 1350 5500 50  0001 C CNN
+F 2 "Resistor_SMD:R_0603_1608Metric" H 1350 5500 50  0001 C CNN
 F 3 "~" H 1350 5500 50  0001 C CNN
 F 4 "0.1%" H 1500 5350 50  0000 C CNN "Tolerance"
@@
 F 0 "R109" H 1750 5550 50  0000 L CNN
 F 1 "15k" H 1800 5450 50  0000 L CNN
-F 2 "" H 2000 5500 50  0001 C CNN
+F 2 "Resistor_SMD:R_0603_1608Metric" H 2000 5500 50  0001 C CNN
 F 3 "~" H 2000 5500 50  0001 C CNN
 F 4 "0.1%" H 1850 5350 50  0000 C CNN "Tolerance"
@@
 ISET1
 $Comp
-L Connector:TestPoint TP?
+L Connector:TestPoint TP1
 U 1 1 5FA3EAF1
 P 1100 6800
-F 0 "TP?" H 1158 6918 50  0000 L CNN
+F 0 "TP1" H 1158 6918 50  0000 L CNN
 F 1 "VFB" H 1158 6827 50  0000 L CNN
 F 2 "TestPoint:TestPoint_Pad_D1.0mm" H 1300 6800 50  0001 C CNN
@@
 	600  6950 1100 6950
 $Comp
-L Connector:TestPoint TP?
+L Connector:TestPoint TP3
 U 1 1 5FA86C77
 P 7200 5300
-F 0 "TP?" H 7258 5418 50  0000 L CNN
+F 0 "TP3" H 7258 5418 50  0000 L CNN
 F 1 "VFB" H 7258 5327 50  0000 L CNN
 F 2 "TestPoint:TestPoint_Pad_D1.0mm" H 7400 5300 50  0001 C CNN
@@
 	2000 5400 2250 5400
 $Comp
-L Connector:TestPoint TP?
+L Connector:TestPoint TP2
 U 1 1 5FB46CF0
 P 7050 2450
-F 0 "TP?" H 7108 2568 50  0000 L CNN
+F 0 "TP2" H 7108 2568 50  0000 L CNN
 F 1 "SW_NODE" H 7108 2477 50  0000 L CNN
 F 2 "TestPoint:TestPoint_Pad_D1.0mm" H 7250 2450 50  0001 C CNN
