File: Frank/chum-bucket/PCB/CHARGER.sch (KiCad schematic (older format))
At the start: 61 parts, among them Q101 2N7002K, Q102 BSS84, U100 BTS6142DAUMA1, U101 BQ2461x, U102 INA196, U103 CSD87331

Commit message: First Official Schematic Release
yeet
Parts:
- removed R123: 1k, Resistor_SMD:R_0603_1608Metric, symbol Device:R_Small
- added R123: 100, Resistor_SMD:R_0603_1608Metric, symbol Device:R
- added R?: 0, symbol Device:R_Small
- C104, C105: Voltage (none) -> 50V
- C115: Voltage (none) -> 25V
- R124: value 4.7k -> 68k; Digikey RHM4.7DTR-ND -> (none); Power (none) -> 1/10W
- R125: value 1k -> 68k; Power (none) -> 1/10W
Connections:
- net ~AC_DRV: now also R?.1; no longer C119.2, Q102.1 (G), R125.2
- net at C118.2, Q102.3 (D), R124.1: now also R123.1; no longer Q101.1 (G)
- new net: C119.2, Q102.1 (G), R125.2, R?.2
- new net: Q101.1 (G), R123.2
Other:
- moved on the sheet: C118

Commit message: first (hopefully final) routing pass
Parts:
- removed TP3: VFB, TestPoint:TestPoint_Pad_D1.0mm, symbol Connector:TestPoint
- added C120: 0.1uF, Capacitor_SMD:C_0603_1608Metric, symbol Device:C_Small
- added D105, D106: CUS520, Diode_SMD:D_SOD-323, symbol Device:D_Schottky_Small
- added F102: 100mA, Fuse:Fuse_0603_1608Metric, symbol Device:Fuse
- added Q103: SIS413DN, CHUM_BUCKET_FOOTPRINTS:SIS413DN, symbol Device:Q_PMOS_GDS
- added R126: 1k, Resistor_SMD:R_0603_1608Metric, symbol Device:R_Small
- added R127: 100k, Resistor_SMD:R_0603_1608Metric, symbol Device:R_Small
- C109: Voltage 6V -> 10V
- C111: Voltage 25V -> 50V
- L101: value 4.7uH -> 6.8uH; footprint CHUM_BUCKET_FOOTPRINTS:PA5005 -> CHUM_BUCKET_FOOTPRINTS:icantdesignbuckconverters; Digikey 553-4104-2-ND -> 445-SPM10065VT-6R8M-DCT-ND
- R128: renamed from R?; footprint (none) -> Resistor_SMD:R_0603_1608Metric
Connections:
- net +BATT: now also Q103.2 (D)
- net SYS_PWR_OUT: now also C120.1, F102.2, Q103.3 (S), R127.2
- net at R107.2: now also D105.1 (K), D106.1 (K); no longer F101.2
- net AC_FUSED renamed CHG_UNFUSED
- net CHG_UNFUSED: now also F101.2, R114.1, U100.3 (VBB)
- removed net AC_FUSED_IN: F101.1, R114.1, U100.3 (VBB)
- net POWER_GOOD renamed BQ24617_PG
- net ~BQ24617_BATT_DRV renamed ~BATTDRV
- net ~BATTDRV: now also R126.2
- new net: D105.2 (A), F101.1
- new net: D106.2 (A), F102.1
- new net: C120.2, Q103.1 (G), R126.1, R127.1
Other:
- note added: "- ISET1 sets max current during charge (0.5C*8A = 4A)\n- ISET2 sets precharge AND termination charge current (100mA)\n- ACSET sets the max AC adapter current (10A) \n- Place these close to IC"
- note added: "Diode OR the System Bus and AC Charge Power.\nIC pulls from CHG while charging, System otherwise."
- note removed: "- ISET1 sets max current during charge (0.5C*8A = 4A)\n- ISET2 sets precharge AND termination charge current (100mA)\n- ACSET sets the max AC adapter current (10A)"
- moved on the sheet: C103, F101, R107

Commit message: lowered kicad version. Also tided up routing DRC cleared.
Parts:
- U101: symbol chum-bucket:BQ2461x -> chum-bucket-rescue:BQ2461x-chum-bucket
Changed lines of the file:
@@
 $EndComp
 $Comp
-L chum-bucket:BQ2461x U?
+L chum-bucket-rescue:BQ2461x-chum-bucket U?
 U 1 1 5F99F765
 P 5700 2500

Commit message: post-BOM order
Parts:
- C101, C103, C109: Digikey (none) -> 1276-6470-1-ND
- C102: Digikey 399-7874-2-ND -> 399-7874-1-ND
- C104, C108, C113, C114: Digikey 399-7845-2-ND -> 399-7845-1-ND
- C105, C111, C115: value 0.1u -> 0.1uF; Digikey 399-7845-2-ND -> 399-7845-1-ND
- C106, C110, C112, C116, C117: Digikey 478-9622-2-ND -> 478-9622-1-ND
- C107: Digikey 490-1644-2-ND -> 490-1644-1-ND
- C118, C119: Digikey 399-7842-2-ND -> 1276-1009-1-ND
- C120: Digikey (none) -> 399-7845-1-ND
- D101, D102, D103: Digikey 160-1446-2-ND -> 160-1446-1-ND
- D104: Digikey BAT54T1GOSTR-ND -> BAT54T1GOSCT-ND
- D105, D106: Digikey CUS520H3FTR-ND -> CUS520H3FCT-ND
- F101, F102: Digikey 478-6872-2-ND -> 478-6872-1-ND
- Q101: Digikey 2N7002KTR-ND -> 2N7002KCT-ND
- Q102: Digikey BSS84-TPMSTR-ND -> BSS84-TPMSCT-ND
- R101, R105, R108: Digikey (none) -> RNCP0603FTD10K0CT-ND
- R102: Digikey (none) -> 311-3.30KHRCT-ND
- R103: Digikey (none) -> RMCF0603FT499KCT-ND
- R104: Digikey (none) -> RR08P100KDCT-ND
- R106: Digikey (none) -> P19915CT-ND
- R107: Digikey 541-10UATR-ND -> 541-10UACT-ND
- R109: Digikey (none) -> 311-15.0KHRCT-ND
- R110: Digikey P19915TR-ND -> P19915CT-ND
- R111, R113, R115: Digikey (none) -> RHM1.0KDCT-ND; Power (none) -> 1/4W
- R112, R114, R117, R118, R128: Digikey (none) -> RMCF0603ZT0R00CT-ND
- R116, R122: Digikey CRF1206-FZ-R010ELFTR-ND -> CRF1206-FZ-R010ELFCT-ND
- R119: Digikey (none) -> RMCF0603FT9K31CT-ND
- R120: Digikey (none) -> 311-430KGRCT-ND
- R121, R123, RIN_1: Digikey 311-100HRTR-ND -> RMCF0603FT100RCT-ND
- R125: Digikey (none) -> YAG5967CT-ND
- R126: Digikey (none) -> RHM1.0KDCT-ND
- R127: value 100k -> 68k; Digikey (none) -> YAG5967CT-ND; Power (none) -> 1/10W
- TH101: Digikey P12014TR-ND -> P12014CT-ND
- U100: Digikey BTS6142DAUMA1TR-ND -> BTS6142DAUMA1CT-ND
- U101: Digikey 296-25779-2-ND -> 296-25779-1-ND
- U102: Digikey 296-17166-2-ND -> 296-17166-1-ND
- U103: Digikey 296-29695-2-ND -> 296-29695-1-ND
Connections:
- net SYS_PWR_OUT: now also R127.1; no longer R127.2
- net at C120.2, Q103.1 (G), R126.1: now also R127.2; no longer R127.1
