File: Frank/chum-bucket/PCB/MCU.sch (KiCad schematic (older format))
At the start: 47 parts

Commit message: minor schematic update + inrush sim
Parts:
- removed J?: JTAG, symbol Connector_Generic:Conn_02x03_Odd_Even
- added C? (x2): 0.1uF, symbol Device:C_Small
- added D?: D, symbol Device:D_Small
- added D? (x2): D_Z, symbol Device:D_Zener_Small
- added J?: SWD_DIAGS, symbol Connector_Generic:Conn_01x06
- added R? (x2): 100, symbol Device:R
Connections:
- net labels added: ANALOG_I_CHG, ANALOG_I_SYS, STM32_SWCLK, STM32_SWDIO, UART_DIAGS_STM_RX, UART_DIAGS_STM_TX
- wire segments 138 -> 171
Other:
- moved on the sheet: C?, J?, R?, TP?

Commit message: Weekends work. Final component selection then ready for review :)
huge oof
Parts:
- removed C?: 0.1uF, symbol Device:C_Small
- removed C?: 1uF, symbol Device:C_Small
- removed C?: 10uF, symbol Device:C_Small
- removed U?: MIC5283-3.3ML-TR, symbol chum-bucket:MIC5283-3.3ML-TR
- added C?: 0.1uF, symbol Device:C_Small
- added C? (x3): 10nF, symbol Device:C_Small
- added D? (x2): D_Small, symbol Device:D_Small
- added F?: 200mA, symbol Device:Fuse
- added FB?: FB, symbol Device:Ferrite_Bead
- added R?: 10k, symbol Device:R
- added R?: 10k, symbol Device:R_Small
- added SW?: LV_EN, symbol Switch:SW_DIP_x01
- added U?: TPS70933DRVT, Package_SON:WSON-6-1EP_2x2mm_P0.65mm_EP1x1.6mm, symbol chum-bucket:TPS70933DRVT
- F?: value 50mA -> 200mA
- R? (x2): value R_Small -> 1k
Connections:
- net labels added: +BATT, CHG_PWR_UNFUSED, ESC_PWR_EN
- net labels removed: POS_BAT_FUSED
- wire segments 171 -> 189
Other:
- note added: "Diode OR allows 3V3 systems to be powered\neven when there's no battery present"
- note added: "Dip switch to disable \nall 3v3 quiescent current when\nsystem is in storage."
- moved on the sheet: C?, D?, F?, J?, R?, SW?, TP?, U?, Y?

Commit message: batt-management sheet updates
Parts:
- removed C?: 10nF, symbol Device:C_Small
- removed R?: 10k, symbol Device:R_Small
- FB?: value FB -> Choke; footprint (none) -> Inductor_SMD:L_0603_1608Metric; Digikey (none) -> 490-17350-2-ND
- SW?: Digikey (none) -> 563-1004-2-ND
Other:
- note added: "Dip switch to disable \nall 3v3 quiescent current when\nsystem is in storage.\nEN is internally pulled High"
- note removed: "Dip switch to disable \nall 3v3 quiescent current when\nsystem is in storage."
- moved on the sheet: C?, D?, J?, R?

Commit message: Minor schematic organization changes
Parts:
- removed D?: D_Small, symbol Device:D_Small
- removed F?: 200mA, symbol Device:Fuse
- added D?: CUS520, Diode_SMD:D_SOD-323, symbol Device:D_Small
- added F?: 200mA, Fuse:Fuse_0603_1608Metric, symbol Device:Fuse
- D?: value D_Small -> CUS520; footprint (none) -> Diode_SMD:D_SOD-323; Digikey (none) -> CUS520H3FTR-ND
- F?: footprint (none) -> Fuse:Fuse_0603_1608Metric; Digikey (none) -> P15127TR-ND
- FB?: value Choke -> BLM18
- U?: footprint (none) -> Package_DFN_QFN:DFN-8-1EP_3x3mm_P0.65mm_EP1.55x2.4mm; Digikey (none) -> MCP2562FDT-E/MFTR-ND
Connections:
- wire segments 189 -> 188
Other:
- moved on the sheet: C?, D?, J?, R?, SW?, Y?

Commit message: more work
Parts:
- removed C? (x4): 10nF, symbol Device:C_Small
- removed C? (x3): 10p, symbol Device:C_Small
- removed C? (x3): 1uF, symbol Device:C_Small
- removed D?: D, symbol Device:D_Small
- removed D? (x2): CUS520, Diode_SMD:D_SOD-323, symbol Device:D_Small
- removed D? (x2): LED, symbol Device:LED
- removed D?: D_Z, symbol Device:D_Zener_Small
- removed R? (x2): R, symbol Device:R
- removed R? (x2): 1k, symbol Device:R_Small
- removed R? (x2): 10k, symbol Device:R_Small
- removed SW?: SW_SPST, symbol Switch:SW_SPST
- removed U?: MCP2562, Package_DFN_QFN:DFN-8-1EP_3x3mm_P0.65mm_EP1.55x2.4mm, symbol chum-bucket:MCP2562
- added C224, C249, C255, C256: 10nF, Capacitor_SMD:C_0603_1608Metric, symbol Device:C_Small
- added C242, C248: 0.1uF, Capacitor_SMD:C_0603_1608Metric, symbol Device:C_Small
- added C243: 10p, Capacitor_SMD:C_0603_1608Metric, symbol Device:C_Small
- added C245, C246, C247: 1uF, Capacitor_SMD:C_0805_2012Metric, symbol Device:C_Small
- added D208, D209, D214, D?: CUS520, Diode_SMD:D_SOD-323, symbol Device:D_Schottky_Small
- added D210, D211: GN, LED_SMD:LED_0603_1608Metric, symbol Device:D_Small
- added D213: BZT52, Diode_SMD:D_SOD-123, symbol Device:D_Zener_Small
- added R251, R252, R253, R254: 1k, Resistor_SMD:R_0603_1608Metric, symbol Device:R_Small
- added R271: 0, Resistor_SMD:R_0603_1608Metric, symbol Device:R
- added R?: 10k, Resistor_SMD:R_0603_1608Metric, symbol Device:R_Small
- added SW201: B3U-1000P, Button_Switch_SMD:SW_SPST_B3U-1000P, symbol Switch:SW_SPST
- added U?: SN65HVD232, Package_SO:SOIC-8_3.9x4.9mm_P1.27mm, symbol Interface_CAN_LIN:SN65HVD232
- C241: renamed from C?; footprint (none) -> Capacitor_SMD:C_0603_1608Metric; Digikey (none) -> 311-1058-2-ND; Tolerance (none) -> C0G
- C250, C251, C254, C257: renamed from C?; footprint (none) -> Capacitor_SMD:C_0603_1608Metric
- C252: renamed from C?; value 0.1uF -> 10nF; footprint (none) -> Capacitor_SMD:C_0603_1608Metric
- D212: renamed from D?; value D_Z -> BZT52; footprint (none) -> Diode_SMD:D_SOD-123
- R257, R258, R259, R260, R261, R262, R263, R264, R265, R266, R267, R268, R269, R270: renamed from R?; footprint (none) -> Resistor_SMD:R_0603_1608Metric
- SW203: renamed from SW?; footprint (none) -> Button_Switch_SMD:SW_SPST_B3U-1000P; Digikey (none) -> SW1020CT-ND
- TP201: renamed from TP?; value TP_1 -> STM_RX; footprint (none) -> TestPoint:TestPoint_Pad_D1.0mm
- TP202: renamed from TP?; value TP_1 -> STM_TX; footprint (none) -> TestPoint:TestPoint_Pad_D1.0mm
- TP203: renamed from TP?; value TP_1 -> BQ_Wake; footprint (none) -> TestPoint:TestPoint_Pad_D1.0mm
- TP204: renamed from TP?; value TP_1 -> BQ_Fault; footprint (none) -> TestPoint:TestPoint_Pad_D1.0mm
- Y201: renamed from Y?; value Crystal -> 32MHz; Digikey (none) -> XC3036TR-ND
- gave numbers to parts that had none: 9
Connections:
- net labels removed: ~MCP2562_SHDN
- wire segments 188 -> 185
- no-connect marks 1 -> 0
Other:
- note added: "Place RC of analog pins near MCU"
- note removed: "DNC"
- moved on the sheet: C241, C250, C251, C252, C253, C254, C257, D212, J205, J206, R257, R258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

Commit message: more changes :)
Parts:
- added C?: 0.1uF, Capacitor_SMD:C_0603_1608Metric, symbol Device:C_Small
- added D?: BZT52, Diode_SMD:D_SOD-123, symbol Device:D_Zener_Small
- added R? (x3): 100, Resistor_SMD:R_0603_1608Metric, symbol Device:R
Connections:
- net ANALOG_I_CHG: now also C257.1, D213.1 (K), R266.2
- net ANALOG_I_SYS: now also C254.1, D212.1 (K), R265.2
- net BQ_24617_CHG_EN: no longer C254.1, C257.1, D212.1 (K), D213.1 (K), R265.2, R266.2
- net GND: now also C?.2, D?.2 (A)
- new net ANALOG_I_ESCS: C?.1, D?.1 (K), R?.1, R?.2
- new net ANALOG_V_ESCS: R?.1
- new net ANALOG_V_SYSTEM: R?.1, R?.2
Other:
- moved on the sheet: C252, C253, C254, C257, D212, D213, R257, R259, R265, R266

Commit message: changes
Parts:
- removed C250: 0.1uF, Capacitor_SMD:C_0603_1608Metric, symbol Device:C_Small
- removed D210, D211: GN, LED_SMD:LED_0603_1608Metric, symbol Device:D_Small
- added C? (x2): 0.1uF, Capacitor_SMD:C_0603_1608Metric, symbol Device:C_Small
- added D210, D211, D? (x3): GN, Diode_SMD:D_0603_1608Metric, symbol Device:LED_Small
- added D? (x2): BZT52, Diode_SMD:D_SOD-123, symbol Device:D_Zener_Small
- added R? (x2): 10k, Resistor_SMD:R_0603_1608Metric, symbol Device:R_Small
- added R?: 1k, Resistor_SMD:R_0603_1608Metric, symbol Device:R_Small
- added TP?: TP_I_CHARGE, TestPoint:TestPoint_Pad_D1.0mm, symbol Connector:TestPoint
- added TP?: TP_I_SYS, TestPoint:TestPoint_Pad_D1.0mm, symbol Connector:TestPoint
- added TP?: TP_I_ESCS, TestPoint:TestPoint_Pad_D1.0mm, symbol Connector:TestPoint
- C253: footprint (none) -> Capacitor_SMD:C_0603_1608Metric
- J206: footprint (none) -> Connector_PinHeader_1.27mm:PinHeader_2x03_P1.27mm_Vertical; Digikey (none) -> 2057-HPH2-A-04-UA-ND
- SW203: value SW_SPST -> B3U-1000P
- TP201, TP202: footprint TestPoint:TestPoint_Pad_D1.0mm -> TestPoint:TestPoint_Keystone_5000-5004_Miniature; Digikey (none) -> 36-5001-ND
Connections:
- net +3V3: now also D?.2 (A), D?.2 (A)
- net ANALOG_I_CHG: now also TP?.1
- net ANALOG_I_ESCS: now also TP?.1
- net ANALOG_I_SYS: now also TP?.1
- net ANALOG_V_ESCS: now also R?.2, C?.1, D?.1 (K)
- net ANALOG_V_SYSTEM: now also C?.1, D?.1 (K)
- net GND: now also C?.2, C?.2, D210.1 (K), D211.1 (K), D?.1 (K), D?.2 (A), D?.2 (A)
- net UART_CAN_STM_RX: now also R?.2
- net UART_CAN_STM_TX: now also R?.2
- net at C249.2, FB201.1, U216.1 (OUT): now also R?.1
- net at R252.2: now also D210.2 (A)
- net at R253.2: now also D211.2 (A)
- net ~RESET: now reaches C242.2, R251.2, SW201.1 (A), U215.4 (NRST)
- new net: D?.1 (K), R?.1 (x2)
- new net: D?.2 (A), R?.2
Other:
- note added: "Add formulas for TPs on SS. \nNo need for voltage TPs"
- moved on the sheet: C224, C241, C242, C243, C245, C246, C247, C249, C251, C252, C253, C254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

Commit message: ready for review? maybe. (not really)
Parts:
- removed Y201: 32MHz, symbol Device:Crystal
- added Y201: XTAL, CHUM_BUCKET_FOOTPRINTS:ECX-1048, symbol Device:Crystal_GND24_Small
- C224: value 10nF -> 1uF
- C249: value 10nF -> 2.2uF
- J205: footprint (none) -> Connector_JST:JST_SH_SM04B-SRSS-TB_1x04-1MP_P1.00mm_Horizontal; Digikey (none) -> 455-1422-2-ND
- SW202: footprint (none) -> CHUM_BUCKET_FOOTPRINTS:CHS-01TB; Digikey 563-1004-2-ND -> 563-1003-2-ND
- gave numbers to parts that had none: 21
Connections:
- net GND: now also Y201.4
- net XTAL_N: now also Y201.3
- net XTAL_P: now also Y201.1
- no-connect marks 0 -> 1
