File: Frank/chum-bucket/PCB/MCU.sch (KiCad schematic (older format))
At the start: 85 parts, among them J205 CAN_CONN, J206 SWD_DIAGS, Q201 BSS84, SW201 B3U-1000P, SW202 LV_EN, SW203 B3U-1000P, U2 SN65HVD232, U215 STM32F042K6Tx, U216 TPS70933DRVT, Y201 XTAL

Commit message: routing V2
Parts:
- Y201: Freq (none) -> 32MHz
Connections:
- net ANALOG_I_CHG: no longer C257.1, D213.1 (K), R266.2, U215.11 (PA5)
- net ANALOG_I_ESCS: no longer C17.1, D9.1 (K), R12.2, U215.10 (PA4)
- net ANALOG_I_SYS: no longer C254.1, D212.1 (K), R265.2, U215.7 (PA1)
- net ANALOG_V_ESCS: no longer C16.1, D8.1 (K), R11.2, U215.9 (PA3)
- net ANALOG_V_SYSTEM: no longer C15.1, D7.1 (K), R10.2, U215.6 (PA0)
- net BQ24617_PG: now also TP204.1; no longer R1.2, U215.28 (PB5)
- net BQ79606_WAKE: no longer C255.2, R262.2, R269.2, TP203.1, U215.15 (PB1)
- net BQ_24617_CHG_EN: no longer C253.1, R259.1, R264.2, U215.13 (PA7)
- net ESC_PWR_EN: no longer C252.1, R257.1, R271.2, U215.12 (PA6)
- net ~BQ79606_FAULT: now also TP203.1; no longer C256.2, R263.2, R270.2, TP204.1, U215.14 (PB0)
- new net ANALOG_I_CHG_JMP: C257.1, D213.1 (K), R266.2, U215.11 (PA5)
- new net ANALOG_I_ESCS_JMP: C17.1, D9.1 (K), R12.2, U215.10 (PA4)
- new net ANALOG_I_SYS_JMP: C254.1, D212.1 (K), R265.2, U215.7 (PA1)
- new net ANALOG_V_ESCS_JMP: C16.1, D8.1 (K), R11.2, U215.9 (PA3)
- new net ANALOG_V_SYSTEM_JMP: C15.1, D7.1 (K), R10.2, U215.6 (PA0)
- new net BQ24617_PG_JMP: R1.2, U215.28 (PB5)
- new net BQ79606_WAKE_JMP: C255.2, R262.2, R269.2, U215.15 (PB1)
- new net BQ_24617_CHG_EN_JMP: C253.1, R259.1, R264.2, U215.13 (PA7)
- new net ESC_PWR_EN_JMP: C252.1, R257.1, R271.2, U215.12 (PA6)
- new net ~BQ79606_FAULT_JMP: C256.2, R263.2, R270.2, U215.14 (PB0)
Other:
- note removed: "Add formulas for TPs on SS. \nNo need for voltage TPs"
- moved on the sheet: C15, C17, C245, C246, C247, C252, C253, C254, C255, C256, C257, D212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

Commit message: routing v2.1.
Parts:
- removed C17: 0.1uF, Capacitor_SMD:C_0603_1608Metric, symbol Device:C_Small
- removed D9: BZT52, Diode_SMD:D_SOD-123, symbol Device:D_Zener_Small
- removed R12: 100, Resistor_SMD:R_0603_1608Metric, symbol Device:R
- TP210: value TP_I_ESCS -> TestPoint
Connections:
- net ANALOG_I_ESCS_JMP is gone; now on net STM_PA4: U215.10 (PA4)
- net ANALOG_I_ESCS renamed STM_PA4
Other:
- moved on the sheet: C15, C16, C254, C257, D212, D213, D7, D8, R10, R11, R265, R266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

Commit message: post-BOM order
Parts:
- C15, C16, C251, C254, C257: Digikey (none) -> 399-7845-1-ND
- C201, C252, C253: Digikey (none) -> 1276-1009-1-ND
- C241, C243: Digikey 311-1058-2-ND -> 311-1058-1-ND
- C242, C248: Digikey 399-7845-2-ND -> 399-7845-1-ND
- C245, C246, C247: Digikey (none) -> 1276-6470-1-ND
- C249: Digikey 399-7842-2-ND -> 1276-2016-1-ND
- C255, C256: Digikey 399-7842-2-ND -> 1276-1009-1-ND
- D201: Digikey (none) -> 732-4978-1-ND
- D208, D209, D214, D6: Digikey CUS520H3FTR-ND -> CUS520H3FCT-ND
- D210, D211, D3, D4, D5: Digikey 160-1446-2-ND -> 160-1446-1-ND
- D212, D213, D7: Digikey (none) -> BZT52C3V6-FDICT-ND
- F202, F203: Digikey P15127TR-ND -> P15127CT-ND
- FB201: Digikey 490-17350-2-ND -> 490-17350-1-ND
- J205: Digikey 455-1422-2-ND -> 455-1422-1-ND
- J206: Digikey 2057-HPH2-A-04-UA-ND -> S9015E-03-ND
- Q201: Digikey BSS84-TPMSTR-ND -> BSS84-TPMSCT-ND
- R1, R264, R267, R268, R269, R270, R271: Digikey (none) -> RMCF0603ZT0R00CT-ND
- R10, R11, R265, R266: Digikey (none) -> RMCF0603FT100RCT-ND
- R201, R251, R252, R253, R254, R9: Digikey (none) -> RHM1.0KDCT-ND
- R257, R259, R262, R263, R6, R7, R8: Digikey (none) -> RNCP0603FTD10K0CT-ND
- R258: Digikey (none) -> 311-120HRCT-ND
- SW202: Digikey 563-1003-2-ND -> 563-1003-1-ND
- U2: Digikey (none) -> 296-12282-5-ND
- U215: Digikey (none) -> 497-STM32F042K6T6CT-ND
- U216: Digikey 296-37252-2-ND -> 296-37252-1-ND
- Y201: Digikey XC3036TR-ND -> XC3036CT-ND
Other:
- moved on the sheet: C15, C16, C254, C257, D212, D213, D7, D8, R10, R11, R265, R266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
