File: Frank/chum-bucket/PCB/chum-bucket.sch (KiCad schematic (older format))
At the start: 7 parts

Commit message: more work
Parts:
- C202: renamed from C?; value 470uF -> 100uF; footprint (none) -> Capacitor_THT:CP_Radial_D8.0mm_P3.50mm; Digikey P15451TR-ND -> 1189-1662-1-ND; Voltage (none) -> 50V
- gave numbers to parts that had none: 6
Connections:
- net CHARGER/AC_FUSED_IN: now also C202.1
Other:
- note added: "Chum Bucket Features:\n- 3s8p Lithium Cell config\n- 1A Balancing Current\n- 8A (1C) cell charging\n- 1kW peak power delievery\n- e-fused I/O for decreased footprint\n- Power telemetry broadcasted via CAN"
- note added: "Key for Component Names:\nEG: CYXX (X being sequential number)\nY Numbers:\n0: General Peripheral\n1: Charger IC\n2: MCU and Signal I/O\n3: Battery Management\n4: Power Management and Output Protections\n(Capacitor voltage ratings given as minimums)\n"
- note added: "No need to fuse due to use of \nconventionial and e-fuses downstream.\nTVS diode supress plug in transients\nTVS, MLCC then CP placed close to power inputs"
- note removed: "- 1kW peak power delievery\n- e-fused I/O for decreased footprint\n- Power telemetry broadcasted via CAN"
- note removed: "- 3s8p Lithium cell holders\n- 1A Balancing Current\n- 8A cell charging"
- note removed: "No need to fuse due to use of \nconventionial and e-fuses downstream.\nTVS diode supress plug in transients"
Changed lines of the file:
@@
 P 1200 2750
 AR Path="/5ECF1AA9/5FA029D9" Ref="#PWR?"  Part="1"
-AR Path="/5FA029D9" Ref="#PWR?"  Part="1"
-F 0 "#PWR?" H 1200 2500 50  0001 C CNN
+AR Path="/5FA029D9" Ref="#PWR0201"  Part="1"
+F 0 "#PWR0201" H 1200 2500 50  0001 C CNN
 F 1 "GND" H 1205 2577 50  0000 C CNN
 F 2 "" H 1200 2750 50  0001 C CNN
@@
 P 900 2650
 AR Path="/5ECF1AA9/5FA029DF" Ref="J?"  Part="1"
-AR Path="/5FA029DF" Ref="J?"  Part="1"
-F 0 "J?" H 818 2325 50  0000 C CNN
+AR Path="/5FA029DF" Ref="J201"  Part="1"
+F 0 "J201" H 818 2325 50  0000 C CNN
 F 1 "AC_ADPTR" H 818 2416 50  0000 C CNN
 F 2 "" H 900 2650 50  0001 C CNN
@@
 	-1   0    0    1
 $EndComp
-Text Notes 5100 1000 0    157  ~ 31
+Text Notes 4900 950  0    157  ~ 31
 CHUM BUCKET
-Text Notes 4200 1200 0    79   ~ 0
+Text Notes 4000 1150 0    79   ~ 0
 Highly Integrated, Small Footprint, Managed Lithium Battery
-Text Notes 4900 1550 0    39   ~ 0
-- 3s8p Lithium cell holders\n- 1A Balancing Current\n- 8A cell charging
-Text Notes 6150 1550 0    39   ~ 0
-- 1kW peak power delievery\n- e-fused I/O for decreased footprint\n- Power telemetry broadcasted via CAN
+Text Notes 4600 1750 0    39   ~ 0
+Chum Bucket Features:\n- 3s8p Lithium Cell config\n- 1A Balancing Current\n- 8A (1C) cell charging\n- 1kW peak power delievery\n- e-fused I/O for decreased footprint\n- Power telemetry broadcasted via CAN
+Text Notes 6000 1850 0    39   ~ 0
+Key for Component Names:\nEG: CYXX (X being sequential number)\nY Numbers:\n0: General Peripheral\n1: Charger IC\n2: MCU and Signal I/O\n3: Battery Management\n4: Power Management and Output Protections\n(Capacitor voltage ratings given as minimums)\n
 Text Notes 7900 3200 0    118  ~ 24
 SYS MGMT +\nOUTPUT PROT
@@
 P 1200 3450
 AR Path="/5ECF1AA9/5EF08F0F" Ref="#PWR?"  Part="1"
-AR Path="/5EF08F0F" Ref="#PWR?"  Part="1"
-F 0 "#PWR?" H 1200 3200 50  0001 C CNN
+AR Path="/5EF08F0F" Ref="#PWR0202"  Part="1"
+F 0 "#PWR0202" H 1200 3200 50  0001 C CNN
 F 1 "GND" H 1205 3277 50  0000 C CNN
 F 2 "" H 1200 3450 50  0001 C CNN
@@
 P 900 3350
 AR Path="/5ECF1AA9/5EF08F15" Ref="J?"  Part="1"
-AR Path="/5EF08F15" Ref="J?"  Part="1"
-F 0 "J?" H 818 3025 50  0000 C CNN
+AR Path="/5EF08F15" Ref="J202"  Part="1"
+F 0 "J202" H 818 3025 50  0000 C CNN
 F 1 "WPT_CONN" H 818 3116 50  0000 C CNN
 F 2 "" H 900 3350 50  0001 C CNN
@@
 $EndComp
 Text Notes 1450 2400 0    39   ~ 0
-No need to fuse due to use of \nconventionial and e-fuses downstream.\nTVS diode supress plug in transients
+No need to fuse due to use of \nconventionial and e-fuses downstream.\nTVS diode supress plug in transients\nTVS, MLCC then CP placed close to power inputs
 Wire Wire Line
 	1100 3250 1450 3250
@@
 P 10300 2650
 AR Path="/5ECF1AA9/5F3C2735" Ref="#PWR?"  Part="1"
-AR Path="/5F3C2735" Ref="#PWR?"  Part="1"
-F 0 "#PWR?" H 10300 2400 50  0001 C CNN
+AR Path="/5F3C2735" Ref="#PWR0206"  Part="1"
+F 0 "#PWR0206" H 10300 2400 50  0001 C CNN
 F 1 "GND" H 10305 2477 50  0000 C CNN
 F 2 "" H 10300 2650 50  0001 C CNN
@@
 P 10650 2550
 AR Path="/5ECF1AA9/5F3C273B" Ref="J?"  Part="1"
-AR Path="/5F3C273B" Ref="J?"  Part="1"
-F 0 "J?" H 10568 2225 50  0000 C CNN
+AR Path="/5F3C273B" Ref="J203"  Part="1"
+F 0 "J203" H 10568 2225 50  0000 C CNN
 F 1 "SYS_PWR" H 10568 2316 50  0000 C CNN
 F 2 "" H 10650 2550 50  0001 C CNN
@@
 P 10300 3350
 AR Path="/5ECF1AA9/5F3C2743" Ref="#PWR?"  Part="1"
-AR Path="/5F3C2743" Ref="#PWR?"  Part="1"
-F 0 "#PWR?" H 10300 3100 50  0001 C CNN
+AR Path="/5F3C2743" Ref="#PWR0207"  Part="1"
+F 0 "#PWR0207" H 10300 3100 50  0001 C CNN
 F 1 "GND" H 10305 3177 50  0000 C CNN
 F 2 "" H 10300 3350 50  0001 C CNN
@@
 P 10650 3250
 AR Path="/5ECF1AA9/5F3C2749" Ref="J?"  Part="1"
-AR Path="/5F3C2749" Ref="J?"  Part="1"
-F 0 "J?" H 10568 2925 50  0000 C CNN
+AR Path="/5F3C2749" Ref="J204"  Part="1"
+F 0 "J204" H 10568 2925 50  0000 C CNN
 F 1 "ESC_PWR" H 10568 3016 50  0000 C CNN
 F 2 "" H 10650 3250 50  0001 C CNN
@@
 P 1900 2850
 AR Path="/5F507ADF/5EFB8FC1" Ref="D?"  Part="1"
-AR Path="/5EFB8FC1" Ref="D?"  Part="1"
-F 0 "D?" V 1854 2929 50  0000 L CNN
+AR Path="/5EFB8FC1" Ref="D201"  Part="1"
+F 0 "D201" V 1854 2929 50  0000 L CNN
 F 1 "SMBJ26A" V 1945 2929 50  0000 L CNN
 F 2 "Diode_SMD:D_SMB" H 1900 2850 50  0001 C CNN
@@
 P 1900 3100
 AR Path="/5F507ADF/5EFB8FC7" Ref="#PWR?"  Part="1"
-AR Path="/5EFB8FC7" Ref="#PWR?"  Part="1"
-F 0 "#PWR?" H 1900 2850 50  0001 C CNN
+AR Path="/5EFB8FC7" Ref="#PWR0203"  Part="1"
+F 0 "#PWR0203" H 1900 2850 50  0001 C CNN
 F 1 "GND" H 1905 2927 50  0000 C CNN
 F 2 "" H 1900 3100 50  0001 C CNN
@@
 P 2100 2850
 AR Path="/5F507ADF/5EFB8FCE" Ref="C?"  Part="1"
-AR Path="/5EFB8FCE" Ref="C?"  Part="1"
-F 0 "C?" H 2192 2896 50  0000 L CNN
+AR Path="/5EFB8FCE" Ref="C201"  Part="1"
+F 0 "C201" H 2192 2896 50  0000 L CNN
 F 1 "10nF" H 2192 2805 50  0000 L CNN
 F 2 "" H 2100 2850 50  0001 C CNN
@@
 P 2100 3100
 AR Path="/5F507ADF/5EFB8FD4" Ref="#PWR?"  Part="1"
-AR Path="/5EFB8FD4" Ref="#PWR?"  Part="1"
-F 0 "#PWR?" H 2100 2850 50  0001 C CNN
+AR Path="/5EFB8FD4" Ref="#PWR0204"  Part="1"
+F 0 "#PWR0204" H 2100 2850 50  0001 C CNN
 F 1 "GND" H 2105 2927 50  0000 C CNN
 F 2 "" H 2100 3100 50  0001 C CNN
@@
 Connection ~ 2100 2550
 Wire Wire Line
-	2100 2550 2850 2550
+	2100 2550 2450 2550
 Wire Wire Line
 	1450 2550 1900 2550
@@
 P 2450 3100
 AR Path="/5F507ADF/5EF84B97" Ref="#PWR?"  Part="1"
-AR Path="/5EF84B97" Ref="#PWR?"  Part="1"
-F 0 "#PWR?" H 2450 2850 50  0001 C CNN
+AR Path="/5EF84B97" Ref="#PWR0205"  Part="1"
+F 0 "#PWR0205" H 2450 2850 50  0001 C CNN
 F 1 "GND" H 2455 2927 50  0000 C CNN
 F 2 "" H 2450 3100 50  0001 C CNN
@@
 Wire Wire Line
 	2450 3100 2450 2950
-Wire Wire Line
-	2450 2750 2450 2550
-$Comp
-L Device:CP_Small C?
+$Comp
+L Device:CP_Small C202
 U 1 1 5EF85CBA
 P 2450 2850
-F 0 "C?" H 2538 2896 50  0000 L CNN
-F 1 "470uF" H 2538 2805 50  0000 L CNN
-F 2 "" H 2450 2850 50  0001 C CNN
-F 3 "~" H 2450 2850 50  0001 C CNN
+F 0 "C202" H 2538 2896 50  0000 L CNN
+F 1 "100uF" H 2538 2805 50  0000 L CNN
+F 2 "Capacitor_THT:CP_Radial_D8.0mm_P3.50mm" H 2450 2850 50  0001 C CNN
+F 3 "http://www.rubycon.co.jp/en/catalog/e_pdfs/aluminum/e_ZLJ.pdf" H 2450 2850 50  0001 C CNN
 F 4 "P15451TR-ND" H 2450 2850 50  0001 C CNN "Digikey"
+F 5 "50V" H 2600 2700 50  0000 C CNN "Voltage"
+F 6 "1189-1662-1-ND" H 2450 2850 50  0001 C CNN "Digikey"
 	1    2450 2850
 	1    0    0    -1
 $EndComp
+Wire Wire Line
+	2450 2750 2450 2550
+Connection ~ 2450 2550
+Wire Wire Line
+	2450 2550 2850 2550
 $EndSCHEMATC

Commit message: more changes :)
Other:
- note added: "MCU"
- note added: "SYS MGMT"
- note removed: "MCU & I/O"
- note removed: "SYS MGMT +\nOUTPUT PROT"
- note removed: "To do: \n- add voltage monitoring for output busses\n- add current monitoring for ESC bus (hall effect sensor?)"
Changed lines of the file:
@@
 Comment4 ""
 $EndDescr
-Text Notes 4750 4400 0    118  ~ 24
-MCU & I/O
+Text Notes 5050 4450 0    118  ~ 24
+MCU
 Text Notes 4950 5900 0    118  ~ 24
 CELLS
@@
 Text Notes 6000 1850 0    39   ~ 0
 Key for Component Names:\nEG: CYXX (X being sequential number)\nY Numbers:\n0: General Peripheral\n1: Charger IC\n2: MCU and Signal I/O\n3: Battery Management\n4: Power Management and Output Protections\n(Capacitor voltage ratings given as minimums)\n
-Text Notes 7900 3200 0    118  ~ 24
-SYS MGMT +\nOUTPUT PROT
+Text Notes 8250 2950 0    118  ~ 24
+SYS MGMT
 Wire Wire Line
 	6350 2550 7550 2550
@@
 F5 "ESC_PWR_EN" I L 7550 3350 50
 F6 "~BQ24617_BAT_DRV" I L 7550 2650 50
+F7 "ANALOG_I_ESCS" I L 7550 3250 50
+F8 "ANALOG_V_SYSTEM" I L 7550 3050 50
+F9 "ANALOG_V_ESCS" I L 7550 3150 50
 $EndSheet
 Wire Wire Line
@@
 Wire Wire Line
 	6700 3200 6350 3200
-Wire Wire Line
-	6350 4150 6850 4150
-Wire Wire Line
-	6850 4150 6850 3350
-Wire Wire Line
-	6850 3350 7550 3350
 Connection ~ 1450 2550
 Wire Wire Line
@@
 F8 "ANALOG_I_CHG" I R 6350 4050 50
 F9 "CHG_PWR_UNFUSED" I L 4150 3900 50
-F10 "ESC_PWR_EN" I R 6350 4150 50
+F10 "ESC_PWR_EN" I R 6350 4450 50
+F11 "ANALOG_I_ESCS" I R 6350 4350 50
+F12 "ANALOG_V_SYSTEM" I R 6350 4150 50
+F13 "ANALOG_V_ESCS" I R 6350 4250 50
 $EndSheet
 $Comp
@@
 Wire Wire Line
 	1900 2550 2100 2550
-Text Notes 7650 4250 0    50   Italic 0
-To do: \n- add voltage monitoring for output busses\n- add current monitoring for ESC bus (hall effect sensor?)
 $Comp
 L power:GND #PWR?
@@
 Wire Wire Line
 	2450 2550 2850 2550
+Wire Wire Line
+	6350 4150 6800 4150
+Wire Wire Line
+	6800 4150 6800 3050
+Wire Wire Line
+	6800 3050 7550 3050
+Wire Wire Line
+	6350 4250 6900 4250
+Wire Wire Line
+	6900 4250 6900 3150
+Wire Wire Line
+	6900 3150 7550 3150
+Wire Wire Line
+	6350 4350 7000 4350
+Wire Wire Line
+	7000 4350 7000 3250
+Wire Wire Line
+	7000 3250 7550 3250
+Wire Wire Line
+	6350 4450 7100 4450
+Wire Wire Line
+	7100 4450 7100 3350
+Wire Wire Line
+	7100 3350 7550 3350
 $EndSCHEMATC

Commit message: ready for review? maybe. (not really)
Parts:
- removed J201: AC_ADPTR, symbol Connector_Generic:Conn_01x02
- removed J202: WPT_CONN, symbol Connector_Generic:Conn_01x02
- removed J203: SYS_PWR, symbol Connector_Generic:Conn_01x02
- removed J204: ESC_PWR, symbol Connector_Generic:Conn_01x02
- added C3, C4, C5, C6: 10nF, Capacitor_SMD:C_0603_1608Metric, symbol Device:C_Small
- added H1: Top_Left, MountingHole:MountingHole_2.5mm_Pad_Via, symbol Mechanical:MountingHole_Pad
- added H2: Bot_Left, MountingHole:MountingHole_2.5mm_Pad_Via, symbol Mechanical:MountingHole_Pad
- added H3: Top_Right, MountingHole:MountingHole_2.5mm_Pad_Via, symbol Mechanical:MountingHole_Pad
- added H4: Bot_Right, MountingHole:MountingHole_2.5mm_Pad_Via, symbol Mechanical:MountingHole_Pad
- added J1, J2, J3: Conn_01x02, Connector_Molex:Molex_Micro-Fit_3.0_43650-0200_1x02_P3.00mm_Horizontal, symbol Connector_Generic:Conn_01x02
- added J7: ESC_PWR, CHUM_BUCKET_FOOTPRINTS:Keystone_7771, symbol Connector:Conn_01x01_Female
- added J8: ESC_GND, CHUM_BUCKET_FOOTPRINTS:Keystone_7771, symbol Connector:Conn_01x01_Female
- C1: renamed from C201; footprint (none) -> Capacitor_SMD:C_0603_1608Metric
- renumbered C202 to C2, D201 to D1
Connections:
- net CHARGER/AC_FUSED_IN: now also J1.2 (Pin_2), J2.2 (Pin_2)
- net GND: now also C3.2, C4.2, C5.2, C6.2, J1.1 (Pin_1), J2.1 (Pin_1), J3.2 (Pin_2), J8.1 (Pin_1)
- net SYS_MGMT/ESC_PWR_OUT: now also J7.1 (Pin_1)
- net SYS_MGMT/SYS_PWR_OUT_PROT: now also J3.1 (Pin_1)
- new net: C3.1, H1.1
- new net: C4.1, H2.1
- new net: C5.1, H3.1
- new net: C6.1, H4.1
