File: Frank/chum-bucket/PCB/chum-bucket.sch (KiCad schematic (older format))
At the start: 16 parts, among them J1 Conn_01x02, J2 Conn_01x02, J3 Conn_01x02, J7 ESC_PWR, J8 ESC_GND

Commit message: some layout
Parts:
- H1, H2, H4: footprint MountingHole:MountingHole_2.5mm_Pad_Via -> MountingHole:MountingHole_3.2mm_M3_Pad_Via
- H3: footprint MountingHole:MountingHole_2.5mm_Pad_Via -> MountingHole:MountingHole_3.2mm_M3
Changed lines of the file:
@@
 F 0 "H4" H 10100 5299 50  0000 L CNN
 F 1 "Bot_Right" H 10100 5208 50  0000 L CNN
-F 2 "MountingHole:MountingHole_2.5mm_Pad_Via" H 10000 5250 50  0001 C CNN
+F 2 "MountingHole:MountingHole_3.2mm_M3_Pad_Via" H 10000 5250 50  0001 C CNN
 F 3 "~" H 10000 5250 50  0001 C CNN
 	1    10000 5250
@@
 F 0 "H3" H 9600 5299 50  0000 L CNN
 F 1 "Top_Right" H 9600 5208 50  0000 L CNN
-F 2 "MountingHole:MountingHole_2.5mm_Pad_Via" H 9500 5250 50  0001 C CNN
+F 2 "MountingHole:MountingHole_3.2mm_M3" H 9500 5250 50  0001 C CNN
 F 3 "~" H 9500 5250 50  0001 C CNN
 	1    9500 5250
@@
 F 0 "H2" H 9100 5299 50  0000 L CNN
 F 1 "Bot_Left" H 9100 5208 50  0000 L CNN
-F 2 "MountingHole:MountingHole_2.5mm_Pad_Via" H 9000 5250 50  0001 C CNN
+F 2 "MountingHole:MountingHole_3.2mm_M3_Pad_Via" H 9000 5250 50  0001 C CNN
 F 3 "~" H 9000 5250 50  0001 C CNN
 	1    9000 5250
@@
 F 0 "H1" H 8600 5299 50  0000 L CNN
 F 1 "Top_Left" H 8600 5208 50  0000 L CNN
-F 2 "MountingHole:MountingHole_2.5mm_Pad_Via" H 8500 5250 50  0001 C CNN
+F 2 "MountingHole:MountingHole_3.2mm_M3_Pad_Via" H 8500 5250 50  0001 C CNN
 F 3 "~" H 8500 5250 50  0001 C CNN
 	1    8500 5250

Commit message: First Official Schematic Release
yeet
Parts:
- C1: Voltage (none) -> 50V
- J1: value Conn_01x02 -> UMBILLICAL_PWR
- J2: value Conn_01x02 -> WIRELESS_PWR
- J3: value Conn_01x02 -> LV_PWR
