File: Frank/chum-bucket/PCB/chum-bucket.kicad_pcb (KiCad board)
At the start: 4 copper layers, 105.4 x 50.8 mm, 275 parts, among them J1 Conn_01x02, J2 Conn_01x02, J205 CAN_CONN, J206 SWD_DIAGS, J3 Conn_01x02, J7 ESC_PWR, J8 ESC_GND, Q101 2N7002K, Q102 BSS84, Q301 AON2406, Q302 AON2406, Q303 AON2406, Q401 BSS84, Q402 2N7002K, Q403 Q_NMOS_DGS, SW201 B3U-1000P, SW202 LV_EN, SW203 B3U-1000P, U1 INA194, U100 BTS6142DAUMA1, U101 BQ2461x, U102 INA196, U103 CSD87331, U2 SN65HVD232, U215 STM32F042K6Tx, U216 TPS70933DRVT, U301 BQ79606, U401 SN74LVC1G08DRYR, U402 MCP6241-E, U403 NCP81080, U404 MP5000ADQ, Y201 XTAL

Commit message: some layout
Parts:
- added BT1: 18650, CHUM_BUCKET_FOOTPRINTS:Keystone_1042p_18650_Holder, F.Cu at (90.0, 120.0)
- added BT10: 18650, CHUM_BUCKET_FOOTPRINTS:Keystone_1042p_18650_Holder, F.Cu at (198.2, 118.0)
- added BT11: 18650, CHUM_BUCKET_FOOTPRINTS:Keystone_1042p_18650_Holder, F.Cu at (154.9, 118.0)
- added BT12: 18650, CHUM_BUCKET_FOOTPRINTS:Keystone_1042p_18650_Holder, F.Cu at (90.0, 118.0)
- added BT13: 18650, CHUM_BUCKET_FOOTPRINTS:Keystone_1042p_18650_Holder, B.Cu at (176.6, 120.0)
- added BT14: 18650, CHUM_BUCKET_FOOTPRINTS:Keystone_1042p_18650_Holder, B.Cu at (133.3, 120.0)
- added BT15: 18650, CHUM_BUCKET_FOOTPRINTS:Keystone_1042p_18650_Holder, B.Cu at (90.0, 120.0)
- added BT16: 18650, CHUM_BUCKET_FOOTPRINTS:Keystone_1042p_18650_Holder, B.Cu at (198.2, 120.0)
- added BT17: 18650, CHUM_BUCKET_FOOTPRINTS:Keystone_1042p_18650_Holder, B.Cu at (154.9, 120.0)
- added BT18: 18650, CHUM_BUCKET_FOOTPRINTS:Keystone_1042p_18650_Holder, B.Cu at (111.7, 120.0)
- added BT19: 18650, CHUM_BUCKET_FOOTPRINTS:Keystone_1042p_18650_Holder, B.Cu at (176.6, 118.0)
- added BT2: 18650, CHUM_BUCKET_FOOTPRINTS:Keystone_1042p_18650_Holder, F.Cu at (176.6, 120.0)
- added BT20: 18650, CHUM_BUCKET_FOOTPRINTS:Keystone_1042p_18650_Holder, B.Cu at (133.3, 118.0)
- added BT21: 18650, CHUM_BUCKET_FOOTPRINTS:Keystone_1042p_18650_Holder, B.Cu at (90.0, 118.0)
- added BT22: 18650, CHUM_BUCKET_FOOTPRINTS:Keystone_1042p_18650_Holder, B.Cu at (198.2, 118.0)
- added BT23: 18650, CHUM_BUCKET_FOOTPRINTS:Keystone_1042p_18650_Holder, B.Cu at (154.9, 118.0)
- added BT24: 18650, CHUM_BUCKET_FOOTPRINTS:Keystone_1042p_18650_Holder, B.Cu at (111.7, 118.0)
- added BT3: 18650, CHUM_BUCKET_FOOTPRINTS:Keystone_1042p_18650_Holder, F.Cu at (133.3, 120.0)
- added BT4: 18650, CHUM_BUCKET_FOOTPRINTS:Keystone_1042p_18650_Holder, F.Cu at (198.2, 120.0)
- added BT5: 18650, CHUM_BUCKET_FOOTPRINTS:Keystone_1042p_18650_Holder, F.Cu at (154.9, 120.0)
- added BT6: 18650, CHUM_BUCKET_FOOTPRINTS:Keystone_1042p_18650_Holder, F.Cu at (111.7, 120.0)
- added BT7: 18650, CHUM_BUCKET_FOOTPRINTS:Keystone_1042p_18650_Holder, F.Cu at (176.6, 118.0)
- added BT8: 18650, CHUM_BUCKET_FOOTPRINTS:Keystone_1042p_18650_Holder, F.Cu at (133.3, 118.0)
- added BT9: 18650, CHUM_BUCKET_FOOTPRINTS:Keystone_1042p_18650_Holder, F.Cu at (111.7, 118.0)
- added TP7: TP_BQ2417_CHG_EN, TestPoint:TestPoint_Pad_D1.0mm, F.Cu at (134.9, 314.5)
- H1, H2, H3, H4: footprint MountingHole:MountingHole_2.5mm_Pad_Via -> MountingHole:MountingHole_3.2mm_M3_Pad_Via
- moved R116 260.8 mm to (96.6, 290.0)
- moved F301 260.5 mm to (155.5, 289.5)
- moved R270 257.9 mm to (121.9, 322.6)
- moved C255 257.1 mm to (119.3, 316.7)
- moved R261 256.6 mm to (105.8, 320.6)
- moved R6 255.0 mm to (117.8, 322.2)
- moved R259 255.0 mm to (115.3, 314.7)
- moved R414 253.9 mm to (161.2, 316.2)
- moved D5 253.9 mm to (107.1, 318.0)
- moved C112 253.4 mm to (98.0, 284.9)
- moved R101 253.0 mm to (117.5, 282.3)
- moved R106 253.0 mm to (123.3, 292.3)
- moved C314 252.9 mm to (156.2, 284.5)
- moved R317 252.9 mm to (156.2, 287.0)
- moved C224 252.5 mm to (115.3, 317.2)
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Connections:
- U215 pad 10: Net-(U215-Pad10) -> /MCU/ANALOG_V_ESCS
- U215 pad 11: Net-(U215-Pad11) -> /MCU/ANALOG_V_SYSTEM
- U215 pad 12: Net-(U215-Pad12) -> /MCU/ESC_PWR_EN
- U215 pad 13: Net-(U215-Pad13) -> /CHARGER/BQ24617_CHG_EN
- U215 pad 14: Net-(U215-Pad14) -> /BATT_MGMT/~BQ79606_FAULT
- U215 pad 15: Net-(U215-Pad15) -> /BATT_MGMT/BQ79606_WAKE
- U215 pad 25: Net-(U215-Pad25) -> /MCU/UART_DIAGS_STM_RX
- U215 pad 29: Net-(U215-Pad29) -> /MCU/USR_BUTTON
- U215 pad 30: Net-(U215-Pad30) -> /MCU/SM1_LED
- U215 pad 31: Net-(U215-Pad31) -> /MCU/SM0_LED
- U215 pad 6: Net-(U215-Pad6) -> /CHARGER/ANALOG_I_SYS
- U215 pad 7: Net-(U215-Pad7) -> /CHARGER/ANALOG_I_CHG
- U215 pad 9: /MCU/UART_DIAGS_STM_RX -> /MCU/ANALOG_I_ESCS
Routing:
- net +BATT: track 0.00 -> 3.49 mm
Other:
- board size 105.4 x 50.8 mm -> 131.7 x 219 mm

Commit message: push
Parts:
- moved C103 48.7 mm to (150.6, 316.6)
- moved C107 48.7 mm to (145.8, 320.4)
- moved C113 48.7 mm to (161.5, 308.6)
- moved C114 48.7 mm to (144.1, 325.6)
- moved C13 48.7 mm to (191.7, 356.6)
- moved C245 48.7 mm to (139.7, 346.9)
- moved C248 48.7 mm to (145.9, 355.1)
- moved C251 48.7 mm to (161.5, 338.9)
- moved C255 48.7 mm to (145.9, 357.6)
- moved C256 48.7 mm to (161.5, 341.5)
- moved C314 48.7 mm to (182.8, 325.4)
- moved C323 48.7 mm to (201.7, 313.6)
- moved C405 48.7 mm to (204.8, 338.9)
- moved C413 48.7 mm to (203.8, 351.5)
- moved D103 48.7 mm to (150.5, 319.4)
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Other:
- board size 131.7 x 219 mm -> 130.7 x 220 mm

Commit message: First Official Schematic Release
yeet
Parts:
- moved C103 46.4 mm to (133.1, 273.7)
- moved C104 46.4 mm to (138.6, 281.4)
- moved C107 46.4 mm to (128.2, 277.4)
- moved C113 46.4 mm to (144.0, 265.6)
- moved C114 46.4 mm to (126.6, 282.7)
- moved C115 46.4 mm to (125.1, 286.3)
- moved C17 46.4 mm to (134.8, 302.9)
- moved C245 46.4 mm to (122.2, 303.9)
- moved C248 46.4 mm to (128.4, 312.1)
- moved C301 46.4 mm to (184.9, 265.6)
- moved C302 46.4 mm to (180.8, 265.6)
- moved C305 46.4 mm to (169.3, 284.9)
- moved C310 46.4 mm to (165.4, 277.2)
- moved C311 46.4 mm to (169.3, 282.4)
- moved C314 46.4 mm to (165.2, 282.4)
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