File: Frank/chum-bucket/PCB/chum-bucket.kicad_pcb (KiCad board)
At the start: 4 copper layers, 130.7 x 220 mm, 293 parts, among them Q101 2N7002K, Q102 BSS84, Q103 SIS413DN, Q201 BSS84, Q301 AON2406, Q302 AON2406, Q303 AON2406, Q401 SIR140DP, SW202 LV_EN, U100 BTS6142DAUMA1, U101 BQ2461x, U102 INA196, U103 CSD87331, U2 SN65HVD232, U215 STM32F042K6Tx, U216 TPS70933DRVT, U301 BQ79606, U401 MIC5014, U402 INA194, Y201 XTAL

Commit message: lowered kicad version. Also tided up routing DRC cleared.
Parts:
- removed the G*** at (91.4, 221.0)
- removed the G*** at (168.7, 238.3)
- removed the G*** at (179.3, 236.0)
- removed the G*** at (87.6, 228.1)
- removed the G*** at (86.4, 223.5)
- removed the G*** at (91.4, 224.8)
- removed the G*** at (124.2, 238.5)
- removed the G*** at (111.8, 246.4)
Routing:
- net GND: track 263.2 -> 266.9 mm, vias 437 -> 436
- net +3V3: track 84.5 -> 81.7 mm
- net +BATT: track 50.8 -> 53.1 mm, vias 313 -> 312
- net /BATT_MGMT/SERIES_BANK_1: track 14.0 -> 15.9 mm
- net /CHARGER/ANALOG_I_SYS: track 133.5 -> 134.5 mm
- net /CHARGER/SYS_PWR_OUT: vias 25 -> 24
- added copper zone on Signal.1, net +3V3
- added copper zone on Signal.1, net +BATT
- added copper zone on Signal.2, net +BATT
- added copper zone on Signal.1, net /BATT_MGMT/SERIES_BANK_1
- added copper zone on Signal.2, net /BATT_MGMT/SERIES_BANK_1
- added copper zone on Signal.1, net /BATT_MGMT/SERIES_BANK_2
- added copper zone on Signal.2, net /BATT_MGMT/SERIES_BANK_2
- added copper zone on Signal.1, net /CHARGER/SYS_PWR_OUT
- added copper zone on Signal.1, net /SYS_MGMT/ESC_PWR_OUT
- added copper zone on Signal.2, net /SYS_MGMT/ESC_PWR_OUT
- added copper zone on Signal.1, net GND
- added copper zone on Signal.2, net GND
- added copper zone on Signal.1, net Net-(C224-Pad2)
- added copper zone on Signal.1, net Net-(D105-Pad1)
- removed copper zone on In1.Cu, net +3V3
- removed copper zone on In1.Cu, net +BATT
- removed copper zone on In2.Cu, net +BATT
- removed copper zone on In1.Cu, net /BATT_MGMT/SERIES_BANK_1
- removed copper zone on In2.Cu, net /BATT_MGMT/SERIES_BANK_1
- removed copper zone on In1.Cu, net /BATT_MGMT/SERIES_BANK_2
- removed copper zone on In2.Cu, net /BATT_MGMT/SERIES_BANK_2
- removed copper zone on In1.Cu, net /CHARGER/SYS_PWR_OUT
- removed copper zone on In1.Cu, net /SYS_MGMT/ESC_PWR_OUT
- removed copper zone on In2.Cu, net /SYS_MGMT/ESC_PWR_OUT
- removed copper zone on In1.Cu, net GND
- removed copper zone on In2.Cu, net GND
- removed copper zone on In1.Cu, net Net-(C224-Pad2)
- removed copper zone on In1.Cu, net Net-(D105-Pad1)
Other:
- net class Default added: clearance 0.2, trace_width 0.25, via_dia 0.8, via_drill 0.4

Commit message: routing V2
Parts:
- removed ESC_OUT: ESC_PWR, CHUM_BUCKET_FOOTPRINTS:Keystone_7771
- added ESC_POS: ESC_PWR, CHUM_BUCKET_FOOTPRINTS:Keystone_7771, F.Cu at (201.9, 211.1)
- <- 3V3 DISABLE: renamed from SW202
- C245, R112, R114: moved to B.Cu
- C249, FB201, U216: moved to F.Cu
- SWD HEADER: renamed from DEBUG
- U301: footprint Package_QFP:LQFP-48-1EP_7x7mm_P0.5mm_EP3.6x3.6mm_ThermalVias -> CHUM_BUCKET_FOOTPRINTS:LQFP-48-1EP_7x7mm_P0.5mm_EP4x4mm_Thermalvias
- moved R104 26.8 mm to (160.0, 205.8), turned to 180 degrees
- moved C401 24.6 mm to (162.9, 207.3), turned to 180 degrees
- moved VFB 24.2 mm to (160.3, 207.6), turned to 270 degrees
- moved R103 23.2 mm to (163.0, 205.8), turned to 180 degrees
- moved C102 22.0 mm to (163.0, 204.2), turned to 180 degrees
- moved I_CHG 21.7 mm to (142.8, 249.8)
- moved I_ESC 21.7 mm to (139.6, 249.8)
- moved I_SYS 21.7 mm to (136.4, 249.8)
- moved R10 20.5 mm to (128.1, 242.5), turned to 180 degrees
- moved R265 19.0 mm to (128.1, 240.9), turned to 180 degrees
- moved R11 17.6 mm to (128.1, 239.3), turned to 180 degrees
- moved R12 16.5 mm to (128.1, 237.7), turned to 180 degrees
- moved R266 15.3 mm to (126.6, 233.8), turned to 180 degrees
- moved C246 13.1 mm to (117.5, 220.0), turned to 180 degrees
- moved FB201 12.7 mm to (156.2, 215.9)
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- renumbered TP202 to BMS_UART_RX, TP201 to BMS_UART_TX, D3 to CAN_RX, D4 to CAN_TX, CHG_INPUT to CHARGER_IN, ~BMS_FAULT to CHG_PG, ESC_GND to ESC_NEG, I_ESCs to I_ESC, SYS_OUTPUT to LOW_CURRNET_OUT, SW to TP2, CHG_FB to VFB, BMS_WAKE to ~BMS_FAULT, RESET to ~RESET
Connections:
- C15 pad 1: /MCU/ANALOG_V_SYSTEM -> /MCU/ANALOG_V_SYSTEM_JMP
- C16 pad 1: /MCU/ANALOG_V_ESCS -> /MCU/ANALOG_V_ESCS_JMP
- C17 pad 1: /MCU/ANALOG_I_ESCS -> /MCU/ANALOG_I_ESCS_JMP
- C252 pad 1: /MCU/ESC_PWR_EN -> /MCU/ESC_PWR_EN_JMP
- C253 pad 1: /CHARGER/BQ24617_CHG_EN -> /MCU/BQ_24617_CHG_EN_JMP
- C254 pad 1: /CHARGER/ANALOG_I_SYS -> /MCU/ANALOG_I_SYS_JMP
- C255 pad 2: /BATT_MGMT/BQ79606_WAKE -> /MCU/BQ79606_WAKE_JMP
- C256 pad 2: /BATT_MGMT/~BQ79606_FAULT -> /MCU/~BQ79606_FAULT_JMP
- C257 pad 1: /CHARGER/ANALOG_I_CHG -> /MCU/ANALOG_I_CHG_JMP
- CHG_PG pad 1: /BATT_MGMT/~BQ79606_FAULT -> /CHARGER/BQ24617_PG
- D212 pad 1: /CHARGER/ANALOG_I_SYS -> /MCU/ANALOG_I_SYS_JMP
- D213 pad 1: /CHARGER/ANALOG_I_CHG -> /MCU/ANALOG_I_CHG_JMP
- D7 pad 1: /MCU/ANALOG_V_SYSTEM -> /MCU/ANALOG_V_SYSTEM_JMP
- D8 pad 1: /MCU/ANALOG_V_ESCS -> /MCU/ANALOG_V_ESCS_JMP
- D9 pad 1: /MCU/ANALOG_I_ESCS -> /MCU/ANALOG_I_ESCS_JMP
- R1 pad 2: /CHARGER/BQ24617_PG -> /MCU/BQ24617_PG_JMP
- R10 pad 2: /MCU/ANALOG_V_SYSTEM -> /MCU/ANALOG_V_SYSTEM_JMP
- R11 pad 2: /MCU/ANALOG_V_ESCS -> /MCU/ANALOG_V_ESCS_JMP
- R12 pad 2: /MCU/ANALOG_I_ESCS -> /MCU/ANALOG_I_ESCS_JMP
- R257 pad 1: /MCU/ESC_PWR_EN -> /MCU/ESC_PWR_EN_JMP
- R259 pad 1: /CHARGER/BQ24617_CHG_EN -> /MCU/BQ_24617_CHG_EN_JMP
- R262 pad 2: /BATT_MGMT/BQ79606_WAKE -> /MCU/BQ79606_WAKE_JMP
- R263 pad 2: /BATT_MGMT/~BQ79606_FAULT -> /MCU/~BQ79606_FAULT_JMP
- R264 pad 2: /CHARGER/BQ24617_CHG_EN -> /MCU/BQ_24617_CHG_EN_JMP
- R265 pad 2: /CHARGER/ANALOG_I_SYS -> /MCU/ANALOG_I_SYS_JMP
- R266 pad 2: /CHARGER/ANALOG_I_CHG -> /MCU/ANALOG_I_CHG_JMP
- R269 pad 2: /BATT_MGMT/BQ79606_WAKE -> /MCU/BQ79606_WAKE_JMP
- R270 pad 2: /BATT_MGMT/~BQ79606_FAULT -> /MCU/~BQ79606_FAULT_JMP
- R271 pad 2: /MCU/ESC_PWR_EN -> /MCU/ESC_PWR_EN_JMP
- U215 pad 10: /MCU/ANALOG_I_ESCS -> /MCU/ANALOG_I_ESCS_JMP
- U215 pad 11: /CHARGER/ANALOG_I_CHG -> /MCU/ANALOG_I_CHG_JMP
- U215 pad 12: /MCU/ESC_PWR_EN -> /MCU/ESC_PWR_EN_JMP
- U215 pad 13: /CHARGER/BQ24617_CHG_EN -> /MCU/BQ_24617_CHG_EN_JMP
- U215 pad 14: /BATT_MGMT/~BQ79606_FAULT -> /MCU/~BQ79606_FAULT_JMP
- U215 pad 15: /BATT_MGMT/BQ79606_WAKE -> /MCU/BQ79606_WAKE_JMP
- U215 pad 28: /CHARGER/BQ24617_PG -> /MCU/BQ24617_PG_JMP
- U215 pad 6: /MCU/ANALOG_V_SYSTEM -> /MCU/ANALOG_V_SYSTEM_JMP
- U215 pad 7: /CHARGER/ANALOG_I_SYS -> /MCU/ANALOG_I_SYS_JMP
- U215 pad 9: /MCU/ANALOG_V_ESCS -> /MCU/ANALOG_V_ESCS_JMP
- ~BMS_FAULT pad 1: /BATT_MGMT/BQ79606_WAKE -> /BATT_MGMT/~BQ79606_FAULT
Routing:
- net +3V3: track 81.7 -> 371.2 mm, vias 25 -> 26
- net /BATT_MGMT/TSREF: track 770.0 -> 544.8 mm, vias 18 -> 14
- net /MCU/ANALOG_V_SYSTEM_JMP: track 0.00 -> 37.7 mm
- net /BATT_MGMT/THERM5: track 257.7 -> 221.4 mm
- net /CHARGER/BQ24617_CHG_EN: track 80.6 -> 44.5 mm, vias 5 -> 3
- net /BATT_MGMT/THERM2: track 269.8 -> 237.6 mm
- net /MCU/ANALOG_V_ESCS_JMP: track 0.00 -> 31.6 mm
- net /MCU/ANALOG_V_SYSTEM: track 138.0 -> 106.4 mm
- net /CHARGER/ANALOG_I_SYS: track 134.5 -> 103.0 mm
- net /MCU/ANALOG_I_SYS_JMP: track 0.00 -> 29.8 mm
- net /CHARGER/ANALOG_I_CHG: track 113.2 -> 84.9 mm, vias 4 -> 2
- net /MCU/ANALOG_I_ESCS_JMP: track 0.00 -> 26.2 mm
- net /CHARGER/BQ_24617_VFB: track 52.7 -> 27.0 mm, vias 3 -> 2
- net /MCU/ANALOG_V_ESCS: track 128.9 -> 104.9 mm
- net GND: track 266.9 -> 287.4 mm, vias 436 -> 649
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- added copper zone on F.Cu, net +3V3
- removed copper zone on B.Cu, net +3V3
- removed copper zone on Signal.1, net +3V3
- removed copper zone on B.Cu, net Net-(C224-Pad2)
- removed copper zone on B.Cu, net Net-(C249-Pad2)
- removed copper zone on F.Cu, net Net-(D106-Pad2)
- removed copper zone on F.Cu, net Net-(D208-Pad2)
Other:
- board text added: "NEG"
- board text added: "POS"
- board text added: "SYS & CHG: x20 ESC: x50"

Commit message: routing v2.1.
Parts:
- removed C17, C411: 0.1uF, Capacitor_SMD:C_0603_1608Metric
- removed C402, C403: 10nF, Capacitor_SMD:C_0603_1608Metric
- removed D9: BZT52, Diode_SMD:D_SOD-123
- removed I_ESC: TP_I_ESCS, TestPoint:TestPoint_Pad_D1.0mm
- removed R12: 100, Resistor_SMD:R_0603_1608Metric
- removed R412, R414: 0, Resistor_SMD:R_0603_1608Metric
- removed R413: 500u, Resistor_SMD:R_2512_6332Metric
- removed U402: INA194, Package_TO_SOT_SMD:SOT-23-5
- added STM_PA4: TestPoint, TestPoint:TestPoint_Pad_D1.0mm, F.Cu at (117.7, 233.9)
- H3: footprint MountingHole:MountingHole_3.2mm_M3 -> MountingHole:MountingHole_3.2mm_M3_Pad_Via
- SWD_HEADER: renamed from SWD HEADER
- moved I_CHG 3.96 mm to (138.8, 249.8)
- moved R258 0.54 mm to (86.2, 239.4)
- moved C201 0.51 mm to (88.6, 242.9)
- moved C251 0.51 mm to (95.3, 239.5)
- moved D6 0.51 mm to (88.9, 235.7)
- moved U2 0.51 mm to (90.9, 239.4)
- moved CAN_CONN 0.48 mm to (82.0, 239.0)
- moved H3 0.40 mm to (205.7, 35.1)
- renumbered CHARGER_IN to CHG_PWR_IN, TP2 to SW, LOW_CURRNET_OUT to SYSTEM_POWER_OUT, ~BMS_FAULT to TP203, CHG_PG to TP204, CHG_EN to TP209
Connections:
- Q401 pad 1: /SYS_MGMT/ESC_OUTPUT_UNMEAS -> /SYS_MGMT/ESC_PWR_OUT
- R401 pad 2: /SYS_MGMT/ESC_OUTPUT_UNMEAS -> /SYS_MGMT/ESC_PWR_OUT
- U215 pad 10: /MCU/ANALOG_I_ESCS_JMP -> /MCU/STM_PA4
Routing:
- net /MCU/ANALOG_I_ESCS: track 105.4 -> 0.00 mm, vias 3 -> 0
- net Net-(C306-Pad1): track 22.7 -> 49.1 mm
- net /MCU/ANALOG_I_ESCS_JMP: track 26.2 -> 0.00 mm
- net /SYS_MGMT/ESC_PWR_OUT: track 6.06 -> 18.6 mm, vias 13 -> 15
- net +3V3: track 371.2 -> 358.9 mm, vias 26 -> 24
- net /MCU/STM_PA4: track 0.00 -> 11.3 mm
- net /SYS_MGMT/ESC_OUTPUT_UNMEAS: track 10.4 -> 0.00 mm, vias 1 -> 0
- net /CHARGER/ANALOG_I_SYS: track 103.0 -> 109.6 mm
- net /BATT_MGMT/TSREF: track 544.8 -> 540.2 mm
- net GND: track 287.4 -> 283.0 mm, vias 649 -> 675
- net /MCU/ANALOG_V_SYSTEM: track 106.4 -> 109.5 mm
- net /MCU/USR_BUTTON: track 30.2 -> 33.0 mm
- net /MCU/ANALOG_V_ESCS: track 104.9 -> 107.0 mm
- net Net-(R414-Pad1): track 1.60 -> 0.00 mm
- net Net-(R412-Pad1): track 1.59 -> 0.00 mm
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- removed copper zone on B.Cu, net /SYS_MGMT/ESC_OUTPUT_UNMEAS
Other:
- rule pad_to_mask_clearance: 0.051 -> 0
- board text removed: "SYS & CHG: x20 ESC: x50"
