File: Frank/chum-bucket/PCB/SYS_MGMT.sch (KiCad schematic (older format))
At the start: 43 parts

Commit message: batt-management sheet updates
Other:
- note added: "To do: add flip flop with reset line"
Changed lines of the file:
@@
 Text Notes 8200 4050 0    39   ~ 0
 2mOhm resistor sets for 3.2V at 80A\nP_loss = (2/1000)*80*80 = 12.8W (not good)
+Text Notes 2800 4950 0    39   Italic 0
+To do: add flip flop with reset line
 $EndSCHEMATC

Commit message: more work
Parts:
- gave numbers to parts that had none: 39
- renumbered C_BST1 to C_BST401, C_LIM to C_LIM401
Other:
- note added: "Layout Note: No solder mask on ESC power plane + GND. \nMFG Note: Place tonnes of excess solder on ESC power plane + GND"

Commit message: more changes :)
Parts:
- removed U405: INA196, Package_TO_SOT_SMD:SOT-23-5, symbol Amplifier_Current:INA196
- added R? (x4): R, symbol Device:R
- added U?: INA194, Package_TO_SOT_SMD:SOT-23-5, symbol Amplifier_Current:INA194
- C403, C406: value 100nF -> 10nF; footprint (none) -> Capacitor_SMD:C_0603_1608Metric; Digikey (none) -> 399-7842-2-ND; Voltage (none) -> 25V
- C413: footprint (none) -> Capacitor_SMD:C_0603_1608Metric; Digikey (none) -> 399-7842-2-ND; Voltage (none) -> 25V
- R401: footprint (none) -> Resistor_SMD:R_0603_1608Metric
- R403: footprint (none) -> Resistor_SMD:R_0603_1608Metric; Digikey (none) -> RHM4.7DTR-ND
- R406, R407: value 10k -> 1k; footprint (none) -> Resistor_SMD:R_0603_1608Metric
- R413: value 2m -> 500u; footprint (none) -> Resistor_SMD:R_2512_6332Metric; Power (none) -> 5W
Connections:
- net labels added: ANALOG_I_ESCS, ANALOG_V_ESCS, ANALOG_V_SYSTEM
- wire segments 154 -> 169
Other:
- note added: "- Instrumentation amplifier w/ gain of 50V/V\n- Outputs 2.5V at 100A"
- note added: "500uOhm resistor gives 50mV drop at 100A \nI^R losses are 5W\n"
- note removed: "2mOhm resistor sets for 3.2V at 80A\nP_loss = (2/1000)*80*80 = 12.8W (not good)"
- moved on the sheet: C401, C402, C404, C405, C407, C408, C409, C410, C411, C412, C414, C_BST401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

Commit message: changes
Parts:
- removed C410: C_Small, symbol Device:C_Small
- removed C412: 100nF, symbol Device:C_Small
- removed C414: 10nF, symbol Device:C_Small
- removed D401: D_Zener, symbol Device:D_Zener
- added C? (x5): 10nF, Capacitor_SMD:C_0603_1608Metric, symbol Device:C_Small
- added C? (x2): 1uF, Capacitor_SMD:C_0603_1608Metric, symbol Device:C_Small
- added D?: BZT52, Diode_SMD:D_SOD-123, symbol Device:D_Zener_Small
- C408: value ??xF -> 10pF; footprint (none) -> Capacitor_SMD:C_0603_1608Metric
- R408: footprint (none) -> Resistor_SMD:R_0603_1608Metric
- R410: value R -> 30; footprint (none) -> Resistor_SMD:R_0603_1608Metric; Tolerance (none) -> 1%
- R?: value R -> 10k; footprint (none) -> Resistor_SMD:R_0603_1608Metric
- R?: value R -> 1.5k; footprint (none) -> Resistor_SMD:R_0603_1608Metric
Connections:
- wire segments 169 -> 182
- no-connect marks 19 -> 4
Other:
- note added: "30ohm resistor give hold current of 2.56A\nand trip current of 3.71A"
- note added: "DNP DV/DT cap\n0.9ms turn on time\nif left floating\n"
- note removed: "To do: add flip flop with reset line"
- moved on the sheet: C401, C402, C404, C405, C407, C411, C413, D402, D403, R402, R404, R405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

Commit message: ready for review? maybe. (not really)
Parts:
- removed C404: 0.1uF, symbol Device:C_Small
- removed R405: R_Small, symbol Device:R_Small
- added C7: 0.47uF, Capacitor_SMD:C_0603_1608Metric, symbol Device:C_Small
- added R1: 47, Resistor_SMD:R_0603_1608Metric, symbol Device:R
- C401, C402, C407, C411, C_LIM401: footprint (none) -> Capacitor_SMD:C_0603_1608Metric
- C405: value 0.1uF -> 1uF; footprint (none) -> Capacitor_SMD:C_0603_1608Metric
- C409, C_BST401: footprint (none) -> Capacitor_SMD:C_0805_2012Metric
- Q403: footprint (none) -> CHUM_BUCKET_FOOTPRINTS:CSD1757Q5B
- R4: renamed from R?; value R -> 10k; footprint (none) -> Resistor_SMD:R_0603_1608Metric
- R402: value R_Small -> 266k; footprint (none) -> Resistor_SMD:R_0603_1608Metric
- R404: value 1k -> 100k; footprint (none) -> Resistor_SMD:R_0603_1608Metric
- R409, R411, R412, R414: footprint (none) -> Resistor_SMD:R_0603_1608Metric
- R5: renamed from R?; value R -> 3.6k; footprint (none) -> Resistor_SMD:R_0603_1608Metric
- U401: footprint (none) -> CHUM_BUCKET_FOOTPRINTS:6SON-TI
- U401: footprint (none) -> CHUM_BUCKET_FOOTPRINTS:6SON-TI; Digikey (none) -> 296-21815-2-ND
- U402: footprint (none) -> Package_DFN_QFN:DFN-8-1EP_3x2mm_P0.5mm_EP1.3x1.5mm; Digikey (none) -> MCP6241-E/MC-ND
- U402: footprint (none) -> Package_DFN_QFN:DFN-8-1EP_3x2mm_P0.5mm_EP1.3x1.5mm
- gave numbers to parts that had none: 11
Connections:
- net ANALOG_I_ESCS: now also R1.1
- net GND: now also C7.2
- net at U402.2 (-): now also C7.1, R1.2
- no-connect marks 4 -> 5
Other:
- note removed: "- CLIM allows slew rate control of the ESC bus\n- Increased capacitance increases bus slew rate\n- DNP for first build\n"
- note removed: "Layout Note: No solder mask on ESC power plane + GND. \nMFG Note: Place tonnes of excess solder on ESC power plane + GND"

Commit message: First Official Schematic Release
yeet
Parts:
- removed C401, C402, C407: 0.1uF, Capacitor_SMD:C_0603_1608Metric, symbol Device:C_Small
- removed C405: 1uF, Capacitor_SMD:C_0603_1608Metric, symbol Device:C_Small
- removed C409: 4.7uF, Capacitor_SMD:C_0805_2012Metric, symbol Device:C_Small
- removed C7: 0.47uF, Capacitor_SMD:C_0603_1608Metric, symbol Device:C_Small
- removed C_BST401: 0.1uF, Capacitor_SMD:C_0805_2012Metric, symbol Device:C_Small
- removed D2: BZT52, Diode_SMD:D_SOD-123, symbol Device:D_Zener_Small
- removed R1: 47, Resistor_SMD:R_0603_1608Metric, symbol Device:R
- removed R402: 266k, Resistor_SMD:R_0603_1608Metric, symbol Device:R_Small
- removed R404: 100k, Resistor_SMD:R_0603_1608Metric, symbol Device:R_Small
- removed R406: 1k, Resistor_SMD:R_0603_1608Metric, symbol Device:R_Small
- removed R408: 0, Resistor_SMD:R_0603_1608Metric, symbol Device:R_Small
- removed R409: 3, Resistor_SMD:R_0603_1608Metric, symbol Device:R_Small
- removed R411: 0, Resistor_SMD:R_0603_1608Metric, symbol Device:R
- removed U401: SN74LVC1G08DRYR, CHUM_BUCKET_FOOTPRINTS:6SON-TI, symbol chum-bucket:SN74LVC1G08DRYR
- removed U402: MCP6241-E, Package_DFN_QFN:DFN-8-1EP_3x2mm_P0.5mm_EP1.3x1.5mm, symbol chum-bucket:MCP6241-E
- removed U403: NCP81080, Package_DFN_QFN:DFN-8_2x2mm_P0.5mm, symbol chum-bucket:NCP81080
- added C? (x2): 1uF, Capacitor_SMD:C_0603_1608Metric, symbol Device:C_Small
- added R405: 100, Resistor_SMD:R_0603_1608Metric, symbol Device:R_Small
- added R411, R? (x2): 0, symbol Device:R_Small
- added R499: 0, Resistor_SMD:R_0603_1608Metric, symbol Device:R_Small
- added U?: MIC5014, Package_SO:SOIC-8_3.9x4.9mm_P1.27mm, symbol chum-bucket:MIC5014
- R401: value 1k -> 68k; Power (none) -> 1/10W
- R403: value 4.7k -> 68k; Digikey RHM4.7DTR-ND -> (none); Power (none) -> 1/10W
Connections:
- net +BATT: now also C?.1, U?.1 (V+)
- net AC_FUSED: now also R499.1; no longer Q401.2 (S)
- net ESC_PWR_EN: now also U?.2 (INPUT)
- net GND: now also C?.2, C?.2, U?.4 (GND)
- net SYS_PWR_OUT: now also C?.1
- net ~BQ24617_BAT_DRV: now also R?.2; no longer C403.2, Q401.1 (G), R401.2
- net at C_LIM401.1: now also R411.1, U?.5 (GATE)
- net at C406.2, Q401.3 (D), R403.1: now also R405.2; no longer Q402.1 (G)
- net at Q403.2 (G): now also R411.2
- net at C10.2, C11.1, Q403.3 (S)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: now also R?.2
- new net: Q402.1 (G), R405.1
- new net: C403.2, Q401.1 (G), R401.2, R?.1
- new net: Q401.2 (S), R499.2
- new net: R?.1, U?.3 (SOURCE)
- no-connect marks 5 -> 2
Other:
- note added: "Inverter glue logic for load switch\nR499 gives 'bodge location' in case MP5000-3 pin \ncannot be held high and MUST be floated."
- note removed: "- current sensor, opamp schmitt trigger and AND gate\nused as discrete e-fuse\n- integrating capacitor on opamp determines trip time\n- DNP for initial builds... this is a 'nice to have'"
- note removed: "Inverter glue logic for load switch"
- moved on the sheet: C10, C11, C406, C411, R412, R414, U1

Commit message: first (hopefully final) routing pass
Parts:
- removed C403, C406: 10nF, Capacitor_SMD:C_0603_1608Metric, symbol Device:C_Small
- removed C408: 10pF, Capacitor_SMD:C_0603_1608Metric, symbol Device:C_Small
- removed C8, C9, C?: 1uF, Capacitor_SMD:C_0603_1608Metric, symbol Device:C_Small
- removed Q401: BSS84, Package_TO_SOT_SMD:SOT-23, symbol Transistor_FET:BSS84
- removed Q402: 2N7002K, Package_TO_SOT_SMD:SOT-23, symbol Transistor_FET:2N7002K
- removed Q403: Q_NMOS_DGS, CHUM_BUCKET_FOOTPRINTS:CSD1757Q5B, symbol Device:Q_NMOS_DGS
- removed R401, R403: 68k, Resistor_SMD:R_0603_1608Metric, symbol Device:R_Small
- removed R405: 100, Resistor_SMD:R_0603_1608Metric, symbol Device:R_Small
- removed R407: 1k, Resistor_SMD:R_0603_1608Metric, symbol Device:R_Small
- removed R410: 30, Resistor_SMD:R_0603_1608Metric, symbol Device:R
- removed R499: 0, Resistor_SMD:R_0603_1608Metric, symbol Device:R_Small
- removed R?: 0, symbol Device:R_Small
- removed U404: MP5000ADQ, Package_DFN_QFN:DFN-10-1EP_3x3mm_P0.5mm_EP1.7x2.5mm, symbol chum-bucket:MP5000ADQ
- added Q401: SIR140DP, CHUM_BUCKET_FOOTPRINTS:SIR140DP, symbol Device:Q_NMOS_SGD
- D402: value SMBJ26A -> SMF24A; footprint Diode_SMD:D_SMB -> Diode_SMD:D_SOD-123F; Digikey SMBJ26A-E3/5BGITR-ND -> F5823CT-ND
- D403: value SMBJ17CA -> SMF14A; footprint Diode_SMD:D_SMB -> Diode_SMD:D_SOD-123F; Digikey SMBJ17CA-FDITR-ND -> F5816CT-ND
- R401: renamed from R?; footprint (none) -> Resistor_SMD:R_0603_1608Metric
- R411: footprint (none) -> Resistor_SMD:R_0603_1608Metric
- gave numbers to parts that had none: 2
- renumbered C10 to C402, C11 to C403, C12 to C404, C13 to C405, C14 to C406, R2 to R402, R3 to R403, R4 to R404, R5 to R405, U1 to U402
Connections:
- net +BATT: now also Q401.3 (D)
- net at R411.2: now also Q401.2 (G)
- net ESC_OUTPUT_UNMEAS: now reaches C402.2, C403.1, R401.2, R412.2, R413.2
- net ESC_OUTPUT_UNMEAS: now also Q401.1 (S)
- no-connect marks 2 -> 1
Other:
- note removed: "- Load switch allows battery to power LV systems\n- Controlled by charger IC\n- the enable for this IC is XOR'd with the AC adapter LS"
- note removed: "30ohm resistor give hold current of 2.56A\nand trip current of 3.71A"
- note removed: "DNP DV/DT cap\n0.9ms turn on time\nif left floating\n"
- note removed: "Inverter glue logic for load switch\nR499 gives 'bodge location' in case MP5000-3 pin \ncannot be held high and MUST be floated."

Commit message: routing v2.1.
Parts:
- removed C402, C403: 10nF, Capacitor_SMD:C_0603_1608Metric, symbol Device:C_Small
- removed C411: 0.1uF, Capacitor_SMD:C_0603_1608Metric, symbol Device:C_Small
- removed R412, R414: 0, Resistor_SMD:R_0603_1608Metric, symbol Device:R
- removed R413: 500u, Resistor_SMD:R_2512_6332Metric, symbol Device:R
- removed U402: INA194, Package_TO_SOT_SMD:SOT-23-5, symbol Amplifier_Current:INA194
Connections:
- net ESC_OUTPUT_UNMEAS is gone; now on net ESC_PWR_OUT: Q401.1 (S), R401.2
Other:
- note removed: "- Instrumentation amplifier w/ gain of 50V/V\n- Outputs 2.5V at 100A"
Changed lines of the file:
@@
 	9800 1500 9800 1150
 $Comp
-L Device:R R413
-U 1 1 5F702E62
-P 7500 3700
-F 0 "R413" V 7400 3450 50  0000 C CNN
-F 1 "500u" V 7400 3700 50  0000 C CNN
-F 2 "Resistor_SMD:R_2512_6332Metric" V 7430 3700 50  0001 C CNN
-F 3 "https://www.bourns.com/docs/Product-Datasheets/css2h-2512.pdf" H 7500 3700 50  0001 C CNN
-F 4 "5W" V 7400 3900 50  0000 C CNN "Power"
-	1    7500 3700
-	0    1    1    0
-$EndComp
-$Comp
-L power:+3.3V #PWR?
-U 1 1 5F71891D
-P 7050 4650
-AR Path="/5ECF1AA9/5F71891D" Ref="#PWR?"  Part="1"
-AR Path="/5F507ADF/5F71891D" Ref="#PWR0422"  Part="1"
-F 0 "#PWR0422" H 7050 4500 50  0001 C CNN
-F 1 "+3.3V" H 7065 4823 50  0000 C CNN
-F 2 "" H 7050 4650 50  0001 C CNN
-F 3 "" H 7050 4650 50  0001 C CNN
-	1    7050 4650
-	1    0    0    -1
-$EndComp
-Wire Wire Line
-	7400 4600 7400 4450
-Wire Wire Line
-	7600 4600 7600 4450
-$Comp
-L Device:R R?
-U 1 1 5F71892C
-P 7600 4300
-AR Path="/5ECF1AA9/5F71892C" Ref="R?"  Part="1"
-AR Path="/5F507ADF/5F71892C" Ref="R414"  Part="1"
-F 0 "R414" H 7750 4250 50  0000 C CNN
-F 1 "0" H 7700 4350 50  0000 C CNN
-F 2 "Resistor_SMD:R_0603_1608Metric" V 7530 4300 50  0001 C CNN
-F 3 "~" H 7600 4300 50  0001 C CNN
-	1    7600 4300
-	1    0    0    1
-$EndComp
-$Comp
-L Device:C_Small C?
-U 1 1 5F718936
-P 7050 4900
-AR Path="/5ECF1AA9/5F718936" Ref="C?"  Part="1"
-AR Path="/5F507ADF/5F718936" Ref="C411"  Part="1"
-F 0 "C411" H 7142 4946 50  0000 L CNN
-F 1 "0.1uF" H 7142 4855 50  0000 L CNN
-F 2 "Capacitor_SMD:C_0603_1608Metric" H 7050 4900 50  0001 C CNN
-F 3 "~" H 7050 4900 50  0001 C CNN
-	1    7050 4900
-	-1   0    0    -1
-$EndComp
-$Comp
-L power:GND #PWR?
-U 1 1 5F71893C
-P 7050 5000
-AR Path="/5ECF1AA9/5F71893C" Ref="#PWR?"  Part="1"
-AR Path="/5F507ADF/5F71893C" Ref="#PWR0423"  Part="1"
-F 0 "#PWR0423" H 7050 4750 50  0001 C CNN
-F 1 "GND" H 7055 4827 50  0000 C CNN
-F 2 "" H 7050 5000 50  0001 C CNN
-F 3 "" H 7050 5000 50  0001 C CNN
-	1    7050 5000
-	1    0    0    -1
-$EndComp
-Wire Wire Line
-	7050 4650 7050 4800
-Wire Wire Line
-	7050 4800 7200 4800
-Connection ~ 7050 4800
-$Comp
-L power:GND #PWR?
-U 1 1 5F76305C
-P 7850 4900
-AR Path="/5ECF1AA9/5F76305C" Ref="#PWR?"  Part="1"
-AR Path="/5F507ADF/5F76305C" Ref="#PWR0424"  Part="1"
-F 0 "#PWR0424" H 7850 4650 50  0001 C CNN
-F 1 "GND" H 7855 4727 50  0000 C CNN
-F 2 "" H 7850 4900 50  0001 C CNN
-F 3 "" H 7850 4900 50  0001 C CNN
-	1    7850 4900
-	1    0    0    -1
-$EndComp
-Wire Wire Line
-	7800 4800 7850 4800
-Wire Wire Line
-	7400 4150 7400 4100
-Wire Wire Line
-	7400 4100 7350 4100
-Wire Wire Line
-	7600 4150 7600 4100
-Wire Wire Line
-	7600 4100 7650 4100
-Wire Wire Line
-	7400 3950 7350 3950
-Connection ~ 7350 3950
-Wire Wire Line
-	7350 3950 7350 4100
-Wire Wire Line
-	7600 3950 7650 3950
-Wire Wire Line
-	7650 3950 7650 4100
-$Comp
-L power:GND #PWR?
-U 1 1 5F7A8457
-P 7050 4200
-AR Path="/5ECF1AA9/5F7A8457" Ref="#PWR?"  Part="1"
-AR Path="/5F7A8457" Ref="#PWR?"  Part="1"
-AR Path="/5F507ADF/5F7A8457" Ref="#PWR0421"  Part="1"
-F 0 "#PWR0421" H 7050 3950 50  0001 C CNN
-F 1 "GND" H 7055 4027 50  0000 C CNN
-F 2 "" H 7050 4200 50  0001 C CNN
-F 3 "" H 7050 4200 50  0001 C CNN
-	1    7050 4200
-	1    0    0    -1
-$EndComp
-Wire Wire Line
-	7050 4000 7050 3950
-Wire Wire Line
-	7050 3950 7350 3950
-Wire Wire Line
-	7500 5200 7500 5500
-$Comp
 L power:+BATT #PWR0401
 U 1 1 5FA71BA5
@@
 500uOhm resistor gives 50mV drop at 100A \nI^R losses are 5W\n
 $Comp
-L Amplifier_Current:INA194 U402
-U 1 1 5FF33ECB
-P 7500 4900
-F 0 "U402" V 7250 4450 50  0000 R CNN
-F 1 "INA194" V 7350 4550 50  0000 R CNN
-F 2 "Package_TO_SOT_SMD:SOT-23-5" H 7500 4900 50  0001 C CNN
-F 3 "http://www.ti.com/lit/ds/symlink/ina193.pdf" H 7500 4900 50  0001 C CNN
-	1    7500 4900
-	0    -1   1    0
-$EndComp
-Text Notes 6950 5700 0    39   ~ 0
-- Instrumentation amplifier w/ gain of 50V/V\n- Outputs 2.5V at 100A
-Wire Wire Line
-	7500 5500 6950 5500
-Text HLabel 6950 5500 0    39   Input ~ 0
-ANALOG_I_ESCS
-$Comp
 L Device:C_Small C?
 U 1 1 600D3098
@@
 Wire Wire Line
 	8900 3800 8900 3700
-Text HLabel 8500 4150 0    39   Input ~ 0
-ANALOG_V_ESCS
 Connection ~ 8900 1150
 Wire Wire Line
@@
 Wire Wire Line
 	6450 3700 6500 3700
-Wire Wire Line
-	7650 3700 8900 3700
 Connection ~ 8900 3700
 Wire Wire Line
@@
 $EndComp
 $Comp
-L Device:R R?
-U 1 1 5F718925
-P 7400 4300
-AR Path="/5ECF1AA9/5F718925" Ref="R?"  Part="1"
-AR Path="/5F507ADF/5F718925" Ref="R412"  Part="1"
-F 0 "R412" H 7250 4250 50  0000 C CNN
-F 1 "0" H 7300 4350 50  0000 C CNN
-F 2 "Resistor_SMD:R_0603_1608Metric" V 7330 4300 50  0001 C CNN
-F 3 "~" H 7400 4300 50  0001 C CNN
-	1    7400 4300
-	1    0    0    1
-$EndComp
-$Comp
 L power:GND #PWR?
 U 1 1 605F6239
@@
 Wire Wire Line
 	8700 1600 8900 1600
-$Comp
-L Device:C_Small C?
-U 1 1 60A3508A
-P 7050 4100
-AR Path="/5ECF1AA9/60A3508A" Ref="C?"  Part="1"
-AR Path="/60A3508A" Ref="C?"  Part="1"
-AR Path="/5F507ADF/60A3508A" Ref="C402"  Part="1"
-F 0 "C402" H 6958 4054 50  0000 R CNN
-F 1 "10nF" H 6958 4145 50  0000 R CNN
-F 2 "Capacitor_SMD:C_0603_1608Metric" H 7050 4100 50  0001 C CNN
-F 3 "~" H 7050 4100 50  0001 C CNN
-F 4 "25V" H 6900 4250 50  0000 C CNN "Voltage"
-F 5 "399-7842-2-ND" H 7050 4100 50  0001 C CNN "Digikey"
-	1    7050 4100
-	1    0    0    1
-$EndComp
-$Comp
-L Device:C_Small C?
-U 1 1 60A35E9C
-P 7500 3950
-AR Path="/5ECF1AA9/60A35E9C" Ref="C?"  Part="1"
-AR Path="/60A35E9C" Ref="C?"  Part="1"
-AR Path="/5F507ADF/60A35E9C" Ref="C403"  Part="1"
-F 0 "C403" V 7350 3750 50  0000 R CNN
-F 1 "10nF" V 7450 3750 50  0000 R CNN
-F 2 "Capacitor_SMD:C_0603_1608Metric" H 7500 3950 50  0001 C CNN
-F 3 "~" H 7500 3950 50  0001 C CNN
-F 4 "25V" V 7550 3650 50  0000 C CNN "Voltage"
-F 5 "399-7842-2-ND" H 7500 3950 50  0001 C CNN "Digikey"
-	1    7500 3950
-	0    -1   1    0
-$EndComp
 NoConn ~ 6250 4600
 $Comp
@@
 	6500 4050 6500 3700
 Connection ~ 6500 3700
-Wire Wire Line
-	6500 3700 7350 3700
 $Comp
 L Device:R_Small R411
@@
 	5800 4250 5750 4250
 Wire Wire Line
-	7350 3950 7350 3700
-Connection ~ 7350 3700
-Wire Wire Line
-	7650 3950 7650 3700
-Connection ~ 7650 3950
-Connection ~ 7650 3700
-Wire Wire Line
-	7850 4900 7850 4800
-Wire Wire Line
 	4450 4350 4950 4350
 $Bitmap
@@
 	0    -1   -1   0
 $EndComp
-Text Label 6500 3700 0    39   ~ 0
-ESC_OUTPUT_UNMEAS
+Text HLabel 8500 4150 0    39   Input ~ 0
+ANALOG_V_ESCS
+Wire Wire Line
+	6500 3700 8900 3700
 $EndSCHEMATC
