File: Frank/chum-bucket/PCB/SYS_MGMT.sch (KiCad schematic (older format))
At the start: 16 parts, among them Q401 SIR140DP, U401 MIC5014

Commit message: post-BOM order
Parts:
- C401: Digikey (none) -> 1276-1860-1-ND; Temp Co (none) -> X5R; Tempco X5R -> (none)
- C404, C405, C406, C413: Digikey 399-7842-2-ND -> 1276-1009-1-ND
- C_LIM401: Digikey (none) -> 1276-1009-1-ND
- R401, R411: Digikey (none) -> RMCF0603ZT0R00CT-ND
- R402, R404: Digikey (none) -> RNCP0603FTD10K0CT-ND
- R403: Digikey (none) -> A130092CT-ND
- R405: Digikey (none) -> 2019-RK73B1JTTD362JCT-ND
Other:
- note removed: "500uOhm resistor gives 50mV drop at 100A \nI^R losses are 5W\n"
Changed lines of the file:
@@
 F 2 "Capacitor_SMD:C_0603_1608Metric" H 6250 4600 50  0001 C CNN
 F 3 "~" H 6250 4600 50  0001 C CNN
+F 4 "1276-1009-1-ND" H 6250 4600 50  0001 C CNN "Digikey"
 	1    6250 4600
 	1    0    0    -1
@@
 Wire Wire Line
 	9800 1150 10350 1150
-Text Notes 7100 3550 0    39   ~ 0
-500uOhm resistor gives 50mV drop at 100A \nI^R losses are 5W\n
 $Comp
 L Device:C_Small C?
@@
 F 3 "~" H 9800 1600 50  0001 C CNN
 F 4 "25V" H 9650 1750 50  0000 C CNN "Voltage"
-F 5 "399-7842-2-ND" H 9800 1600 50  0001 C CNN "Digikey"
+F 5 "1276-1009-1-ND" H 9800 1600 50  0001 C CNN "Digikey"
 	1    9800 1600
 	-1   0    0    1
@@
 F 2 "Resistor_SMD:R_0603_1608Metric" V 8830 1400 50  0001 C CNN
 F 3 "~" H 8900 1400 50  0001 C CNN
+F 4 "RNCP0603FTD10K0CT-ND" H 8900 1400 50  0001 C CNN "Digikey"
 	1    8900 1400
 	1    0    0    -1
@@
 F 2 "Resistor_SMD:R_0603_1608Metric" V 8830 1800 50  0001 C CNN
 F 3 "~" H 8900 1800 50  0001 C CNN
+F 4 "A130092CT-ND" H 8900 1800 50  0001 C CNN "Digikey"
 	1    8900 1800
 	1    0    0    -1
@@
 F 2 "Resistor_SMD:R_0603_1608Metric" V 8830 3950 50  0001 C CNN
 F 3 "~" H 8900 3950 50  0001 C CNN
+F 4 "RNCP0603FTD10K0CT-ND" H 8900 3950 50  0001 C CNN "Digikey"
 	1    8900 3950
 	1    0    0    -1
@@
 F 2 "Resistor_SMD:R_0603_1608Metric" V 8830 4350 50  0001 C CNN
 F 3 "~" H 8900 4350 50  0001 C CNN
+F 4 "2019-RK73B1JTTD362JCT-ND" H 8900 4350 50  0001 C CNN "Digikey"
 	1    8900 4350
 	1    0    0    -1
@@
 F 3 "~" H 9800 4150 50  0001 C CNN
 F 4 "25V" H 9650 4300 50  0000 C CNN "Voltage"
-F 5 "399-7842-2-ND" H 9800 4150 50  0001 C CNN "Digikey"
+F 5 "1276-1009-1-ND" H 9800 4150 50  0001 C CNN "Digikey"
 	1    9800 4150
 	-1   0    0    1
@@
 F 3 "~" H 8700 4350 50  0001 C CNN
 F 4 "25V" H 8550 4500 50  0000 C CNN "Voltage"
-F 5 "399-7842-2-ND" H 8700 4350 50  0001 C CNN "Digikey"
+F 5 "1276-1009-1-ND" H 8700 4350 50  0001 C CNN "Digikey"
 	1    8700 4350
 	1    0    0    1
@@
 F 3 "~" H 8700 1800 50  0001 C CNN
 F 4 "25V" H 8550 1950 50  0000 C CNN "Voltage"
-F 5 "399-7842-2-ND" H 8700 1800 50  0001 C CNN "Digikey"
+F 5 "1276-1009-1-ND" H 8700 1800 50  0001 C CNN "Digikey"
 	1    8700 1800
 	1    0    0    1
@@
 	-1   0    0    -1
 $EndComp
-$Comp
-L Device:C_Small C?
-U 1 1 5FA2A915
-P 4550 3900
-AR Path="/5FA2A915" Ref="C?"  Part="1"
-AR Path="/5ECF181C/5FA2A915" Ref="C?"  Part="1"
-AR Path="/5F507ADF/5FA2A915" Ref="C401"  Part="1"
-F 0 "C401" H 4642 3946 50  0000 L CNN
-F 1 "1uF" H 4642 3855 50  0000 L CNN
-F 2 "Capacitor_SMD:C_0603_1608Metric" H 4550 3900 50  0001 C CNN
-F 3 "~" H 4550 3900 50  0001 C CNN
-F 4 "25V" H 4700 3650 50  0000 C CNN "Voltage"
-F 5 "X5R" H 4700 3750 50  0000 C CNN "Tempco"
-	1    4550 3900
-	-1   0    0    -1
-$EndComp
 Wire Wire Line
 	950  3700 4750 3700
@@
 F 2 "Resistor_SMD:R_0603_1608Metric" H 6250 4250 50  0001 C CNN
 F 3 "~" H 6250 4250 50  0001 C CNN
+F 4 "RMCF0603ZT0R00CT-ND" H 6250 4250 50  0001 C CNN "Digikey"
 	1    6250 4250
 	-1   0    0    1
@@
 F 2 "Resistor_SMD:R_0603_1608Metric" H 5900 4250 50  0001 C CNN
 F 3 "~" H 5900 4250 50  0001 C CNN
+F 4 "RMCF0603ZT0R00CT-ND" V 5900 4250 50  0001 C CNN "Digikey"
 	1    5900 4250
 	0    -1   1    0
@@
 Wire Wire Line
 	6500 3700 8900 3700
+$Comp
+L Device:C_Small C?
+U 1 1 600190A7
+P 4550 3900
+AR Path="/600190A7" Ref="C?"  Part="1"
+AR Path="/5ECF181C/600190A7" Ref="C?"  Part="1"
+AR Path="/5F507ADF/600190A7" Ref="C401"  Part="1"
+F 0 "C401" H 4642 3946 50  0000 L CNN
+F 1 "1uF" H 4642 3855 50  0000 L CNN
+F 2 "Capacitor_SMD:C_0603_1608Metric" H 4550 3900 50  0001 C CNN
+F 3 "~" H 4550 3900 50  0001 C CNN
+F 4 "1276-1860-1-ND" H 4550 3900 50  0001 C CNN "Digikey"
+F 5 "X5R" H 4750 3650 50  0000 C CNN "Temp Co"
+F 6 "25V" H 4700 3750 50  0000 C CNN "Voltage"
+	1    4550 3900
+	-1   0    0    -1
+$EndComp
 $EndSCHEMATC
