File: Frank/chum-bucket/PCB/BATT_MGMT.sch (KiCad schematic (older format))
At the start: 71 parts, among them Q301 AON2406, Q302 AON2406, Q303 AON2406, U301 BQ79606

Commit message: first (hopefully final) routing pass
Parts:
- removed R309, R312: 10k, Resistor_SMD:R_0603_1608Metric, symbol Device:R_Small
Connections:
- net BQ79606A_PWR_FUSED: now reaches F301.2, R325.1, R326.1
- net UART_BQ79606_STM_RX renamed UART_BQ79606_STM_JMP_P
- net UART_BQ79606_STM_TX renamed UART_BQ79606_STM_JMP_N
Changed lines of the file:
@@
 	1    0    0    -1
 $EndComp
-Wire Wire Line
-	2550 5950 2550 5850
-Wire Wire Line
-	2250 5950 2250 5850
-Wire Wire Line
-	2550 6150 2550 6500
-Wire Wire Line
-	2250 6150 2250 6400
-$Comp
-L Device:R_Small R?
-U 1 1 5F942689
-P 2250 6050
-AR Path="/5ECF1AA9/5F942689" Ref="R?"  Part="1"
-AR Path="/5F942689" Ref="R?"  Part="1"
-AR Path="/5ECF181C/5F942689" Ref="R309"  Part="1"
-F 0 "R309" H 2100 6000 50  0000 C CNN
-F 1 "10k" H 2100 6100 50  0000 C CNN
-F 2 "Resistor_SMD:R_0603_1608Metric" H 2250 6050 50  0001 C CNN
-F 3 "~" H 2250 6050 50  0001 C CNN
-	1    2250 6050
-	-1   0    0    1
-$EndComp
-$Comp
-L Device:R_Small R?
-U 1 1 5F942693
-P 2550 6050
-AR Path="/5ECF1AA9/5F942693" Ref="R?"  Part="1"
-AR Path="/5F942693" Ref="R?"  Part="1"
-AR Path="/5ECF181C/5F942693" Ref="R312"  Part="1"
-F 0 "R312" H 2450 5950 50  0000 C CNN
-F 1 "10k" H 2450 6050 50  0000 C CNN
-F 2 "Resistor_SMD:R_0603_1608Metric" H 2550 6050 50  0001 C CNN
-F 3 "~" H 2550 6050 50  0001 C CNN
-	1    2550 6050
-	-1   0    0    1
-$EndComp
 $Comp
 L chum-bucket:BQ79606 U?
@@
 	1550 6200 1650 6200
 Text HLabel 1550 6200 0    50   Input ~ 0
-UART_BQ79606_STM_RX
+UART_BQ79606_STM_JMP_P
 Wire Wire Line
 	1550 6300 1950 6300
@@
 Wire Wire Line
 	2850 5900 2850 5850
-Connection ~ 1650 6200
 Connection ~ 1950 5850
 Connection ~ 1950 6300
-Connection ~ 2250 5850
-Connection ~ 2250 6400
-Wire Wire Line
-	2250 6400 1550 6400
-Connection ~ 2550 5850
-Connection ~ 2550 6500
-Wire Wire Line
-	2550 6500 1550 6500
 Connection ~ 2850 5850
 Wire Wire Line
-	2250 6400 3100 6400
-Wire Wire Line
-	2550 6500 3100 6500
-Wire Wire Line
-	1950 5850 2250 5850
-Wire Wire Line
-	2550 5850 2850 5850
-Wire Wire Line
-	2250 5850 2550 5850
-Wire Wire Line
 	1950 6300 3100 6300
 Wire Wire Line
-	1650 6200 3100 6200
-Wire Wire Line
 	2850 5850 3100 5850
 Wire Wire Line
@@
 	8750 1000 9050 1000
 Text HLabel 1550 6300 0    50   Input ~ 0
-UART_BQ79606_STM_TX
+UART_BQ79606_STM_JMP_N
 Text Notes 4450 1700 0    39   ~ 0
 NOTE ABOUT THERMISTORS:\n- Voltage divider used for liniarization\n- Voltage divider and capacitor to be placed close\n   to BQ GPIO pins\n- Thermistors to be placed near cells
@@
 Data
 89 50 4E 47 0D 0A 1A 0A 00 00 00 0D 49 48 44 52 00 00 00 7D 00 00 00 A3 08 02 00 00 00 28 D6 86
-2D 00 00 00 03 73 42 49 54 08 08 08 DB E1 4F E0 00 00 00 09 70 48 59 73 00 00 0B 12 00 00 0B 12
-01 D2 DD 7E FC 00 00 20 00 49 44 41 54 78 9C D4 BD 79 B4 AD D9 51 1F 56 C3 DE FB 1B CE 39 77 7E
+2D 00 00 00 03 73 42 49 54 08 08 08 DB E1 4F E0 00 00 00 09 70 48 59 73 00 00 0A F0 00 00 0A F0
+01 42 AC 34 98 00 00 20 00 49 44 41 54 78 9C D4 BD 79 B4 AD D9 51 1F 56 C3 DE FB 1B CE 39 77 7E
 F7 BE F9 BD 1E D4 DD 92 50 B7 7A 50 4B 20 30 48 80 20 42 16 92 49 C0 18 DB C9 5A 31 CB 09 06 16
 38 4E 62 93 38 B1 13 3B 0B 42 08 2B B6 63 B3 02 C1 CB 22 31 C6 0C 06 6C 21 29 12 12 66 06 21 A1
@@
 Data
 89 50 4E 47 0D 0A 1A 0A 00 00 00 0D 49 48 44 52 00 00 01 1F 00 00 00 98 08 02 00 00 00 52 F7 7A
-CE 00 00 00 03 73 42 49 54 08 08 08 DB E1 4F E0 00 00 00 09 70 48 59 73 00 00 0E C3 00 00 0E C3
-01 C7 6F A8 64 00 00 20 00 49 44 41 54 78 9C EC BD 7B B8 6C 5B 55 1F F8 1B 63 CC B9 56 55 ED 7D
+CE 00 00 00 03 73 42 49 54 08 08 08 DB E1 4F E0 00 00 00 09 70 48 59 73 00 00 0E 74 00 00 0E 74
+01 6B 24 B3 D6 00 00 20 00 49 44 41 54 78 9C EC BD 7B B8 6C 5B 55 1F F8 1B 63 CC B9 56 55 ED 7D
 CE 7D 80 88 2F 30 B6 B6 0F B4 8D 69 A5 A3 9F 9F 7E DA 9D 48 A2 12 C4 74 8C 69 44 10 35 1A 1F 98
 F0 19 D0 26 1A 1B A2 A2 02 51 5E 09 F8 8A 46 04 1A 01 81 0B A8 10 5B 23 BE 00 45 13 5F 41 45 9E
@@
 Data
 89 50 4E 47 0D 0A 1A 0A 00 00 00 0D 49 48 44 52 00 00 00 7D 00 00 00 A3 08 02 00 00 00 28 D6 86
-2D 00 00 00 03 73 42 49 54 08 08 08 DB E1 4F E0 00 00 00 09 70 48 59 73 00 00 0B 12 00 00 0B 12
-01 D2 DD 7E FC 00 00 20 00 49 44 41 54 78 9C D4 BD 79 B4 AD D9 51 1F 56 C3 DE FB 1B CE 39 77 7E
+2D 00 00 00 03 73 42 49 54 08 08 08 DB E1 4F E0 00 00 00 09 70 48 59 73 00 00 0A F0 00 00 0A F0
+01 42 AC 34 98 00 00 20 00 49 44 41 54 78 9C D4 BD 79 B4 AD D9 51 1F 56 C3 DE FB 1B CE 39 77 7E
 F7 BE F9 BD 1E D4 DD 92 50 B7 7A 50 4B 20 30 48 80 20 42 16 92 49 C0 18 DB C9 5A 31 CB 09 06 16
 38 4E 62 93 38 B1 13 3B 0B 42 08 2B B6 63 B3 02 C1 CB 22 31 C6 0C 06 6C 21 29 12 12 66 06 21 A1
@@
 EndData
 $EndBitmap
+Text Label 8800 1000 0    39   ~ 0
+BQ79606A_PWR_FUSED
+Wire Wire Line
+	1550 6400 3100 6400
+Connection ~ 1650 6200
+Wire Wire Line
+	1650 6200 3100 6200
+Wire Wire Line
+	1550 6500 3100 6500
+Wire Wire Line
+	1950 5850 2850 5850
 $EndSCHEMATC

Commit message: routing V2
Parts:
- U301: footprint Package_QFP:LQFP-48-1EP_7x7mm_P0.5mm_EP3.6x3.6mm_ThermalVias -> CHUM_BUCKET_FOOTPRINTS:LQFP-48-1EP_7x7mm_P0.5mm_EP4x4mm_Thermalvias
Changed lines of the file:
@@
 F 0 "U301" H 3125 5315 50  0000 C CNN
 F 1 "BQ79606" H 3125 5224 50  0000 C CNN
-F 2 "Package_QFP:LQFP-48-1EP_7x7mm_P0.5mm_EP3.6x3.6mm_ThermalVias" H 3550 4650 50  0001 C CNN
+F 2 "CHUM_BUCKET_FOOTPRINTS:LQFP-48-1EP_7x7mm_P0.5mm_EP4x4mm_Thermalvias" H 3550 4650 50  0001 C CNN
 F 3 "https://www.ti.com/lit/ds/symlink/bq79606a-q1.pdf?HQS=TI-null-null-digikeymode-df-pf-null-wwe&ts=1592931025445" H 3450 4600 50  0001 C CNN
 F 4 "296-BQ79606APHPTQ1TR-ND" H 3450 4600 50  0001 C CNN "Digikey"

Commit message: post-BOM order
Parts:
- C301, C304, C305, C306, C309: Digikey (none) -> 1276-2016-1-ND
- C302, C303, C307, C308, C311, C312: Digikey (none) -> 1276-1009-1-ND
- C310: Digikey (none) -> 490-14466-1-ND; Voltage (none) -> 6V
- C313, C314, C315: Digikey (none) -> 1276-1860-1-ND
- C316, C317: value 0.33uF -> 1uF; Digikey (none) -> 1276-1860-1-ND
- C318, C319, C320, C321: value 0.47uF -> 1uF; Digikey (none) -> 1276-1860-1-ND
- C322, C323, C324: value 1nF -> 10nF; Digikey (none) -> 1276-1009-1-ND; Voltage (none) -> 6V
- D301, D302, D303: Digikey BAS16HT3GOSTR-ND -> BAS16HT3GOSCT-ND
- F301: Digikey P15127TR-ND -> P15127CT-ND
- Q301, Q302, Q303: Digikey 785-1491-2-ND -> 785-1491-1-ND
- R305, R306: Digikey (none) -> RNCP0603FTD10K0CT-ND
- R313: Digikey (none) -> RMCF0603ZT0R00CT-ND
- R318, R319, R320, R321: Digikey (none) -> RMCF0603FT100RCT-ND
- R322, R323, R324: Digikey (none) -> RHM1.0KDCT-ND
- R325: Digikey (none) -> RHM47DCT-ND; Power (none) -> 1/4W
- R326: Digikey (none) -> P100BZCT-ND; Power (none) -> 1/4W
- R327, R328, R329, R330: Digikey (none) -> RHM47DCT-ND
- R331, R332, R333: Digikey A121248TR-ND -> A121248CT-ND
- TH301, TH302, TH303, TH304, TH305, TH306: Digikey P12014TR-ND -> P12014CT-ND
- U301: Digikey 296-BQ79606APHPTQ1TR-ND -> 296-BQ79606APHPTQ1CT-ND
Connections:
- net PACK_GND: now also C324.1; no longer C324.2
- net SERIES_BANK_1: now also C323.1; no longer C323.2
- net SERIES_BANK_2: now also C322.1; no longer C322.2
- net at D302.1 (K), Q302.2 (G), R323.1: now also C323.2; no longer C323.1
- net at D303.1 (K), Q303.2 (G), R324.1: now also C324.2; no longer C324.1
- net at D301.1 (K), Q301.2 (G), R322.1: now also C322.2; no longer C322.1
