File: Frank/chum-bucket/PCB/CELLS.sch (KiCad schematic (older format))
At the start: 9 parts

Commit message: Weekends work. Final component selection then ready for review :)
huge oof
Parts:
- removed F?: 10A, symbol Device:Fuse
Connections:
- net SERIES_BANK_3 renamed +BATT
Changed lines of the file:
@@
 $Descr A4 11693 8268
 encoding utf-8
-Sheet 3 5
+Sheet 5 6
 Title ""
 Date ""
@@
 	1    0    0    -1
 $EndComp
-$Comp
-L Device:Fuse F?
-U 1 1 5F95ACF7
-P 5700 1600
-AR Path="/5F95ACF7" Ref="F?"  Part="1"
-AR Path="/5ECF2209/5F95ACF7" Ref="F?"  Part="1"
-F 0 "F?" H 5850 1450 50  0000 C CNN
-F 1 "10A" H 5850 1550 50  0000 C CNN
-F 2 "" V 5630 1600 50  0001 C CNN
-F 3 "~" H 5700 1600 50  0001 C CNN
-	1    5700 1600
-	-1   0    0    1
-$EndComp
 Wire Wire Line
 	5000 5900 5700 5900
@@
 	5700 5900 6400 5900
 Wire Wire Line
-	5700 1750 5700 1800
-Wire Wire Line
 	5000 2700 5000 2850
 Wire Wire Line
@@
 Wire Wire Line
 	5000 4600 5000 5050
-Text HLabel 5450 1200 0    50   Input ~ 0
-POS_BAT_FUSED
-Wire Wire Line
-	5700 1200 5450 1200
-Wire Wire Line
-	5700 1200 5700 1450
 Wire Wire Line
 	5700 1800 4050 1800
-Connection ~ 5700 1800
 Wire Wire Line
 	5700 1800 5700 2200
@@
 Text Notes 6750 3450 0    39   Italic 0
 To do: change 3 module cell numbering\nfor 'flipped' cell modules on the bottom of the board
+$Comp
+L power:+BATT #PWR?
+U 1 1 5FA4C998
+P 5700 1600
+F 0 "#PWR?" H 5700 1450 50  0001 C CNN
+F 1 "+BATT" H 5715 1773 50  0000 C CNN
+F 2 "" H 5700 1600 50  0001 C CNN
+F 3 "" H 5700 1600 50  0001 C CNN
+	1    5700 1600
+	1    0    0    -1
+$EndComp
+Wire Wire Line
+	5700 1600 5700 1800
+Connection ~ 5700 1800
 $EndSCHEMATC

Commit message: more work
Parts:
- gave numbers to parts that had none: 8
Changed lines of the file:
@@
 P 5350 4350
 AR Path="/5F95AC4A" Ref="U?"  Part="1"
-AR Path="/5ECF2209/5F95AC4A" Ref="U?"  Part="1"
-F 0 "U?" V 4850 4100 50  0000 L CNN
+AR Path="/5ECF2209/5F95AC4A" Ref="U209"  Part="1"
+F 0 "U209" V 4850 4100 50  0000 L CNN
 F 1 "CM" V 4950 4100 50  0000 L CNN
 F 2 "" H 5350 4400 50  0001 C CNN
@@
 P 5350 5300
 AR Path="/5F95AC50" Ref="U?"  Part="1"
-AR Path="/5ECF2209/5F95AC50" Ref="U?"  Part="1"
-F 0 "U?" V 4850 5050 50  0000 L CNN
+AR Path="/5ECF2209/5F95AC50" Ref="U210"  Part="1"
+F 0 "U210" V 4850 5050 50  0000 L CNN
 F 1 "CM" V 4950 5050 50  0000 L CNN
 F 2 "" H 5350 5350 50  0001 C CNN
@@
 P 6050 5300
 AR Path="/5F95AC56" Ref="U?"  Part="1"
-AR Path="/5ECF2209/5F95AC56" Ref="U?"  Part="1"
-F 0 "U?" V 5500 5450 50  0000 L CNN
+AR Path="/5ECF2209/5F95AC56" Ref="U214"  Part="1"
+F 0 "U214" V 5500 5450 50  0000 L CNN
 F 1 "CM" V 5600 5450 50  0000 L CNN
 F 2 "" H 6050 5350 50  0001 C CNN
@@
 P 6050 2450
 AR Path="/5F95AC5C" Ref="U?"  Part="1"
-AR Path="/5ECF2209/5F95AC5C" Ref="U?"  Part="1"
-F 0 "U?" V 5550 2200 50  0000 L CNN
+AR Path="/5ECF2209/5F95AC5C" Ref="U211"  Part="1"
+F 0 "U211" V 5550 2200 50  0000 L CNN
 F 1 "CM" V 5650 2200 50  0000 L CNN
 F 2 "" H 6050 2500 50  0001 C CNN
@@
 P 6050 3400
 AR Path="/5F95AC62" Ref="U?"  Part="1"
-AR Path="/5ECF2209/5F95AC62" Ref="U?"  Part="1"
-F 0 "U?" V 5550 3150 50  0000 L CNN
+AR Path="/5ECF2209/5F95AC62" Ref="U212"  Part="1"
+F 0 "U212" V 5550 3150 50  0000 L CNN
 F 1 "CM" V 5650 3150 50  0000 L CNN
 F 2 "" H 6050 3450 50  0001 C CNN
@@
 P 6050 4350
 AR Path="/5F95AC68" Ref="U?"  Part="1"
-AR Path="/5ECF2209/5F95AC68" Ref="U?"  Part="1"
-F 0 "U?" V 5550 4100 50  0000 L CNN
+AR Path="/5ECF2209/5F95AC68" Ref="U213"  Part="1"
+F 0 "U213" V 5550 4100 50  0000 L CNN
 F 1 "CM" V 5650 4100 50  0000 L CNN
 F 2 "" H 6050 4400 50  0001 C CNN
@@
 P 5350 2450
 AR Path="/5F95AC6E" Ref="U?"  Part="1"
-AR Path="/5ECF2209/5F95AC6E" Ref="U?"  Part="1"
-F 0 "U?" V 4900 2200 50  0000 L CNN
+AR Path="/5ECF2209/5F95AC6E" Ref="U207"  Part="1"
+F 0 "U207" V 4900 2200 50  0000 L CNN
 F 1 "CM" V 5000 2200 50  0000 L CNN
 F 2 "" H 5350 2500 50  0001 C CNN
@@
 P 5350 3400
 AR Path="/5F95AC74" Ref="U?"  Part="1"
-AR Path="/5ECF2209/5F95AC74" Ref="U?"  Part="1"
-F 0 "U?" V 4900 3150 50  0000 L CNN
+AR Path="/5ECF2209/5F95AC74" Ref="U208"  Part="1"
+F 0 "U208" V 4900 3150 50  0000 L CNN
 F 1 "CM" V 5000 3150 50  0000 L CNN
 F 2 "" H 5350 3450 50  0001 C CNN
@@
 P 5700 6050
 AR Path="/5F95ACF1" Ref="#PWR?"  Part="1"
-AR Path="/5ECF2209/5F95ACF1" Ref="#PWR?"  Part="1"
-F 0 "#PWR?" H 5700 5800 50  0001 C CNN
+AR Path="/5ECF2209/5F95ACF1" Ref="#PWR0260"  Part="1"
+F 0 "#PWR0260" H 5700 5800 50  0001 C CNN
 F 1 "GND" H 5705 5877 50  0000 C CNN
 F 2 "" H 5700 6050 50  0001 C CNN
@@
 To do: change 3 module cell numbering\nfor 'flipped' cell modules on the bottom of the board
 $Comp
-L power:+BATT #PWR?
+L power:+BATT #PWR0259
 U 1 1 5FA4C998
 P 5700 1600
-F 0 "#PWR?" H 5700 1450 50  0001 C CNN
+F 0 "#PWR0259" H 5700 1450 50  0001 C CNN
 F 1 "+BATT" H 5715 1773 50  0000 C CNN
 F 2 "" H 5700 1600 50  0001 C CNN

Commit message: some layout
Parts:
- removed U207, U208, U209, U210, U211, U212, U213, U214: CM, symbol chum-bucket:3_Cell_Module
- added BT1, BT10, BT11, BT12, BT13, BT14, BT15, BT16, BT17, BT18, BT19, BT2, BT20, BT21, BT22, BT23, BT24, BT3, BT4, BT5, BT6, BT7, BT8, BT9: 18650, CHUM_BUCKET_FOOTPRINTS:Keystone_1042p_18650_Holder, symbol Device:Battery_Cell
Connections:
- net +BATT: now also BT10.1 (+), BT13.1 (+), BT16.1 (+), BT19.1 (+), BT2.1 (+), BT22.1 (+), BT4.1 (+), BT7.1 (+)
- net GND: now also BT1.2 (-), BT12.2 (-), BT15.2 (-), BT18.2 (-), BT21.2 (-), BT24.2 (-), BT6.2 (-), BT9.2 (-)
- net SERIES_BANK_1: now also BT1.1 (+), BT11.2 (-), BT12.1 (+), BT14.2 (-), BT15.1 (+), BT17.2 (-), BT18.1 (+), BT20.2 (-), BT21.1 (+), BT23.2 (-), BT24.1 (+), BT3.2 (-), BT5.2 (-), BT6.1 (+), BT8.2 (-), BT9.1 (+)
- net SERIES_BANK_2: now also BT10.2 (-), BT11.1 (+), BT13.2 (-), BT14.1 (+), BT16.2 (-), BT17.1 (+), BT19.2 (-), BT2.2 (-), BT20.1 (+), BT22.2 (-), BT23.1 (+), BT3.1 (+), BT4.2 (-), BT5.1 (+), BT7.2 (-), BT8.1 (+)
Other:
- note removed: "To do: change 3 module cell numbering\nfor 'flipped' cell modules on the bottom of the board"

Commit message: post-BOM order
Parts:
- BT1, BT10, BT11, BT12, BT13, BT14, BT15, BT16, BT17, BT18, BT19, BT2, BT20, BT21, BT22, BT23, BT24, BT3, BT4, BT5, BT6, BT7, BT8, BT9: Digikey (none) -> 36-1042-ND
Changed lines of the file:
@@
 F 2 "CHUM_BUCKET_FOOTPRINTS:Keystone_1042p_18650_Holder" V 5350 4860 50  0001 C CNN
 F 3 "~" V 5350 4860 50  0001 C CNN
+F 4 "36-1042-ND" H 5350 4800 50  0001 C CNN "Digikey"
 	1    5350 4800
 	1    0    0    -1
@@
 F 2 "CHUM_BUCKET_FOOTPRINTS:Keystone_1042p_18650_Holder" V 5850 4860 50  0001 C CNN
 F 3 "~" V 5850 4860 50  0001 C CNN
+F 4 "36-1042-ND" H 5850 4800 50  0001 C CNN "Digikey"
 	1    5850 4800
 	1    0    0    -1
@@
 F 2 "CHUM_BUCKET_FOOTPRINTS:Keystone_1042p_18650_Holder" V 6300 4860 50  0001 C CNN
 F 3 "~" V 6300 4860 50  0001 C CNN
+F 4 "36-1042-ND" H 6300 4800 50  0001 C CNN "Digikey"
 	1    6300 4800
 	1    0    0    -1
@@
 F 2 "CHUM_BUCKET_FOOTPRINTS:Keystone_1042p_18650_Holder" V 6750 4860 50  0001 C CNN
 F 3 "~" V 6750 4860 50  0001 C CNN
+F 4 "36-1042-ND" H 6750 4800 50  0001 C CNN "Digikey"
 	1    6750 4800
 	1    0    0    -1
@@
 F 2 "CHUM_BUCKET_FOOTPRINTS:Keystone_1042p_18650_Holder" V 7200 4860 50  0001 C CNN
 F 3 "~" V 7200 4860 50  0001 C CNN
+F 4 "36-1042-ND" H 7200 4800 50  0001 C CNN "Digikey"
 	1    7200 4800
 	1    0    0    -1
 $EndComp
-$Comp
-L Device:Battery_Cell BT18
-U 1 1 5FADEDB1
-P 7700 4800
-F 0 "BT18" H 7818 4896 50  0000 L CNN
-F 1 "18650" H 7818 4805 50  0000 L CNN
-F 2 "CHUM_BUCKET_FOOTPRINTS:Keystone_1042p_18650_Holder" V 7700 4860 50  0001 C CNN
-F 3 "~" V 7700 4860 50  0001 C CNN
-	1    7700 4800
-	1    0    0    -1
-$EndComp
-$Comp
-L Device:Battery_Cell BT21
-U 1 1 5FADEDB7
-P 8150 4800
-F 0 "BT21" H 8268 4896 50  0000 L CNN
-F 1 "18650" H 8268 4805 50  0000 L CNN
-F 2 "CHUM_BUCKET_FOOTPRINTS:Keystone_1042p_18650_Holder" V 8150 4860 50  0001 C CNN
-F 3 "~" V 8150 4860 50  0001 C CNN
-	1    8150 4800
-	1    0    0    -1
-$EndComp
-$Comp
-L Device:Battery_Cell BT24
-U 1 1 5FADEDBD
-P 8600 4800
-F 0 "BT24" H 8718 4896 50  0000 L CNN
-F 1 "18650" H 8718 4805 50  0000 L CNN
-F 2 "CHUM_BUCKET_FOOTPRINTS:Keystone_1042p_18650_Holder" V 8600 4860 50  0001 C CNN
-F 3 "~" V 8600 4860 50  0001 C CNN
-	1    8600 4800
-	1    0    0    -1
-$EndComp
 Wire Wire Line
 	5350 4600 5350 4450
@@
 F 2 "CHUM_BUCKET_FOOTPRINTS:Keystone_1042p_18650_Holder" V 5350 3610 50  0001 C CNN
 F 3 "~" V 5350 3610 50  0001 C CNN
+F 4 "36-1042-ND" H 5350 3550 50  0001 C CNN "Digikey"
 	1    5350 3550
 	1    0    0    -1
@@
 F 2 "CHUM_BUCKET_FOOTPRINTS:Keystone_1042p_18650_Holder" V 5850 3610 50  0001 C CNN
 F 3 "~" V 5850 3610 50  0001 C CNN
+F 4 "36-1042-ND" H 5850 3550 50  0001 C CNN "Digikey"
 	1    5850 3550
 	1    0    0    -1
@@
 F 2 "CHUM_BUCKET_FOOTPRINTS:Keystone_1042p_18650_Holder" V 6300 3610 50  0001 C CNN
 F 3 "~" V 6300 3610 50  0001 C CNN
+F 4 "36-1042-ND" H 6300 3550 50  0001 C CNN "Digikey"
 	1    6300 3550
 	1    0    0    -1
@@
 F 2 "CHUM_BUCKET_FOOTPRINTS:Keystone_1042p_18650_Holder" V 6750 3610 50  0001 C CNN
 F 3 "~" V 6750 3610 50  0001 C CNN
+F 4 "36-1042-ND" H 6750 3550 50  0001 C CNN "Digikey"
 	1    6750 3550
 	1    0    0    -1
@@
 F 2 "CHUM_BUCKET_FOOTPRINTS:Keystone_1042p_18650_Holder" V 7200 3610 50  0001 C CNN
 F 3 "~" V 7200 3610 50  0001 C CNN
+F 4 "36-1042-ND" H 7200 3550 50  0001 C CNN "Digikey"
 	1    7200 3550
 	1    0    0    -1
@@
 F 2 "CHUM_BUCKET_FOOTPRINTS:Keystone_1042p_18650_Holder" V 7700 3610 50  0001 C CNN
 F 3 "~" V 7700 3610 50  0001 C CNN
+F 4 "36-1042-ND" H 7700 3550 50  0001 C CNN "Digikey"
 	1    7700 3550
 	1    0    0    -1
@@
 F 2 "CHUM_BUCKET_FOOTPRINTS:Keystone_1042p_18650_Holder" V 8150 3610 50  0001 C CNN
 F 3 "~" V 8150 3610 50  0001 C CNN
+F 4 "36-1042-ND" H 8150 3550 50  0001 C CNN "Digikey"
 	1    8150 3550
 	1    0    0    -1
@@
 F 2 "CHUM_BUCKET_FOOTPRINTS:Keystone_1042p_18650_Holder" V 8600 3610 50  0001 C CNN
 F 3 "~" V 8600 3610 50  0001 C CNN
+F 4 "36-1042-ND" H 8600 3550 50  0001 C CNN "Digikey"
 	1    8600 3550
 	1    0    0    -1
@@
 F 2 "CHUM_BUCKET_FOOTPRINTS:Keystone_1042p_18650_Holder" V 5300 2460 50  0001 C CNN
 F 3 "~" V 5300 2460 50  0001 C CNN
+F 4 "36-1042-ND" H 5300 2400 50  0001 C CNN "Digikey"
 	1    5300 2400
 	1    0    0    -1
@@
 F 2 "CHUM_BUCKET_FOOTPRINTS:Keystone_1042p_18650_Holder" V 5800 2460 50  0001 C CNN
 F 3 "~" V 5800 2460 50  0001 C CNN
+F 4 "36-1042-ND" H 5800 2400 50  0001 C CNN "Digikey"
 	1    5800 2400
 	1    0    0    -1
@@
 F 2 "CHUM_BUCKET_FOOTPRINTS:Keystone_1042p_18650_Holder" V 6250 2460 50  0001 C CNN
 F 3 "~" V 6250 2460 50  0001 C CNN
+F 4 "36-1042-ND" H 6250 2400 50  0001 C CNN "Digikey"
 	1    6250 2400
 	1    0    0    -1
@@
 F 2 "CHUM_BUCKET_FOOTPRINTS:Keystone_1042p_18650_Holder" V 6700 2460 50  0001 C CNN
 F 3 "~" V 6700 2460 50  0001 C CNN
+F 4 "36-1042-ND" H 6700 2400 50  0001 C CNN "Digikey"
 	1    6700 2400
 	1    0    0    -1
@@
 F 2 "CHUM_BUCKET_FOOTPRINTS:Keystone_1042p_18650_Holder" V 7150 2460 50  0001 C CNN
 F 3 "~" V 7150 2460 50  0001 C CNN
+F 4 "36-1042-ND" H 7150 2400 50  0001 C CNN "Digikey"
 	1    7150 2400
 	1    0    0    -1
@@
 F 2 "CHUM_BUCKET_FOOTPRINTS:Keystone_1042p_18650_Holder" V 7650 2460 50  0001 C CNN
 F 3 "~" V 7650 2460 50  0001 C CNN
+F 4 "36-1042-ND" H 7650 2400 50  0001 C CNN "Digikey"
 	1    7650 2400
 	1    0    0    -1
@@
 F 2 "CHUM_BUCKET_FOOTPRINTS:Keystone_1042p_18650_Holder" V 8100 2460 50  0001 C CNN
 F 3 "~" V 8100 2460 50  0001 C CNN
+F 4 "36-1042-ND" H 8100 2400 50  0001 C CNN "Digikey"
 	1    8100 2400
 	1    0    0    -1
@@
 F 2 "CHUM_BUCKET_FOOTPRINTS:Keystone_1042p_18650_Holder" V 8550 2460 50  0001 C CNN
 F 3 "~" V 8550 2460 50  0001 C CNN
+F 4 "36-1042-ND" H 8550 2400 50  0001 C CNN "Digikey"
 	1    8550 2400
 	1    0    0    -1
@@
 EndData
 $EndBitmap
+$Comp
+L Device:Battery_Cell BT18
+U 1 1 5FADEDB1
+P 7700 4800
+F 0 "BT18" H 7818 4896 50  0000 L CNN
+F 1 "18650" H 7818 4805 50  0000 L CNN
+F 2 "CHUM_BUCKET_FOOTPRINTS:Keystone_1042p_18650_Holder" V 7700 4860 50  0001 C CNN
+F 3 "~" V 7700 4860 50  0001 C CNN
+F 4 "36-1042-ND" H 7700 4800 50  0001 C CNN "Digikey"
+	1    7700 4800
+	1    0    0    -1
+$EndComp
+$Comp
+L Device:Battery_Cell BT21
+U 1 1 5FADEDB7
+P 8150 4800
+F 0 "BT21" H 8268 4896 50  0000 L CNN
+F 1 "18650" H 8268 4805 50  0000 L CNN
+F 2 "CHUM_BUCKET_FOOTPRINTS:Keystone_1042p_18650_Holder" V 8150 4860 50  0001 C CNN
+F 3 "~" V 8150 4860 50  0001 C CNN
+F 4 "36-1042-ND" H 8150 4800 50  0001 C CNN "Digikey"
+	1    8150 4800
+	1    0    0    -1
+$EndComp
+$Comp
+L Device:Battery_Cell BT24
+U 1 1 5FADEDBD
+P 8600 4800
+F 0 "BT24" H 8718 4896 50  0000 L CNN
+F 1 "18650" H 8718 4805 50  0000 L CNN
+F 2 "CHUM_BUCKET_FOOTPRINTS:Keystone_1042p_18650_Holder" V 8600 4860 50  0001 C CNN
+F 3 "~" V 8600 4860 50  0001 C CNN
+F 4 "36-1042-ND" H 8600 4800 50  0001 C CNN "Digikey"
+	1    8600 4800
+	1    0    0    -1
+$EndComp
 $EndSCHEMATC
