File: Mark/WPT_RX/WPT_RX.sch (KiCad schematic (older format))
At the start: 0 parts

Commit message: Finished RX Schematic
- Finsihed RX schematic
- Completed RX BOM
- Added all footprints
- Only power resistor 3D model is outstanding, will add that later
Parts:
- added C1, C2, C7, C8, C9: 0.1u, Capacitor_SMD:C_0603_1608Metric, symbol Device:C_Small
- added C10, C11, C12: 330u, Capacitor_SMD:CP_Elec_10x12.5, symbol Device:CP1
- added C3, C4, C5, C6: 100n, Capacitor_SMD:C_2220_5650Metric, symbol Device:C_Small
- added D1, D2, D3, D4: FSV12100V, Package_TO_SOT_SMD:TO-277B, symbol Device:D_Schottky
- added D5: RED, LED_SMD:LED_0805_2012Metric, symbol Device:LED
- added J1, J2, J6, J7: Conn_01x01, WPT_RX:SolderWirePad_single_SMD_5x10mm, symbol Connector_Generic:Conn_01x01
- added J3, J4, J5: SMA, WPT_RX:SMA_Amphenol_901-144_Vertical, symbol Connector:Conn_Coaxial
- added J8: From PI Board, WPT_RX:70553-02, symbol Connector_Generic:Conn_01x02
- added NT1, NT2: Net-Tie_2, WPT_RX:NetTie-2_SMD_Pad0.25mm, symbol Device:Net-Tie_2
- added Q1: NMOS, WPT_RX:TDSON-8-1, symbol Device:Q_NMOS_SGD
- added R1: 11.5k, Resistor_SMD:R_0603_1608Metric, symbol Device:R_US
- added R10, R5, R7: 10k, Resistor_SMD:R_0603_1608Metric, symbol Device:R_US
- added R11: 5m, WPT_RX:R_2512_Sense, symbol Device:R_US
- added R12, R13, R14, R9: 10R, Package_TO_SOT_THT:TO-220F-2_Horizontal_TabDown, symbol Device:R_US
- added R2: 9.09k, Resistor_SMD:R_0603_1608Metric, symbol Device:R_US
- added R3: 18.0k, Resistor_SMD:R_0603_1608Metric, symbol Device:R_US
- added R4: 2.0k, Resistor_SMD:R_0603_1608Metric, symbol Device:R_US
- added R6, R8: 0.4k, Resistor_SMD:R_0603_1608Metric, symbol Device:R_US
- added TP1, TP2, TP3, TP4, TP5, TP6, TP7, TP8: TestPoint, TestPoint:TestPoint_Loop_D1.80mm_Drill1.0mm_Beaded, symbol Connector:TestPoint
- added U1: LMC6032, Package_SO:SOIC-8_3.9x4.9mm_P1.27mm, symbol Amplifier_Operational:LMC6082
- added U2: INA240D, Package_SO:SOIC-8_3.9x4.9mm_P1.27mm, symbol Amplifier_Current:INA240A1D
- added U3: MUN, WPT_RX:MUNLOGO, symbol WPT_RX:Munlogo
Connections:
- new net: C3.2, C4.2, C5.2, C6.2, J1.1 (Pin_1)
- new net: D1.2 (A), D2.1 (K), J2.1 (Pin_1), J3.2 (Ext), J5.1 (In), TP3.1
- new net: C3.1, C4.1, C5.1, C6.1, D3.2 (A), D4.1 (K), J3.1 (In), J4.1 (In), TP2.1
- new net: Q1.3 (D), R12.2, R13.2, R14.2, R9.2
- new net: R5.1, U2.5
- new net: R6.2, U1.1, U1.2 (-)
- new net: C8.1, R3.2, R4.1, U1.3 (+)
- new net: R6.1, R7.2, U1.5 (+)
- new net: D5.1 (K), R8.2
- new net +5V: C1.1, C2.1, J8.1 (Pin_1), R1.1, U1.8 (V+), U2.6 (V+)
- new net +BATT: J6.1 (Pin_1), NT2.1, R11.2, R12.1, R13.1, R14.1, R9.1, TP6.1
- new net FAULT_OVP: D5.2 (A), Q1.2 (G), R10.1, R7.1, TP5.1, U1.7
- new net GND: C1.2, C10.2, C11.2, C12.2, C2.2, C7.2, C8.2, C9.2, D2.2 (A), D4.2 (A), J4.2 (Ext), J5.2 (Ext), J7.1 (Pin_1), J8.2 (Pin_2), Q1.1 (S), R10.2, R2.2, R4.2, R8.1, TP7.1, TP8.1, U1.4 (V-), U2.2 (GND), U2.3 (REF2), U2.4 (GND), U2.7 (REF1)
- new net ISEN: C9.1, R5.2, TP4.1
- new net ISEN+: NT1.1, U2.8 (+)
- new net ISEN-: NT2.2, U2.1 (-)
- new net VREF: C7.1, R1.2, R2.1, U1.6 (-)
- new net VSEN: C10.1, C11.1, C12.1, D1.1 (K), D3.1 (K), NT1.2, R11.1, R3.1, TP1.1
Other:
- note added: "Charger+"
- note added: "Extras"
- note added: "Full Bridge Rectifier"
- note added: "GND"
- note added: "Output Current Sense"
- note added: "Over Voltage Fault Detection"
- note added: "Over Voltage Power Drain"
- note added: "RX Coil+"
- note added: "RX Coil-"
