File: Mark/WPT_RX/_autosave-WPT_RX.sch (KiCad schematic (older format))
At the start: 58 parts, among them J1 Conn_01x01, J2 Conn_01x01, J3 SMA, J4 SMA, J5 SMA, J6 Conn_01x01, J7 Conn_01x01, J8 From PI Board, Q1 NMOS, U1 LMC6032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

Commit message: RX Layout
- Completed layout
- Also cleaned up some silkscreen since I was in the zone.
Parts:
- gave numbers to parts that had none: 1
Changed lines of the file:
@@
 $EndComp
 $Comp
-L Device:C_Small C?
+L Device:C_Small C13
 U 1 1 5FBB5F7F
 P 2500 5250
-F 0 "C?" H 2450 5450 50  0000 L CNN
+F 0 "C13" H 2450 5450 50  0000 L CNN
 F 1 "0.1u" H 2400 5075 50  0000 L CNN
 F 2 "Capacitor_SMD:C_0603_1608Metric" H 2500 5250 50  0001 C CNN
