File: Mark/WPT_TX/WPT_TX.sch (KiCad schematic (older format))
At the start: 4 parts

Commit message: Sims and Sch
- Played around with the sims
- Selected FETs for TX board, did calcs to make sure losses are good. (They are reallyyyyy low, even for 200kHz switching)
Parts:
- added Q? (x4): NMOS, WPT_TX:TDSON-8-1, symbol Device:Q_NMOS_SGD
Connections:
- net labels added: +24V, GATE1, GATE2, GATE3, GATE4, GND
- wire segments 0 -> 26
Other:
- note added: "Coil+"
- note added: "Coil-"
- note added: "VIN+"
- note added: "VIN-"
Changed lines of the file:
@@
 Data
 89 50 4E 47 0D 0A 1A 0A 00 00 00 0D 49 48 44 52 00 00 01 1F 00 00 00 98 08 02 00 00 00 52 F7 7A
-CE 00 00 00 03 73 42 49 54 08 08 08 DB E1 4F E0 00 00 00 09 70 48 59 73 00 00 0E C3 00 00 0E C3
-01 C7 6F A8 64 00 00 20 00 49 44 41 54 78 9C EC BD 7B B8 6C 5B 55 1F F8 1B 63 CC B9 56 55 ED 7D
+CE 00 00 00 03 73 42 49 54 08 08 08 DB E1 4F E0 00 00 00 09 70 48 59 73 00 00 0E 74 00 00 0E 74
+01 6B 24 B3 D6 00 00 20 00 49 44 41 54 78 9C EC BD 7B B8 6C 5B 55 1F F8 1B 63 CC B9 56 55 ED 7D
 CE 7D 80 88 2F 30 B6 B6 0F B4 8D 69 A5 A3 9F 9F 7E DA 9D 48 A2 12 C4 74 8C 69 44 10 35 1A 1F 98
 F0 19 D0 26 1A 1B A2 A2 02 51 5E 09 F8 8A 46 04 1A 01 81 0B A8 10 5B 23 BE 00 45 13 5F 41 45 9E
@@
 L Connector_Generic:Conn_01x01 J?
 U 1 1 5F967A9F
-P 1800 1600
-F 0 "J?" H 2000 1600 50  0000 C CNN
-F 1 "Conn_01x01" H 1718 1466 50  0001 C CNN
-F 2 "" H 1800 1600 50  0001 C CNN
-F 3 "~" H 1800 1600 50  0001 C CNN
-	1    1800 1600
+P 3125 1425
+F 0 "J?" H 3325 1425 50  0000 C CNN
+F 1 "Conn_01x01" H 3043 1291 50  0001 C CNN
+F 2 "" H 3125 1425 50  0001 C CNN
+F 3 "~" H 3125 1425 50  0001 C CNN
+	1    3125 1425
 	-1   0    0    1
 $EndComp
@@
 L Connector_Generic:Conn_01x01 J?
 U 1 1 5F969337
-P 1800 2250
-F 0 "J?" H 2000 2250 50  0000 C CNN
-F 1 "Conn_01x01" H 1718 2116 50  0001 C CNN
-F 2 "" H 1800 2250 50  0001 C CNN
-F 3 "~" H 1800 2250 50  0001 C CNN
-	1    1800 2250
+P 3125 2925
+F 0 "J?" H 3325 2925 50  0000 C CNN
+F 1 "Conn_01x01" H 3043 2791 50  0001 C CNN
+F 2 "" H 3125 2925 50  0001 C CNN
+F 3 "~" H 3125 2925 50  0001 C CNN
+	1    3125 2925
 	-1   0    0    1
 $EndComp
@@
 L Connector_Generic:Conn_01x01 J?
 U 1 1 5F96A356
-P 7500 1650
-F 0 "J?" H 7580 1646 50  0000 L CNN
-F 1 "Conn_01x01" H 7418 1516 50  0001 C CNN
-F 2 "" H 7500 1650 50  0001 C CNN
-F 3 "~" H 7500 1650 50  0001 C CNN
-	1    7500 1650
+P 7750 1425
+F 0 "J?" H 7830 1421 50  0000 L CNN
+F 1 "Conn_01x01" H 7668 1291 50  0001 C CNN
+F 2 "" H 7750 1425 50  0001 C CNN
+F 3 "~" H 7750 1425 50  0001 C CNN
+	1    7750 1425
 	1    0    0    -1
 $EndComp
@@
 L Connector_Generic:Conn_01x01 J?
 U 1 1 5F96C377
-P 7500 2250
-F 0 "J?" H 7580 2246 50  0000 L CNN
-F 1 "Conn_01x01" H 7418 2116 50  0001 C CNN
-F 2 "" H 7500 2250 50  0001 C CNN
-F 3 "~" H 7500 2250 50  0001 C CNN
-	1    7500 2250
+P 7750 2925
+F 0 "J?" H 7830 2921 50  0000 L CNN
+F 1 "Conn_01x01" H 7668 2791 50  0001 C CNN
+F 2 "" H 7750 2925 50  0001 C CNN
+F 3 "~" H 7750 2925 50  0001 C CNN
+	1    7750 2925
 	1    0    0    -1
 $EndComp
+$Comp
+L Device:Q_NMOS_SGD Q?
+U 1 1 5F980BB8
+P 5225 1775
+F 0 "Q?" H 5429 1821 50  0000 L CNN
+F 1 "NMOS" H 5429 1730 50  0000 L CNN
+F 2 "WPT_TX:TDSON-8-1" H 5425 1875 50  0001 C CNN
+F 3 "https://www.infineon.com/dgdl/Infineon-IAUC70N08S5N074-DS-v01_00-EN.pdf?fileId=5546d46266a498f50166a531f6aa0013" H 5225 1775 50  0001 C CNN
+F 4 "448-IAUC70N08S5N074ATMA1CT-ND" H 5225 1775 50  0001 C CNN "Digikey"
+	1    5225 1775
+	1    0    0    -1
+$EndComp
+$Comp
+L Device:Q_NMOS_SGD Q?
+U 1 1 5F981A5A
+P 5225 2525
+F 0 "Q?" H 5429 2571 50  0000 L CNN
+F 1 "NMOS" H 5429 2480 50  0000 L CNN
+F 2 "WPT_TX:TDSON-8-1" H 5425 2625 50  0001 C CNN
+F 3 "https://www.infineon.com/dgdl/Infineon-IAUC70N08S5N074-DS-v01_00-EN.pdf?fileId=5546d46266a498f50166a531f6aa0013" H 5225 2525 50  0001 C CNN
+F 4 "448-IAUC70N08S5N074ATMA1CT-ND" H 5225 2525 50  0001 C CNN "Digikey"
+	1    5225 2525
+	1    0    0    -1
+$EndComp
+$Comp
+L Device:Q_NMOS_SGD Q?
+U 1 1 5F985A5D
+P 6150 1775
+F 0 "Q?" H 6354 1821 50  0000 L CNN
+F 1 "NMOS" H 6354 1730 50  0000 L CNN
+F 2 "WPT_TX:TDSON-8-1" H 6350 1875 50  0001 C CNN
+F 3 "https://www.infineon.com/dgdl/Infineon-IAUC70N08S5N074-DS-v01_00-EN.pdf?fileId=5546d46266a498f50166a531f6aa0013" H 6150 1775 50  0001 C CNN
+F 4 "448-IAUC70N08S5N074ATMA1CT-ND" H 6150 1775 50  0001 C CNN "Digikey"
+	1    6150 1775
+	1    0    0    -1
+$EndComp
+$Comp
+L Device:Q_NMOS_SGD Q?
+U 1 1 5F986F7C
+P 6150 2525
+F 0 "Q?" H 6354 2571 50  0000 L CNN
+F 1 "NMOS" H 6354 2480 50  0000 L CNN
+F 2 "WPT_TX:TDSON-8-1" H 6350 2625 50  0001 C CNN
+F 3 "https://www.infineon.com/dgdl/Infineon-IAUC70N08S5N074-DS-v01_00-EN.pdf?fileId=5546d46266a498f50166a531f6aa0013" H 6150 2525 50  0001 C CNN
+F 4 "448-IAUC70N08S5N074ATMA1CT-ND" H 6150 2525 50  0001 C CNN "Digikey"
+	1    6150 2525
+	1    0    0    -1
+$EndComp
+Wire Wire Line
+	5325 1575 5325 1425
+Wire Wire Line
+	5325 1425 6250 1425
+Wire Wire Line
+	6250 1425 6250 1575
+Wire Wire Line
+	5325 1975 5325 2075
+Wire Wire Line
+	6250 2325 6250 2200
+Connection ~ 5325 2075
+Wire Wire Line
+	5325 2075 5325 2325
+Connection ~ 6250 2200
+Wire Wire Line
+	6250 2200 6250 1975
+Wire Wire Line
+	5325 2725 5325 2925
+Wire Wire Line
+	6250 2725 6250 2925
+Wire Wire Line
+	6250 2925 5325 2925
+$Comp
+L power:GND #PWR?
+U 1 1 5F98D578
+P 3500 3100
+F 0 "#PWR?" H 3500 2850 50  0001 C CNN
+F 1 "GND" H 3505 2927 50  0000 C CNN
+F 2 "" H 3500 3100 50  0001 C CNN
+F 3 "" H 3500 3100 50  0001 C CNN
+	1    3500 3100
+	1    0    0    -1
+$EndComp
+Wire Wire Line
+	3500 3100 3500 2925
+Connection ~ 3500 2925
+Wire Wire Line
+	3500 2925 3325 2925
+Wire Wire Line
+	7000 2200 7000 2925
+Wire Wire Line
+	7000 2925 7550 2925
+Wire Wire Line
+	6250 2200 7000 2200
+Wire Wire Line
+	7000 2075 7000 1425
+Wire Wire Line
+	7000 1425 7550 1425
+Wire Wire Line
+	5325 2075 7000 2075
+Text Notes 7525 1275 0    118  Italic 24
+Coil+
+Text Notes 7550 2825 0    118  Italic 24
+Coil-
+Text Notes 2800 1275 0    118  Italic 24
+VIN+
+Text Notes 2825 2825 0    118  Italic 24
+VIN-
+Wire Wire Line
+	5025 1775 4750 1775
+Text Label 4750 1775 0    50   ~ 0
+GATE1
+Wire Wire Line
+	5025 2525 4750 2525
+Text Label 4750 2525 0    50   ~ 0
+GATE3
+Wire Wire Line
+	5950 2525 5675 2525
+Text Label 5675 2525 0    50   ~ 0
+GATE4
+Wire Wire Line
+	5950 1775 5675 1775
+Text Label 5675 1775 0    50   ~ 0
+GATE2
+$Comp
+L power:+24V #PWR?
+U 1 1 5F9917BD
+P 3500 1300
+F 0 "#PWR?" H 3500 1150 50  0001 C CNN
+F 1 "+24V" H 3515 1473 50  0000 C CNN
+F 2 "" H 3500 1300 50  0001 C CNN
+F 3 "" H 3500 1300 50  0001 C CNN
+	1    3500 1300
+	1    0    0    -1
+$EndComp
+Connection ~ 3500 1425
+Wire Wire Line
+	3500 1425 3325 1425
+Wire Wire Line
+	3500 1425 3500 1300
+Wire Wire Line
+	3500 2925 5325 2925
+Connection ~ 5325 2925
+Wire Wire Line
+	3500 1425 5325 1425
+Connection ~ 5325 1425
 $EndSCHEMATC

Commit message: TX Schematic
- Finished up TX schematic.
Parts:
- added C1, C14, C15, C16, C19, C20, C3, C4, C7, C9, C? (x5): 0.1u, Capacitor_SMD:C_0603_1608Metric, symbol Device:C_Small
- added C10, C11, C12, C13: 100n, Capacitors_SMD:C_2220, symbol Device:C_Small
- added C17, C18, C2, C5, C6: 22p, Capacitor_SMD:C_0603_1608Metric, symbol Device:C_Small
- added C8: 10u, Capacitor_SMD:C_0603_1608Metric, symbol Device:C_Small
- added C? (x3): 10u, Capacitors_SMD:C_1206, symbol Device:C_Small
- added C? (x2): 33n, Capacitors_SMD:C_0805, symbol Device:C_Small
- added C? (x2): 0.47u, Capacitors_SMD:C_0805, symbol Device:C_Small
- added D1: Orange, LED_SMD:LED_0805_2012Metric, symbol Device:LED
- added D2: GREEN, LED_SMD:LED_0805_2012Metric, symbol Device:LED
- added D?: ORANGE, LED_SMD:LED_0805_2012Metric, symbol Device:LED
- added D? (x2): BLUE, LED_SMD:LED_0805_2012Metric, symbol Device:LED
- added D?: RED, LED_SMD:LED_0805_2012Metric, symbol Device:LED
- added D? (x2): D_Schottky, Diodes_SMD:D_SMA, symbol Device:D_Schottky
- added FB1: FB, Inductor_SMD:L_0805_2012Metric, symbol Device:Ferrite_Bead_Small
- added J5: Conn_02x05_Odd_Even, Pin_Headers:Pin_Header_Straight_2x05_Pitch1.27mm, symbol Connector_Generic:Conn_02x05_Odd_Even
- added J6: Conn_01x03, symbol Connector_Generic:Conn_01x03
- added J7: Conn_01x04, symbol Connector_Generic:Conn_01x02
- added NT1, NT2: Net-Tie_2, WPT_TX:NetTie-2_SMD_Pad0.25mm, symbol Device:Net-Tie_2
- added R1: 0.005, WPT_TX:R_2512_Sense, symbol Device:R_US
- added R10, R4, R6, R7, R? (x6): 10k, Resistor_SMD:R_0603_1608Metric, symbol Device:R_US
- added R11: 120, Resistor_SMD:R_0603_1608Metric, symbol Device:R_US
- added R2, R?: 2k, Resistor_SMD:R_0603_1608Metric, symbol Device:R_US
- added R3, R5: 80k, Resistor_SMD:R_0603_1608Metric, symbol Device:R_US
- added R8: 330, Resistor_SMD:R_0603_1608Metric, symbol Device:R_US
- added R9, R? (x5): 1k, Resistor_SMD:R_0603_1608Metric, symbol Device:R_US
- added R? (x2): 680, Resistor_SMD:R_0603_1608Metric, symbol Device:R_US
- added TP? (x10): TestPoint, symbol Connector:TestPoint
- added U2: LMC6032, Housings_SOIC:SOIC-8_3.9x4.9mm_Pitch1.27mm, symbol Amplifier_Operational:LMC6082
- added U?: ATSAMD21G16B-MFT, digikey-footprints:TQFP-48_7x7mm, symbol WPT_TX:ATSAMD21G16B-MFT
- added U?: MCP2515-QFN20, Package_SO:TSSOP-20_4.4x6.5mm_P0.65mm, symbol mcp2515-qfn20:MCP2515-QFN20
- added U?: MCP2562-E-MF, Package_DFN_QFN:DFN-8-1EP_3x3mm_P0.65mm_EP1.55x2.4mm, symbol Interface_CAN_LIN:MCP2562-E-MF
- added U?: INA240A1D, Package_SO:SOIC-8_3.9x4.9mm_P1.27mm, symbol Amplifier_Current:INA240A1D
- added U?: BTS6142DAUMA1, Package_TO_SOT_SMD:TO-252-4, symbol chum-bucket:BTS6142DAUMA1
- added U?: LM2937IMP-3.3, TO_SOT_Packages_SMD:SOT-223-3_TabPin2, symbol Regulator_Linear:LM2937xMP
- added U?: LM2936-5.0, TO_SOT_Packages_SMD:SOT-223-3_TabPin2, symbol Regulator_Linear:LM2936-5.0
- added U?: CD4043BDR, Housings_SOIC:SOIC-16_3.9x9.9mm_Pitch1.27mm, symbol CD4043BDR:CD4043BDR
- added U? (x2): LM5106, WPT_TX:LM5106SD, symbol LM5106SD:LM5106SD_NOPB
- added U?: LM2937IMP-12, TO_SOT_Packages_SMD:SOT-223-3_TabPin2, symbol Regulator_Linear:LM2937xMP
- added U?: SN74LVC1G14DBV, TO_SOT_Packages_SMD:SOT-23-5, symbol 74xGxx:SN74LVC1G14DBV
- added Y1: 32.7680kHz, WPT_TX:Crystal_SMD_3215-2pin_3.2x1.5mm, symbol Device:Crystal
- added Y2: 8MHz, WPT_TX:OSCCC320X250, symbol Device:Crystal_GND2_Small
- gave numbers to parts that had none: 8
Connections:
- net labels added: +12V, +3V3, +5V, 3V3_Filt, CANH, CANL, FAULT_OL, FAULT_OL_MCU, FAULT_OL_SR, HBridge_EN, HBridge_PWM, HD, HS_1, HS_2, ISEN, I_IN+, I_IN-, SPI0_CS, SPI0_MOSI, SPI0_SCLK, SWCLK, SWDIO, UART_RX, UART_TX, ~HBridge_PWM~, ~RST~
- wire segments 26 -> 415
- no-connect marks 0 -> 22
Other:
- note added: "A4"
- note added: "A5"
- note added: "CAN TX/RX"
- note added: "CAN and UART"
- note added: "Cannot reset fault if tripped,\nneed to power cycle to clear"
- note added: "Current Sense"
- note added: "D4"
- note added: "D5"
- note added: "H-Bridge"
- note added: "H-Bridge drivers"
- note added: "Logic Inverter"
- note added: "MCU"
- note added: "Open Load fault detection"
- note added: "Programming Header"
- note added: "Voltage Regulators"
- note added: "\nSR Latch"
- note added: "caps for resonance"

Commit message: TX BOM / Footprints
- Added all BOM and footprint selections to components.
- Imported netlist into pcb file.
- Also 3D models!!
Parts:
- removed R? (x2): 1k, Resistor_SMD:R_0603_1608Metric, symbol Device:R_US
- removed TP? (x9): TestPoint, symbol Connector:TestPoint
- added C33: 0.1u, Capacitor_SMD:C_0603_1608Metric, symbol WPT_TX-rescue:C_Small-Device
- added D9: GREEN, LED_SMD:LED_0805_2012Metric, symbol WPT_TX-rescue:LED-Device
- added J3, J4, J5: Conn_Coaxial, WPT_TX:SMA_Amphenol_901-144_Vertical, symbol WPT_TX-rescue:Conn_Coaxial-Connector
- added R19: 680, Resistor_SMD:R_0603_1608Metric, symbol WPT_TX-rescue:R_US-Device
- added R22, R26: 10k, Resistor_SMD:R_0603_1608Metric, symbol WPT_TX-rescue:R_US-Device
- added TP10, TP11, TP12, TP13, TP2, TP3, TP4, TP5, TP6, TP7, TP8, TP9: TestPoint, Testpoints:TestPoint_Loop_D1.80mm_Drill1.0mm_Beaded, symbol WPT_TX-rescue:TestPoint-Connector
- C1, C11, C16, C2, C3: renamed from C?; symbol Device:C_Small -> WPT_TX-rescue:C_Small-Device
- C10: renamed from C2; symbol Device:C_Small -> WPT_TX-rescue:C_Small-Device; Digikey (none) -> 720-VJ0603A220JXBACCT-ND
- C12: renamed from C5; symbol Device:C_Small -> WPT_TX-rescue:C_Small-Device; Digikey (none) -> 720-VJ0603A220JXBACCT-ND
- C13: renamed from C6; symbol Device:C_Small -> WPT_TX-rescue:C_Small-Device; Digikey (none) -> 720-VJ0603A220JXBACCT-ND
- C14: renamed from C7; symbol Device:C_Small -> WPT_TX-rescue:C_Small-Device
- C15: renamed from C8; symbol Device:C_Small -> WPT_TX-rescue:C_Small-Device
- C17: renamed from C9; symbol Device:C_Small -> WPT_TX-rescue:C_Small-Device
- C18: renamed from C14; symbol Device:C_Small -> WPT_TX-rescue:C_Small-Device
- C19: renamed from C15; symbol Device:C_Small -> WPT_TX-rescue:C_Small-Device
- C20: renamed from C16; symbol Device:C_Small -> WPT_TX-rescue:C_Small-Device
- C21, C24, C30, C32: renamed from C?; footprint Capacitors_SMD:C_0805 -> Capacitor_SMD:C_0805_2012Metric; symbol Device:C_Small -> WPT_TX-rescue:C_Small-Device
- C22: renamed from C17; symbol Device:C_Small -> WPT_TX-rescue:C_Small-Device; Digikey (none) -> 720-VJ0603A220JXBACCT-ND
- C23: renamed from C18; symbol Device:C_Small -> WPT_TX-rescue:C_Small-Device; Digikey (none) -> 720-VJ0603A220JXBACCT-ND
- C25: renamed from C19; symbol Device:C_Small -> WPT_TX-rescue:C_Small-Device
- C26: renamed from C10; footprint Capacitors_SMD:C_2220 -> Capacitor_SMD:C_2220_5650Metric; symbol Device:C_Small -> WPT_TX-rescue:C_Small-Device
- C27: renamed from C11; footprint Capacitors_SMD:C_2220 -> Capacitor_SMD:C_2220_5650Metric; symbol Device:C_Small -> WPT_TX-rescue:C_Small-Device
- C28: renamed from C12; footprint Capacitors_SMD:C_2220 -> Capacitor_SMD:C_2220_5650Metric; symbol Device:C_Small -> WPT_TX-rescue:C_Small-Device
- C29: renamed from C13; footprint Capacitors_SMD:C_2220 -> Capacitor_SMD:C_2220_5650Metric; symbol Device:C_Small -> WPT_TX-rescue:C_Small-Device
- C31: renamed from C20; symbol Device:C_Small -> WPT_TX-rescue:C_Small-Device
- C4: renamed from C1; symbol Device:C_Small -> WPT_TX-rescue:C_Small-Device
- C5: renamed from C4; symbol Device:C_Small -> WPT_TX-rescue:C_Small-Device
- C6, C7, C8: renamed from C?; footprint Capacitors_SMD:C_1206 -> Capacitor_SMD:C_1206_3216Metric; symbol Device:C_Small -> WPT_TX-rescue:C_Small-Device
- C9: renamed from C3; symbol Device:C_Small -> WPT_TX-rescue:C_Small-Device
- D1: renamed from D2; symbol Device:LED -> WPT_TX-rescue:LED-Device; Digikey (none) -> 160-1423-1-ND
- D2: renamed from D?; symbol Device:LED -> WPT_TX-rescue:LED-Device; Digikey (none) -> 160-1413-1-ND
- D3, D4: renamed from D?; symbol Device:LED -> WPT_TX-rescue:LED-Device; Digikey (none) -> 160-1579-1-ND
- D5: renamed from D?; symbol Device:LED -> WPT_TX-rescue:LED-Device; Digikey (none) -> 475-1415-1-ND
- D6: renamed from D1; symbol Device:LED -> WPT_TX-rescue:LED-Device
- D7, D8: renamed from D?; symbol Device:D_Schottky -> WPT_TX-rescue:D_Schottky-Device
- FB1: symbol Device:Ferrite_Bead_Small -> WPT_TX-rescue:Ferrite_Bead_Small-Device
- J1, J2: footprint (none) -> WPT_TX:SolderWirePad_single_SMD_5x10mm; symbol Connector_Generic:Conn_01x01 -> WPT_TX-rescue:Conn_01x01-Connector_Generic
- J10: renamed from J4; footprint (none) -> WPT_TX:SolderWirePad_single_SMD_5x10mm; symbol Connector_Generic:Conn_01x01 -> WPT_TX-rescue:Conn_01x01-Connector_Generic
- J6: renamed from J5; footprint Pin_Headers:Pin_Header_Straight_2x05_Pitch1.27mm -> Connector_PinHeader_1.27mm:PinHeader_2x05_P1.27mm_Vertical; symbol Connector_Generic:Conn_02x05_Odd_Even -> WPT_TX-rescue:Conn_02x05_Odd_Even-Connector_Generic
- J7: renamed from J6; footprint (none) -> WPT_TX:70553-03; symbol Connector_Generic:Conn_01x03 -> WPT_TX-rescue:Conn_01x03-Connector_Generic; Digikey (none) -> WM4154-ND
- J8: renamed from J7; footprint (none) -> WPT_TX:70553-02; symbol Connector_Generic:Conn_01x02 -> WPT_TX-rescue:Conn_01x02-Connector_Generic; Digikey (none) -> WM4900-ND
- J9: renamed from J3; footprint (none) -> WPT_TX:SolderWirePad_single_SMD_5x10mm; symbol Connector_Generic:Conn_01x01 -> WPT_TX-rescue:Conn_01x01-Connector_Generic
- NT1, NT2: symbol Device:Net-Tie_2 -> WPT_TX-rescue:Net-Tie_2-Device
- Q1, Q2, Q3, Q4: symbol Device:Q_NMOS_SGD -> WPT_TX-rescue:Q_NMOS_SGD-Device
- R1: renamed from R2; symbol Device:R_US -> WPT_TX-rescue:R_US-Device; Digikey (none) -> 541-2790-1-ND
- R10, R11, R12, R13, R21, R24: renamed from R?; symbol Device:R_US -> WPT_TX-rescue:R_US-Device
- R14, R16, R9: renamed from R?; symbol Device:R_US -> WPT_TX-rescue:R_US-Device; Digikey (none) -> RHM1.0KDCT-ND
- R15: renamed from R?; symbol Device:R_US -> WPT_TX-rescue:R_US-Device; Digikey (none) -> 541-2790-1-ND
- R17, R6: renamed from R?; symbol Device:R_US -> WPT_TX-rescue:R_US-Device; Digikey (none) -> RHM680DCT-ND
- R18: renamed from R7; symbol Device:R_US -> WPT_TX-rescue:R_US-Device
- R2: renamed from R3; value 80k -> 79.6k; symbol Device:R_US -> WPT_TX-rescue:R_US-Device; Digikey (none) -> 13-RT0603BRD0779K6LCT-ND
- R20: renamed from R9; symbol Device:R_US -> WPT_TX-rescue:R_US-Device; Digikey (none) -> RHM1.0KDCT-ND
- R23: renamed from R10; symbol Device:R_US -> WPT_TX-rescue:R_US-Device
- R25: renamed from R11; symbol Device:R_US -> WPT_TX-rescue:R_US-Device
- R3: renamed from R4; symbol Device:R_US -> WPT_TX-rescue:R_US-Device
- R4: renamed from R8; symbol Device:R_US -> WPT_TX-rescue:R_US-Device; Digikey (none) -> RHM330DCT-ND
- R5: value 80k -> 79.6k; symbol Device:R_US -> WPT_TX-rescue:R_US-Device; Digikey (none) -> 13-RT0603BRD0779K6LCT-ND
- R7: renamed from R6; symbol Device:R_US -> WPT_TX-rescue:R_US-Device
- R8: renamed from R1; symbol Device:R_US -> WPT_TX-rescue:R_US-Device
- TP1: renamed from TP?; footprint (none) -> Testpoints:TestPoint_Loop_D1.80mm_Drill1.0mm_Beaded; symbol Connector:TestPoint -> WPT_TX-rescue:TestPoint-Connector; Digikey (none) -> 36-5000-ND
- U1: renamed from U?; symbol Amplifier_Current:INA240A1D -> WPT_TX-rescue:INA240A1D-Amplifier_Current
- U11: renamed from U?; footprint Package_SO:TSSOP-20_4.4x6.5mm_P0.65mm -> Package_DFN_QFN:QFN-20-1EP_4x4mm_P0.5mm_EP2.5x2.5mm_ThermalVias; Digikey (none) -> MCP2515-E/ML-ND
- U12: renamed from U?; symbol Interface_CAN_LIN:MCP2562-E-MF -> WPT_TX-rescue:MCP2562-E-MF-Interface_CAN_LIN
- U2, U4: renamed from U?; footprint TO_SOT_Packages_SMD:SOT-223-3_TabPin2 -> Package_TO_SOT_SMD:SOT-223-3_TabPin2; symbol Regulator_Linear:LM2937xMP -> WPT_TX-rescue:LM2937xMP-Regulator_Linear
- U3: renamed from U?; footprint TO_SOT_Packages_SMD:SOT-223-3_TabPin2 -> Package_TO_SOT_SMD:SOT-223-3_TabPin2; symbol Regulator_Linear:LM2936-5.0 -> WPT_TX-rescue:LM2936-5.0-Regulator_Linear
- U5: renamed from U2; footprint Housings_SOIC:SOIC-8_3.9x4.9mm_Pitch1.27mm -> Package_SO:SOIC-8_3.9x4.9mm_P1.27mm; symbol Amplifier_Operational:LMC6082 -> WPT_TX-rescue:LMC6082-Amplifier_Operational
- U6: renamed from U?; footprint Housings_SOIC:SOIC-16_3.9x9.9mm_Pitch1.27mm -> Package_SO:SOIC-16_3.9x9.9mm_P1.27mm
- U8: renamed from U?; footprint TO_SOT_Packages_SMD:SOT-23-5 -> Package_TO_SOT_SMD:TSOT-23-5; symbol 74xGxx:SN74LVC1G14DBV -> WPT_TX-rescue:SN74LVC1G14DBV-74xGxx
- U9: renamed from U?; footprint digikey-footprints:TQFP-48_7x7mm -> Package_DFN_QFN:QFN-48-1EP_7x7mm_P0.5mm_EP5.6x5.6mm
- Y1: symbol Device:Crystal -> WPT_TX-rescue:Crystal-Device; Digikey 887-2605-1-ND -> ‎XC1656CT-ND‎
- Y2: symbol Device:Crystal_GND2_Small -> WPT_TX-rescue:Crystal_GND2_Small-Device
- gave numbers to parts that had none: 3
Connections:
- wire segments 415 -> 438
- no-connect marks 22 -> 44
Other:
- note added: "LED Indicators"
