File: Mitchell/AUV_Pi_Expansion/AUV_Pi_Expansion.kicad_pcb (KiCad board)
At the start: 2 copper layers, 100 x 55 mm, 50 parts, among them J1 40HAT, J2 CONN_02X02, J3 CONN_01X02, Q1 DMG2305UX, Q2 DMMT5401

Commit message: Pi4 Remake Done
Parts:
- removed Logo12: Trident, silk:trident
- removed Logo13: Starfish, silk:starfish
- removed Logo15: Dhelmet, silk:diverhel
- removed Logo17: Anchor, silk:anchor
- removed Logo2: luckyvolt1, silk:luckyvolt_small_10mm
- removed Logo3: luckyvolt2, silk:luckyvolt_small_15mm
- removed Logo4: luckyvolt3, silk:luckyvolt_small_20mm
- removed Logo5: luckyvolt4, silk:luckyvolt_small_31mm
- removed R7: 1k, Resistor_SMD:R_0603_1608Metric
- removed RN1: 10k, Resistor_SMD:R_Array_Convex_4x0603
- removed TP8: GND, TestPoint:TestPoint_Pad_D1.0mm
- added C10: 10u, Capacitor_SMD:C_1206_3216Metric, F.Cu at (93.2, 122.2)
- added C11: 1u, Capacitor_SMD:C_0603_1608Metric, F.Cu at (95.6, 121.4)
- added C13: 0.1u, Capacitor_SMD:C_0603_1608Metric, B.Cu at (60.9, 93.6)
- added C14: 1u, Capacitor_SMD:C_0603_1608Metric, B.Cu at (146.0, 103.4)
- added C15: 6.8n, Capacitor_SMD:C_0603_1608Metric, B.Cu at (70.4, 103.3)
- added C16: 120n, Capacitor_SMD:C_0603_1608Metric, B.Cu at (73.7, 103.3)
- added C17: 0.1u, Capacitor_SMD:C_0603_1608Metric, B.Cu at (75.2, 108.3)
- added C18: 22p, Capacitor_SMD:C_0603_1608Metric, F.Cu at (67.5, 104.8)
- added C19: 22p, Capacitor_SMD:C_0603_1608Metric, F.Cu at (75.1, 104.8)
- added C20: 0.1u, Capacitor_SMD:C_0603_1608Metric, B.Cu at (71.8, 111.4)
- added C21: 0.1u, Capacitor_SMD:C_0603_1608Metric, F.Cu at (89.7, 116.6)
- added C22: 0.1u, Capacitor_SMD:C_0603_1608Metric, F.Cu at (106.9, 115.9)
- added C23: 22p, Capacitor_SMD:C_0603_1608Metric, B.Cu at (109.1, 121.3)
- added C24: 22p, Capacitor_SMD:C_0603_1608Metric, B.Cu at (109.1, 125.3)
- added C25: 1u, Capacitor_SMD:C_0603_1608Metric, F.Cu at (89.0, 113.8)
- added C26: 0.1u, Capacitor_SMD:C_0603_1608Metric, F.Cu at (89.0, 112.2)
- added C28: 0.1u, Capacitor_SMD:C_0603_1608Metric, F.Cu at (98.7, 108.3)
- added C29: 0.1u, Capacitor_SMD:C_0603_1608Metric, F.Cu at (104.0, 107.6)
- added C3: 4.7u, Capacitor_SMD:C_1210_3225Metric, B.Cu at (68.5, 121.2)
- added C4: 4.7u, Capacitor_SMD:C_1210_3225Metric, B.Cu at (68.5, 125.8)
- added C5: 4.7u, Capacitor_SMD:C_1210_3225Metric, B.Cu at (68.5, 130.7)
- added C6: 100u, Capacitor_SMD:CP_Elec_8x10, F.Cu at (68.8, 113.5)
- added C7: 4.7u, Capacitor_SMD:C_1210_3225Metric, B.Cu at (73.8, 118.5)
- added C8: 10u, Capacitor_SMD:C_1206_3216Metric, F.Cu at (100.3, 122.2)
- added C9: 1u, Capacitor_SMD:C_0603_1608Metric, F.Cu at (97.9, 121.4)
- added D6: WS2812B, LED_SMD:LED_WS2812B_PLCC4_5.0x5.0mm_P3.2mm, F.Cu at (146.0, 103.2)
- added F1: 5A, Fuse:Fuse_1206_3216Metric, F.Cu at (61.7, 107.8)
- added F2: 1A, Fuse:Fuse_1206_3216Metric, B.Cu at (104.1, 92.7)
- added F3: 5A, Fuse:Fuse_1206_3216Metric, B.Cu at (63.3, 127.4)
- added F4: 1A, Fuse:Fuse_1206_3216Metric, B.Cu at (61.7, 106.3)
- added F5: 5A, Fuse:Fuse_1206_3216Metric, F.Cu at (119.8, 121.7)
- added J10: ESC3C, Connector_JST:JST_SH_BM02B-SRSS-TB_1x02-1MP_P1.00mm_Vertical, F.Cu at (105.2, 129.7)
- added J11: ESC2C, Connector_JST:JST_SH_BM02B-SRSS-TB_1x02-1MP_P1.00mm_Vertical, F.Cu at (98.9, 129.7)
- added J12: ESC1C, Connector_JST:JST_SH_BM02B-SRSS-TB_1x02-1MP_P1.00mm_Vertical, F.Cu at (92.5, 129.7)
- added J13: PWR-, µ104KiCAD_connectors:WtB_Solder_Pad_0.7x0.5, B.Cu at (55.3, 135.8)
- added J14: ESC6P, µ104KiCAD_connectors:XT30PW-M, F.Cu at (136.8, 135.8)
- added J15: ESC5P, µ104KiCAD_connectors:XT30PW-M, F.Cu at (123.1, 135.8)
- added J16: PWR-, µ104KiCAD_connectors:WtB_Solder_Pad_0.7x0.5, B.Cu at (55.5, 119.7)
- added J17: ESC4P, µ104KiCAD_connectors:XT30PW-M, F.Cu at (109.3, 135.8)
- added J18: ESC6C, Connector_JST:JST_SH_BM02B-SRSS-TB_1x02-1MP_P1.00mm_Vertical, F.Cu at (124.3, 129.7)
- added J19: ESC5C, Connector_JST:JST_SH_BM02B-SRSS-TB_1x02-1MP_P1.00mm_Vertical, F.Cu at (117.9, 129.7)
- added J20: ESC4C, Connector_JST:JST_SH_BM02B-SRSS-TB_1x02-1MP_P1.00mm_Vertical, F.Cu at (111.6, 129.7)
- added J21: N_SWITCH, Connector_JST:JST_SH_SM02B-SRSS-TB_1x02-1MP_P1.00mm_Horizontal, B.Cu at (55.3, 106.1)
- added J23: RGB LED, Connector_JST:JST_SH_SM03B-SRSS-TB_1x03-1MP_P1.00mm_Horizontal, F.Cu at (146.7, 110.3)
- added J24: LEAK1, Connector_JST:JST_SH_SM02B-SRSS-TB_1x02-1MP_P1.00mm_Horizontal, B.Cu at (75.0, 88.1)
- added J25: TOF1, Connector_JST:JST_SH_SM04B-SRSS-TB_1x04-1MP_P1.00mm_Horizontal, F.Cu at (69.0, 88.1)
- added J26: TOF2, Connector_JST:JST_SH_SM04B-SRSS-TB_1x04-1MP_P1.00mm_Horizontal, F.Cu at (77.0, 88.1)
- added J27: BlueRobotics Pressure Sense, Connector_Hirose:Hirose_DF13-04P-1.25DS_1x04_P1.25mm_Horizontal, F.Cu at (59.2, 89.8)
- added J28: TOF3, Connector_JST:JST_SH_SM04B-SRSS-TB_1x04-1MP_P1.00mm_Horizontal, F.Cu at (85.0, 88.1)
- added J29: TOF4, Connector_JST:JST_SH_SM04B-SRSS-TB_1x04-1MP_P1.00mm_Horizontal, F.Cu at (93.0, 88.1)
- added J31: LEAK2, Connector_JST:JST_SH_SM02B-SRSS-TB_1x02-1MP_P1.00mm_Horizontal, B.Cu at (81.0, 88.1)
- added J32: TOF5, Connector_JST:JST_SH_SM04B-SRSS-TB_1x04-1MP_P1.00mm_Horizontal, F.Cu at (101.0, 88.1)
- added J33: CAN, Connector_JST:JST_SH_BM04B-SRSS-TB_1x04-1MP_P1.00mm_Vertical, F.Cu at (108.1, 123.0)
- added J34: GPIO, Connector_JST:JST_SH_SM03B-SRSS-TB_1x03-1MP_P1.00mm_Horizontal, B.Cu at (93.8, 88.1)
- added J35: I2C, Connector_JST:JST_SH_SM03B-SRSS-TB_1x03-1MP_P1.00mm_Horizontal, B.Cu at (68.5, 88.1)
- added J36: Rpi Z 1 - IN, Connector_JST:JST_SH_BM08B-SRSS-TB_1x08-1MP_P1.00mm_Vertical, F.Cu at (111.2, 110.1)
- added J37: Rpi Z 1 - OUT SWITCH, µ104KiCAD_connectors:DS1128-05-S8B8P, F.Cu at (118.0, 102.4)
- added J38: Rpi Z 2 - OUT SWITCH, µ104KiCAD_connectors:DS1128-05-S8B8P, F.Cu at (135.3, 102.4)
- added J39: Rpi Z 3 - OUT SWITCH, µ104KiCAD_connectors:DS1128-05-S8B8P, F.Cu at (132.4, 126.7)
- added J4: PWR-, µ104KiCAD_connectors:WtB_Solder_Pad_7x3.5, F.Cu at (55.7, 111.0)
- added J42: Rpi Z 2 - IN, Connector_JST:JST_SH_BM08B-SRSS-TB_1x08-1MP_P1.00mm_Vertical, F.Cu at (128.5, 110.1)
- added J43: Rpi Z 3 - IN, Connector_JST:JST_SH_BM08B-SRSS-TB_1x08-1MP_P1.00mm_Vertical, F.Cu at (124.4, 120.0)
- added J5: PWR+, µ104KiCAD_connectors:WtB_Solder_Pad_0.7x0.5, B.Cu at (55.5, 126.0)
- added J6: ESC3P, µ104KiCAD_connectors:XT30PW-M, F.Cu at (95.6, 135.8)
- added J7: ESC2P, µ104KiCAD_connectors:XT30PW-M, F.Cu at (81.8, 135.8)
- added J8: ESC1P, µ104KiCAD_connectors:XT30PW-M, F.Cu at (68.1, 135.7)
- added J9: PWR+, µ104KiCAD_connectors:WtB_Solder_Pad_0.7x0.5, F.Cu at (55.3, 135.8)
- added JP3: C120, Jumper:SolderJumper-2_P1.3mm_Open_RoundedPad1.0x1.5mm, B.Cu at (115.5, 116.4)
- added Logo18: Cod, silk:cod, B.Cu at (88.1, 126.9)
- added Q3: MMBT3904, Package_TO_SOT_SMD:SOT-23, B.Cu at (75.8, 93.4)
- added Q4: MMBT3904, Package_TO_SOT_SMD:SOT-23, B.Cu at (87.5, 93.2)
- added R12: 100k, Resistor_SMD:R_0603_1608Metric, B.Cu at (65.5, 113.0)
- added R13: 470, Resistor_SMD:R_0603_1608Metric, B.Cu at (146.0, 101.5)
- added R14: 10k, Resistor_SMD:R_0603_1608Metric, B.Cu at (65.5, 106.7)
- added R15: 10k, Resistor_SMD:R_0603_1608Metric, F.Cu at (75.2, 108.2)
- added R16: 10k, Resistor_SMD:R_0603_1608Metric, B.Cu at (68.4, 111.4)
- added R17: 1k, Resistor_SMD:R_0603_1608Metric, B.Cu at (72.1, 93.5)
- added R18: 1k, Resistor_SMD:R_0603_1608Metric, B.Cu at (72.1, 91.9)
- added R19: 100k, Resistor_SMD:R_0603_1608Metric, B.Cu at (72.1, 95.1)
- added R20: 1k, Resistor_SMD:R_0603_1608Metric, B.Cu at (83.9, 91.3)
- added R21: 1k, Resistor_SMD:R_0603_1608Metric, B.Cu at (83.9, 92.9)
- added R22: 100k, Resistor_SMD:R_0603_1608Metric, B.Cu at (83.9, 94.6)
- added R23: 120, Resistor_SMD:R_0603_1608Metric, B.Cu at (117.9, 116.4)
- added R24: 0, Resistor_SMD:R_0603_1608Metric, B.Cu at (104.2, 116.9)
- added R25: 0, Resistor_SMD:R_0603_1608Metric, B.Cu at (104.2, 114.7)
- added R26: 1k, Resistor_SMD:R_0603_1608Metric, F.Cu at (111.1, 118.6)
- added R27: 10k, Resistor_SMD:R_0603_1608Metric, F.Cu at (87.7, 116.5)
- added R28: 3.9k, Resistor_SMD:R_0603_1608Metric, F.Cu at (80.4, 108.5)
- added R29: 3.9k, Resistor_SMD:R_0603_1608Metric, F.Cu at (80.4, 110.3)
- added R30: 3.9k, Resistor_SMD:R_0603_1608Metric, F.Cu at (80.4, 105.0)
- added R31: 3.9k, Resistor_SMD:R_0603_1608Metric, F.Cu at (80.4, 106.8)
- added R32: 3.9k, Resistor_SMD:R_0603_1608Metric, B.Cu at (80.5, 109.4)
- added R33: 3.9k, Resistor_SMD:R_0603_1608Metric, B.Cu at (80.5, 111.2)
- added R34: 3.9k, Resistor_SMD:R_0603_1608Metric, B.Cu at (80.5, 105.8)
- added R35: 3.9k, Resistor_SMD:R_0603_1608Metric, B.Cu at (80.5, 107.6)
- added R36: 3.9k, Resistor_SMD:R_0603_1608Metric, B.Cu at (94.0, 107.6)
- added R37: 3.9k, Resistor_SMD:R_0603_1608Metric, B.Cu at (94.0, 106.0)
- added R38: 3.9k, Resistor_SMD:R_0603_1608Metric, B.Cu at (94.0, 110.8)
- added R39: 3.9k, Resistor_SMD:R_0603_1608Metric, B.Cu at (94.0, 109.2)
- added R40: 3.9k, Resistor_SMD:R_0603_1608Metric, F.Cu at (93.5, 105.9)
- added R41: 3.9k, Resistor_SMD:R_0603_1608Metric, F.Cu at (93.5, 104.3)
- added R42: 3.9k, Resistor_SMD:R_0603_1608Metric, F.Cu at (93.5, 109.1)
- added R43: 3.9k, Resistor_SMD:R_0603_1608Metric, F.Cu at (93.5, 107.5)
- added R44: 10k, Resistor_SMD:R_0603_1608Metric, F.Cu at (98.7, 104.4)
- added RV1: R_POT, Potentiometer_THT:Potentiometer_Bourns_3296W_Vertical, F.Cu at (78.6, 114.6)
- added U1: AZ1117-3.3, Package_TO_SOT_SMD:SOT-223-3_TabPin2, F.Cu at (95.6, 114.5)
- added U10: TXS0108EPW, Package_SO:TSSOP-20_4.4x6.5mm_P0.65mm, B.Cu at (101.2, 107.0)
- added U2: SRBH-06H1A1G, µ104KiCAD_DCDC:SRBH-06H1A1G, F.Cu at (77.1, 125.4)
- added U5: BME280, µ104KiCAD_IC:BME280_Mod_Bosch_LGA-8_2.5x2.5mm_P0.65mm_ClockwisePinNumbering, B.Cu at (58.1, 93.7)
- added U6: BNO055, µ104KiCAD_IC:BNO055_MOD_LGA-28_5.2x3.8mm_P0.5mm, B.Cu at (70.3, 107.3)
- added U7: SN65HVD230, Package_SO:SOIC-8_3.9x4.9mm_P1.27mm, B.Cu at (110.2, 116.5)
- added U8: MCP2515-xSO, Package_SO:SOIC-18W_7.5x11.6mm_P1.27mm, B.Cu at (96.6, 119.9)
- added U9: TCA9548APWR, Package_SO:TSSOP-24_4.4x7.8mm_P0.65mm, B.Cu at (87.2, 108.7)
- added Y1: 32.768kHz, Crystal:Crystal_SMD_3215-2Pin_3.2x1.5mm, F.Cu at (71.3, 104.8)
- added Y2: 8MHz, Crystal:Crystal_SMD_5032-2Pin_5.0x3.2mm, B.Cu at (105.3, 123.2)
- C1: value 0.1u -> 100u; footprint Capacitor_SMD:C_0603_1608Metric -> Capacitor_SMD:CP_Elec_8x10
- C2: value 1u -> 100u; footprint Capacitor_SMD:C_0603_1608Metric -> Capacitor_SMD:CP_Elec_8x10
- D5: value USB -> 26.7 Vb; footprint LED_SMD:LED_0603_1608Metric -> Diode_SMD:D_SMB; moved to B.Cu
- J1, JP1, Logo10, Logo14, Logo16, Logo7, Logo9: moved to B.Cu
- J2: value CONN_02X02 -> FAN; footprint Connector_PinHeader_2.54mm:PinHeader_2x02_P2.54mm_Vertical -> Connector_PinHeader_2.54mm:PinHeader_1x02_P2.54mm_Vertical
- J3: value CONN_01X02 -> PWR+; footprint Connector_PinHeader_2.54mm:PinHeader_1x02_P2.54mm_Vertical -> µ104KiCAD_connectors:WtB_Solder_Pad_7x3.5
- Q1: value DMG2305UX -> Q_NMOS_GDS; footprint Package_TO_SOT_SMD:SOT-23 -> Package_TO_SOT_SMD:TO-252-2; moved to B.Cu
- Q2: value DMMT5401 -> MMBT3904; footprint Package_TO_SOT_SMD:SOT-23-6 -> Package_TO_SOT_SMD:SOT-23; moved to B.Cu
- R1: value 4.7k -> 3.9k; moved to B.Cu
- R2: value 10k -> 3.9k; moved to B.Cu
- R3: value 100k -> 100; moved to B.Cu
- R4: value 1M -> 100; moved to B.Cu
- R5: value 0 -> 1k; moved to B.Cu
- R6: value 33 -> 4.7k; moved to B.Cu
- TP4: value USB -> SYS_ON/OFF
- moved Logo16 295.1 mm to (107.2, 141.9), turned to 90 degrees
- moved Logo6 286.0 mm to (65.2, 143.1)
- moved C1 264.1 mm to (56.1, 127.5), turned to 180 degrees
- moved R3 260.6 mm to (51.8, 93.0), turned to 180 degrees
- moved R1 253.3 mm to (67.3, 93.5), turned to 90 degrees
- moved Logo8 249.2 mm to (113.5, 89.0)
- moved C2 246.1 mm to (56.1, 117.9), turned to 180 degrees
- moved D1 245.1 mm to (51.8, 93.0)
- moved Logo9 242.5 mm to (121.4, 89.8), turned to 180 degrees
- moved R2 239.8 mm to (65.2, 93.5), turned to 90 degrees
- moved Logo14 213.3 mm to (143.5, 136.3), turned to 180 degrees
- moved Logo10 201.3 mm to (126.5, 111.6), turned to 90 degrees
- moved Logo7 200.7 mm to (144.5, 119.8), turned to 180 degrees
- moved Q1 199.5 mm to (57.6, 112.7), turned to 180 degrees
- moved J3 191.8 mm to (55.6, 106.4)
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Connections:
- net /ID_SC_EEPROM renamed ID_SC_EEPROM
- net /ID_SD_EEPROM renamed ID_SD_EEPROM\GPIO0
- net Net-(J1-Pad10) renamed /RXD\GPIO15
- net Net-(J1-Pad11) renamed LOAD0
- net Net-(J1-Pad13) renamed LOAD1
- net Net-(J1-Pad26) renamed /~CE1~\GPIO7
- net Net-(J1-Pad35) renamed /MISO1\GPIO19
- net Net-(J1-Pad36) renamed EXT_TEMP
- net Net-(J1-Pad38) renamed /MOSI1\GPIO20
- net Net-(J1-Pad40) renamed /SCLK1\GPIO21
- net Net-(J1-Pad8) renamed /TXD\GPIO14
- C1 pad 1: Net-(C1-Pad1) -> +V
- C1 pad 2: Net-(C1-Pad2) -> GND
- C2 pad 1: Net-(C2-Pad1) -> +V
- C2 pad 2: Net-(C2-Pad2) -> GND
- D1 pad 1: Net-(D1-Pad1) -> GND
- D5 pad 1: GND -> +V
- D5 pad 2: Net-(D5-Pad2) -> CHASSIS
- J1 pad 12: Net-(J1-Pad12) -> LED_USR2
- J1 pad 15: Net-(J1-Pad15) -> LEAK_2
- J1 pad 16: Net-(J1-Pad16) -> BNO_INT
- J1 pad 18: Net-(J1-Pad18) -> BNO_BL_IND
- J1 pad 19: Net-(J1-Pad19) -> MOSI0\GPIO10
- J1 pad 21: Net-(J1-Pad21) -> MISO0\GPIO9
- J1 pad 22: Net-(J1-Pad22) -> BNO_~RST
- J1 pad 23: Net-(J1-Pad23) -> SCLK0\GPIO11
- J1 pad 24: Net-(J1-Pad24) -> ~CE0~\GPIO8
- J1 pad 29: Net-(J1-Pad29) -> GCLK1\GPIO5
- J1 pad 3: Net-(J1-Pad3) -> SDA\GPIO2
- J1 pad 31: Net-(J1-Pad31) -> GCLK2\GPIO6
- J1 pad 32: Net-(J1-Pad32) -> G_DRV_LED
- J1 pad 33: Net-(J1-Pad33) -> PWM1\GPIO12
- J1 pad 37: Net-(J1-Pad37) -> LEAK_1
- J1 pad 5: Net-(J1-Pad5) -> SCL\GPIO3
- J1 pad 7: Net-(J1-Pad7) -> /LED_USR1
- J2 pad 1: /P3V3 -> GND
- J2 pad 2: /P3V3_HAT -> 5V_EXT\POE
- J3 pad 1: GND -> 5V_PI
- Q1 pad 1: Net-(Q1-Pad1) -> G_DRV_LED
- Q1 pad 2: /P5V_HAT -> /Sensors/LED_CTRL
- Q1 pad 3: /P5V -> GND
- Q2 pad 1: Net-(Q2-Pad1) -> +3V3
- Q2 pad 2: Net-(Q2-Pad1) -> LED_USR2
- Q2 pad 3: Net-(Q2-Pad1) -> +5V
- R1 pad 1: Net-(R1-Pad1) -> +3V3
- R1 pad 2: Net-(R1-Pad2) -> SDA\GPIO2
- R2 pad 1: Net-(R2-Pad1) -> +3V3
- R2 pad 2: Net-(R2-Pad2) -> SCL\GPIO3
- R3 pad 1: Net-(R3-Pad1) -> /LED_USR1
- R3 pad 2: Net-(R3-Pad2) -> Net-(D1-Pad2)
- R4 pad 1: Net-(R4-Pad1) -> +3V3
- R4 pad 2: Net-(R4-Pad2) -> Net-(D2-Pad2)
- R5 pad 1: Net-(R5-Pad1) -> +5V
- R5 pad 2: Net-(R5-Pad2) -> Net-(D3-Pad2)
- R6 pad 1: Net-(R6-Pad1) -> +V
- R6 pad 2: Net-(R6-Pad2) -> Net-(D4-Pad2)
- TP4 pad 1: VBUS -> /Power/SYS_ON\OFF
Routing:
- net +3V3: track 0.00 -> 247.8 mm, vias 0 -> 24
- net GND: track 0.00 -> 134.9 mm, vias 0 -> 153
- net +5V: track 0.00 -> 133.9 mm, vias 0 -> 67
- net LED_USR2: track 0.00 -> 84.3 mm, vias 0 -> 3
- net +V: track 0.00 -> 83.2 mm, vias 0 -> 71
- net CANL: track 0.00 -> 75.1 mm, vias 0 -> 3
- net SCL\GPIO3: track 0.00 -> 74.5 mm, vias 0 -> 2
- net 3V3_Sensors: track 0.00 -> 71.5 mm, vias 0 -> 7
- net SDA\GPIO2: track 0.00 -> 68.9 mm
- net CANH: track 0.00 -> 68.3 mm, vias 0 -> 1
- net 5V_EXT\POE: track 0.00 -> 65.5 mm, vias 0 -> 14
- net TCA_SCL5: track 0.00 -> 47.7 mm, vias 0 -> 1
- net G_DRV_LED: track 0.00 -> 46.5 mm, vias 0 -> 5
- net TCA_SDA5: track 0.00 -> 45.7 mm, vias 0 -> 1
- net LEAK_1: track 0.00 -> 44.5 mm
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- added copper zone on VCC.Cu, net +3V3
- added copper zone on B.Cu, net +5V
- added copper zone on F.Cu, net +5V
- added copper zone on VCC.Cu, net +5V
- added copper zone on B.Cu, net +V
- added copper zone on F.Cu, net +V
- added copper zone on VCC.Cu, net +V
- added copper zone on B.Cu, net /Sensors/LED_CTRL
- added copper zone on F.Cu, net 5V_EXT\POE
- added copper zone on VCC.Cu, net 5V_EXT\POE
- added copper zone on F.Cu, net 5V_PI
- added copper zone on B.Cu, net GND
- added copper zone on F.Cu, net GND
- added copper zone on GND.Cu, net GND
- added copper zone on B.Cu, net LED_PWR
Other:
- board size 100 x 55 mm -> 100 x 65.2 mm
- copper layers 2 -> 4
- net class Default: clearance 0.2 -> 0.1524; trace_width 0.25 -> 0.1524; via_dia 0.8 -> 0.6
- net class power1: via_dia 0.8 -> 0.6
- net class signal1: via_dia 0.4 -> 0.45; via_drill 0.3 -> 0.2
- rule pad_to_mask_clearance: 0.0254 -> 0.05
- rule solder_mask_min_width: 0.127 -> 0.2
- rule trace_clearance: 0.2 -> 0.1524
- rule via_min_drill: 0.3 -> 0.2
- rule via_min_size: 0.4 -> 0.45
- board text added: "AUV PI EXPANSION PCB"
- board text added: "AUV PI Expansion PCB PN: 2020-001 V1.0 SN:"
- board text removed: "(c) Lucky Volt AUV PI Expansion PCB PN: 2020-001 V1.0 SN:"
- board text removed: "Lucky Volt AUV PI EXPANSION PCB"
- board text removed: "PCB #: 2020-001 Sch: Mitchell Stride Layout: Mitchell Stride BOM: Mitchell Stride Review: Mitchell Stride, Frank Walsh, Mark Belbin"
