File: Mitchell/AUV_Pi_Expansion/AUV_Pi_Expansion.kicad_pcb (KiCad board)
At the start: 4 copper layers, 100 x 65.2 mm, 154 parts, among them J1 40HAT, J10 ESC3C, J11 ESC2C, J12 ESC1C, J13 PWR-, J14 ESC6P, J15 ESC5P, J16 PWR-, J17 ESC4P, J18 ESC6C, J19 ESC5C, J2 FAN, J20 ESC4C, J21 N_SWITCH, J23 RGB LED, J24 LEAK1, J25 TOF1, J26 TOF2, J27 BlueRobotics Pressure Sense, J28 TOF3, J29 TOF4, J3 PWR+, J31 LEAK2, J32 TOF5, J33 CAN, J34 GPIO, J35 I2C, J36 Rpi Z 1 - IN, J37 Rpi Z 1 - OUT SWITCH, J38 Rpi Z 2 - OUT SWITCH, J39 Rpi Z 3 - OUT SWITCH, J4 PWR-, J42 Rpi Z 2 - IN, J43 Rpi Z 3 - IN, J5 PWR+, J6 ESC3P, J7 ESC2P, J8 ESC1P, J9 PWR+, Q1 Q_NMOS_GDS, Q2 MMBT3904, Q3 MMBT3904, Q4 MMBT3904, U1 AZ1117-3.3, U10 TXS0108EPW, U2 SRBH-06H1A1G, U5 BME280, U6 BNO055, U7 SN65HVD230, U8 MCP2515-xSO, U9 TCA9548APWR, Y1 32.768kHz, Y2 8MHz

Commit message: fixed gerbs on pi board
Connections:
- J37 pad 4: /POE/Pi1_Data_TP_2-2 -> Net-(J37-Pad4)
- J37 pad 6: Net-(J37-Pad6) -> /POE/Pi1_Data_TP_2-2
- J38 pad 4: /POE/Pi2_Data_TP_2-2 -> Net-(J38-Pad4)
- J38 pad 6: Net-(J38-Pad6) -> /POE/Pi2_Data_TP_2-2
- J39 pad 4: /POE/Pi3_Data_TP_2-2 -> Net-(J39-Pad4)
- J39 pad 6: Net-(J39-Pad6) -> /POE/Pi3_Data_TP_2-2
Routing:
- net /POE/Pi2_Data_TP_2-2: track 9.93 -> 8.19 mm, vias 0 -> 1
- net /POE/Pi3_Data_TP_2-2: track 9.92 -> 8.31 mm, vias 0 -> 1
- net /POE/Pi1_Data_TP_2-2: track 8.75 -> 8.94 mm, vias 0 -> 1
