File: Mitchell/AUV_Pi_Expansion/Interface.sch (KiCad schematic (older format))
At the start: 33 parts, among them J33 CAN, U7 SN65HVD230, U8 MCP2515-xSO, U9 TCA9548APWR, Y2 8MHz

Commit message: Pi4 Remake Done
Parts:
- added C28, C29: 0.1u, Capacitor_SMD:C_0603_1608Metric, symbol Device:C_Small
- added R44: 10k, Resistor_SMD:R_0603_1608Metric, symbol Device:R_Small_US
- added U10: TXS0108EPW, Package_SO:TSSOP-20_4.4x6.5mm_P0.65mm, symbol Logic_LevelTranslator:TXS0108EPW
- J33: footprint Connector_JST:JST_SH_SM04B-SRSS-TB_1x04-1MP_P1.00mm_Horizontal -> Connector_JST:JST_SH_BM04B-SRSS-TB_1x04-1MP_P1.00mm_Vertical; LCSC C160404 -> C160390
Connections:
- net +3V3: now also C28.1, R44.1, U10.2 (VCCA); no longer C21.1, C22.1, J33.4 (Pin_4), R27.1, U7.3 (VCC), U8.18 (VDD)
- net GND: now also C28.2, C29.2
- net MISO0\GPIO9: now also U10.3 (A2); no longer U8.15 (SO)
- net MOSI0\GPIO10: now also U10.1 (A1); no longer U8.14 (SI)
- net SCLK0\GPIO11: now also U10.5 (A4); no longer U8.13 (SCK)
- net ~CE0~\GPIO8: now also U10.4 (A3); no longer U8.16 (~CS)
- net GCLK2\GPIO6: no longer names the net of U8.12 (~INT)
- new net: U10.16 (B4), U8.13 (SCK)
- new net: U10.20 (B1), U8.14 (SI)
- new net: U10.18 (B2), U8.15 (SO)
- new net: U10.17 (B3), U8.16 (~CS)
- new net: R44.2, U10.10 (OE)
- new net +5V: C21.1, C22.1, C29.1, J33.4 (Pin_4), R27.1, U10.19 (VCCB), U7.3 (VCC), U8.18 (VDD)
- no-connect marks 7 -> 8
