File: Mitchell/AUV_Pi_Expansion/Power.sch (KiCad schematic (older format))
At the start: 34 parts, among them J13 PWR-, J16 SYS_PWR, J21 N_SWT_PWR, J3 PWR+, J4 PWR-, J40 LOAD0, J41 LOAD1, J5 5V to Pi, J9 PWR+, U1 AZ1117-3.3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

Commit message: Pi4 Remake Done
Parts:
- removed C12: 10u, Capacitor_SMD:C_1206_3216Metric, symbol Device:C_Small
- removed J16: SYS_PWR, Connector_JST:JST_SH_SM02B-SRSS-TB_1x02-1MP_P1.00mm_Horizontal, symbol Connector_Generic:Conn_01x02
- removed J21: N_SWT_PWR, µ104KiCAD_connectors:microUSB_jing_C40943, symbol Connector:USB_B_Micro
- removed J40: LOAD0, µ104KiCAD_connectors:WtB_Solder_Pad_0.7x0.5, symbol Connector_Generic:Conn_01x01
- removed J41: LOAD1, µ104KiCAD_connectors:WtB_Solder_Pad_0.7x0.5, symbol Connector_Generic:Conn_01x01
- removed J5: 5V to Pi, ESP8266:USB-C-16p, symbol Connector:USB_C_Receptacle_USB2.0
- removed R7, R8: 1k, Resistor_SMD:R_0603_1608Metric, symbol Device:R_Small_US
- removed U3: BTS50302, µ104KiCAD_IC:SOIC-14_N-TAB, symbol u104_KICAD_pwrMgmt:BTS50302
- added J21: N_SWITCH, Connector_JST:JST_SH_SM02B-SRSS-TB_1x02-1MP_P1.00mm_Horizontal, symbol Connector_Generic:Conn_01x02
- F1: footprint µ104KiCAD:5x20_fuseholderx2_XuchengElecC3130 -> Fuse:Fuse_1206_3216Metric; Desc Order x2 and C95690 5A -> (none); LCSC C3130 -> C163128
- F2, F4: footprint µ104KiCAD:5x20_fuseholderx2_XuchengElecC3130 -> Fuse:Fuse_1206_3216Metric; LCSC C3130 -> C553921
- F3, F5: value 10A -> 5A; footprint µ104KiCAD:5x20_fuseholderx2_XuchengElecC3130 -> Fuse:Fuse_1206_3216Metric; Desc Order x2 and C142733 10A -> (none); LCSC C3130 -> C163128
- J3, J4: footprint µ104KiCAD_connectors:WtB_Solder_Pad_0.7x0.5 -> µ104KiCAD_connectors:WtB_Solder_Pad_7x3.5
Connections:
- net 5V_Router: now also J21.2 (Pin_2)
- net GND: now also J21.1 (Pin_1)
- no-connect marks 16 -> 2
Other:
- note removed: "*ALT BACKUP for LED POWER or Control\n"
- moved on the sheet: J3, J4
