File: Mitchell/AUV_Pi_Expansion/Sensors.sch (KiCad schematic (older format))
At the start: 43 parts, among them J22 ESC1P, J23 RGB LED, J24 LEAK1, J25 TOF, J26 TOF, J27 BlueRobotics Pressure Sense, J28 TOF, J29 TOF, J30 TEMP, J31 LEAK2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

Commit message: Sch label net changes to global tags
Parts:
- added C27: 0.1u, Capacitor_SMD:C_0603_1608Metric, symbol Device:C_Small
- J22: value ESC1P -> LED
- J27: footprint Connector_Hirose:Hirose_DF13-03P-1.25DS_1x03_P1.25mm_Horizontal -> Connector_Hirose:Hirose_DF13-04P-1.25DS_1x04_P1.25mm_Horizontal
- U4: footprint Package_SOIC:SOIC-8_3.9x4.9mm_P1.27mm -> Package_SO:SOIC-8_3.9x4.9mm_P1.27mm
- U5: footprint Package_LGA:Bosch_LGA-8_2.5x2.5mm_P0.65mm_ClockwisePinNumbering -> µ104KiCAD_IC:BME280_Mod_Bosch_LGA-8_2.5x2.5mm_P0.65mm_ClockwisePinNumbering
- U6: footprint Package_LGA:LGA-28_5.2x3.8mm_P0.5mm -> µ104KiCAD_IC:BNO055_MOD_LGA-28_5.2x3.8mm_P0.5mm
Connections:
- net +3V3: now also C27.1
- net GND: now also C27.2
Changed lines of the file:
@@
 Wire Wire Line
 	5840 1780 5510 1780
-Text Label 5840 1780 2    39   ~ 0
-SCL\GPIO3
-Text Label 5840 1980 2    39   ~ 0
-SDA\GPIO2
 Wire Wire Line
 	5510 1580 5940 1580
 Wire Wire Line
-	5940 1770 5940 1580
+	5940 1595 5940 1580
 Wire Wire Line
 	5950 2180 5510 2180
 Wire Wire Line
-	5950 2130 5950 2180
+	5950 2170 5950 2180
 $Comp
 L power:+3V3 #PWR?
 U 1 1 5FDADB96
-P 5950 2130
+P 5950 2170
 AR Path="/5FDADB96" Ref="#PWR?"  Part="1"
 AR Path="/5F9D87DA/5FDADB96" Ref="#PWR?"  Part="1"
 AR Path="/5FCB4E5B/5FDADB96" Ref="#PWR0149"  Part="1"
-F 0 "#PWR0149" H 5950 1980 50  0001 C CNN
-F 1 "+3V3" H 5930 2260 31  0000 C CNN
-F 2 "" H 5950 2130 50  0001 C CNN
-F 3 "" H 5950 2130 50  0001 C CNN
-	1    5950 2130
+F 0 "#PWR0149" H 5950 2020 50  0001 C CNN
+F 1 "+3V3" H 6030 2265 31  0000 C CNN
+F 2 "" H 5950 2170 50  0001 C CNN
+F 3 "" H 5950 2170 50  0001 C CNN
+	1    5950 2170
 	1    0    0    -1
 $EndComp
@@
 L power:GND #PWR?
 U 1 1 5FDADB9C
-P 5940 1770
+P 5940 1595
 AR Path="/5FDADB9C" Ref="#PWR?"  Part="1"
 AR Path="/5F9D87DA/5FDADB9C" Ref="#PWR?"  Part="1"
 AR Path="/5FCB4E5B/5FDADB9C" Ref="#PWR0150"  Part="1"
-F 0 "#PWR0150" H 5940 1520 50  0001 C CNN
-F 1 "GND" H 5940 1650 31  0000 C CNN
-F 2 "" H 5940 1770 50  0001 C CNN
-F 3 "" H 5940 1770 50  0001 C CNN
-	1    5940 1770
+F 0 "#PWR0150" H 5940 1345 50  0001 C CNN
+F 1 "GND" H 6030 1505 31  0000 C CNN
+F 2 "" H 5940 1595 50  0001 C CNN
+F 3 "" H 5940 1595 50  0001 C CNN
+	1    5940 1595
 	1    0    0    -1
 $EndComp
@@
 F 0 "U5" H 4481 1926 50  0000 R CNN
 F 1 "BME280" H 4481 1835 50  0000 R CNN
-F 2 "Package_LGA:Bosch_LGA-8_2.5x2.5mm_P0.65mm_ClockwisePinNumbering" H 6410 1430 50  0001 C CNN
+F 2 "µ104KiCAD_IC:BME280_Mod_Bosch_LGA-8_2.5x2.5mm_P0.65mm_ClockwisePinNumbering" H 6410 1430 50  0001 C CNN
 F 3 "https://ae-bst.resource.bosch.com/media/_tech/media/datasheets/BST-BME280-DS002.pdf" H 4910 1680 50  0001 C CNN
 F 4 "C92489" H 4910 1880 50  0001 C CNN "LCSC"
@@
 AR Path="/5FCB4E5B/5FDADCE4" Ref="J22"  Part="1"
 F 0 "J22" H 7880 1190 50  0000 C CNN
-F 1 "ESC1P" H 7810 1470 50  0000 C CNN
+F 1 "LED" H 7810 1470 50  0000 C CNN
 F 2 "µ104KiCAD_connectors:XT30PW-M" H 7870 1370 50  0001 C CNN
 F 3 "~" H 7870 1370 50  0001 C CNN
@@
 AR Path="/5FCB4E5B/5FDADD72" Ref="U4"  Part="1"
 F 0 "U4" H 1860 1780 50  0000 C CNN
-F 1 "CAT24C32" H 2450 1100 50  0000 C CNN
-F 2 "Package_SOIC:SOIC-8_3.9x4.9mm_P1.27mm" H 2220 1440 50  0001 C CNN
+F 1 "CAT24C32" H 2450 1100 50  0001 C CNN
+F 2 "Package_SO:SOIC-8_3.9x4.9mm_P1.27mm" H 2220 1440 50  0001 C CNN
 F 3 "" H 2220 1440 50  0000 C CNN
 F 4 "C81193" H 2220 1440 50  0001 C CNN "LCSC"
@@
 	1    0    0    -1
 $EndComp
-Wire Wire Line
-	2220 1010 2220 1040
 Wire Wire Line
 	1360 1240 1610 1240
@@
 F 0 "U6" H 2190 4290 50  0000 C CNN
 F 1 "BNO055" H 2960 2990 50  0000 C CNN
-F 2 "Package_LGA:LGA-28_5.2x3.8mm_P0.5mm" H 2870 2990 50  0001 L CNN
+F 2 "µ104KiCAD_IC:BNO055_MOD_LGA-28_5.2x3.8mm_P0.5mm" H 2870 2990 50  0001 L CNN
 F 3 "https://ae-bst.resource.bosch.com/media/_tech/media/datasheets/BST_BNO055_DS000_14.pdf" H 2620 3840 50  0001 C CNN
 F 4 "C93216" H 2620 3640 50  0001 C CNN "LCSC"
@@
 Text Notes 1700 4370 0    50   ~ 0
 I2C ADDR: 0x29
-Text Label 3170 1640 2    28   ~ 0
-ID_SD_EEPROM\GPIO0
 $Comp
 L Device:R_Small_US R?
@@
 	2720 1640 3370 1640
 Wire Wire Line
-	2720 1540 3170 1540
-Wire Wire Line
 	3170 1540 3170 1450
-Text Label 3170 1540 2    39   ~ 0
-ID_SC_EEPROM
 $Comp
 L power:+3V3 #PWR?
@@
 F 0 "J27" H 9610 4180 39  0000 C CNN
 F 1 "BlueRobotics Pressure Sense" H 9600 4670 31  0000 C CNN
-F 2 "Connector_Hirose:Hirose_DF13-03P-1.25DS_1x03_P1.25mm_Horizontal" H 9600 4480 50  0001 C CNN
+F 2 "Connector_Hirose:Hirose_DF13-04P-1.25DS_1x04_P1.25mm_Horizontal" H 9600 4480 50  0001 C CNN
 F 3 "~" H 9600 4480 50  0001 C CNN
 F 4 "C597871" H 9600 4480 50  0001 C CNN "LCSC"
@@
 Wire Wire Line
 	9150 5450 8760 5450
-Text Label 1480 3840 0    39   ~ 0
-SDA\GPIO2
-Text Label 1480 3940 0    39   ~ 0
-SCL\GPIO3
 Wire Wire Line
 	5610 3960 5610 4070
@@
 Text GLabel 5960 5630 2    30   Input ~ 0
 LEAK_2
+Text GLabel 3525 1540 2    39   Input ~ 0
+ID_SC_EEPROM
+Text GLabel 3525 1640 2    28   Input ~ 0
+ID_SD_EEPROM\GPIO0
+Wire Wire Line
+	2720 1540 3170 1540
+Connection ~ 3170 1540
+Wire Wire Line
+	3170 1540 3525 1540
+Wire Wire Line
+	3370 1640 3525 1640
+Connection ~ 3370 1640
+$Comp
+L power:GND #PWR?
+U 1 1 600950E2
+P 2420 1030
+AR Path="/600950E2" Ref="#PWR?"  Part="1"
+AR Path="/5F9D87DA/600950E2" Ref="#PWR?"  Part="1"
+AR Path="/5FCB4E5B/600950E2" Ref="#PWR0229"  Part="1"
+F 0 "#PWR0229" H 2420 780 50  0001 C CNN
+F 1 "GND" V 2455 890 31  0000 C CNN
+F 2 "" H 2420 1030 50  0001 C CNN
+F 3 "" H 2420 1030 50  0001 C CNN
+	1    2420 1030
+	0    -1   -1   0
+$EndComp
+Connection ~ 2220 1030
+Wire Wire Line
+	2220 1030 2220 1040
+Wire Wire Line
+	2220 1010 2220 1030
+$Comp
+L Device:C_Small C?
+U 1 1 6008C802
+P 2320 1030
+AR Path="/6008C802" Ref="C?"  Part="1"
+AR Path="/5F9D87DA/6008C802" Ref="C?"  Part="1"
+AR Path="/5FCB4E5B/6008C802" Ref="C27"  Part="1"
+F 0 "C27" V 2430 1000 39  0000 L CNN
+F 1 "0.1u" V 2420 770 35  0000 L CNN
+F 2 "Capacitor_SMD:C_0603_1608Metric" H 2320 1030 50  0001 C CNN
+F 3 "~" H 2320 1030 50  0001 C CNN
+F 4 "C14663" H 2320 1030 50  0001 C CNN "LCSC"
+F 5 "" H 2320 1030 50  0001 C CNN "Digi"
+F 6 "" H 2320 1030 50  0001 C CNN "Desc."
+F 7 "100nF (104) ±10% 50V X7R" H 2320 1030 50  0001 C CNN "Desc"
+	1    2320 1030
+	0    -1   -1   0
+$EndComp
+Text GLabel 5840 1780 2    31   Input ~ 0
+SCL\GPIO3
+Text GLabel 5840 1980 2    31   Input ~ 0
+SDA\GPIO2
+Text GLabel 1480 3840 0    31   Input ~ 0
+SDA\GPIO2
+Text GLabel 1480 3940 0    31   Input ~ 0
+SCL\GPIO3
 $EndSCHEMATC

Commit message: Pi4 Remake Done
Parts:
- removed C27: 0.1u, Capacitor_SMD:C_0603_1608Metric, symbol Device:C_Small
- removed J22: LED, µ104KiCAD_connectors:XT30PW-M, symbol Connector_Generic:Conn_01x02
- removed J30: TEMP, Connector_JST:JST_SH_SM03B-SRSS-TB_1x03-1MP_P1.00mm_Horizontal, symbol Connector_Generic:Conn_01x03
- removed JP2: WP, Jumper:SolderJumper-2_P1.3mm_Open_RoundedPad1.0x1.5mm, symbol Jumper:SolderJumper_2_Open
- removed R10, R9: 3.9k, Resistor_SMD:R_0603_1608Metric, symbol Device:R_Small_US
- removed R11: 10k, Resistor_SMD:R_0603_1608Metric, symbol Device:R_Small_US
- removed U4: CAT24C32, Package_SO:SOIC-8_3.9x4.9mm_P1.27mm, symbol AUV_Pi_Expansion-rescue:CAT24C32-raspberrypi_hat-pitest-rescue-AUV_Pi_Expansion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
- added J16: PWR-, µ104KiCAD_connectors:WtB_Solder_Pad_0.7x0.5, symbol Connector_Generic:Conn_01x01
- added J34: GPIO, Connector_JST:JST_SH_SM03B-SRSS-TB_1x03-1MP_P1.00mm_Horizontal, symbol Connector_Generic:Conn_01x03
- added J35: I2C, Connector_JST:JST_SH_SM03B-SRSS-TB_1x03-1MP_P1.00mm_Horizontal, symbol Connector_Generic:Conn_01x03
- added J5: PWR+, µ104KiCAD_connectors:WtB_Solder_Pad_0.7x0.5, symbol Connector_Generic:Conn_01x01
- J25: value TOF -> TOF1
- J26: value TOF -> TOF2
- J28: value TOF -> TOF3
- J29: value TOF -> TOF4
- J32: value TOF -> TOF5
Connections:
- net GND: now also J34.1 (Pin_1), J35.1 (Pin_1)
- net LED_CTRL: now also J16.1 (Pin_1)
- net LED_PWR: now also J5.1 (Pin_1)
- net SCL\GPIO3: now also J35.2 (Pin_2)
- net SDA\GPIO2: now also J35.3 (Pin_3)
- new net GCLK2\GPIO6: J34.3 (Pin_3)
- new net PWM1\GPIO12: J34.2 (Pin_2)
- no-connect marks 1 -> 0
Other:
- note added: "Alt."
- note added: "Xtra GPIO\n\n"
- note added: "Xtra I2C\n\n"
- note removed: "EEPROM"
- note removed: "Temp\n\n\n"
